File: inputs.sch (KiCad schematic (older format))
At the start: 8 parts, among them U23 2.15K, U25 33k, U27 1NF

Commit message: Fix kicad libs (#14)
* gitignore

* fix tc4427

* fix cache name

* fix 8888

* update lib

* add molex

* fix adc

* update lib

* fix 9201, 4427, digital resistors

* fix usb
Parts:
- removed U23: 2.15K, Resistor_SMD:R_Array_Convex_4x0603, symbol BOSCH_154_PIN:RESISTOR_ARRAY
- removed U25: 33k, Resistor_SMD:R_Array_Convex_4x0603, symbol BOSCH_154_PIN:RESISTOR_ARRAY
- removed U27: 1NF, Resistor_SMD:R_Array_Convex_4x0603, symbol BOSCH_154_PIN:RESISTOR_ARRAY
- added U23: 2.15k, symbol Device:R_Pack04
- added U25: 33k, symbol Device:R_Pack04
- added U27: 1nF, symbol Device:R_Pack04
Changed lines of the file:
@@
 EESchema Schematic File Version 4
-LIBS:MicroRusefi-cache
+LIBS:microRusEfi-cache
 EELAYER 29 0
 EELAYER END
@@
 L power:GND #PWR095
 U 1 1 5C8AAE05
-P 3050 2300
-F 0 "#PWR095" H 3050 2050 50  0001 C CNN
-F 1 "GND" H 3055 2127 50  0000 C CNN
-F 2 "" H 3050 2300 50  0001 C CNN
-F 3 "" H 3050 2300 50  0001 C CNN
-	1    3050 2300
-	1    0    0    -1
-$EndComp
-$Comp
-L BOSCH_154_PIN:RESISTOR_ARRAY U25
-U 1 1 5DC05D63
-P 3750 1450
-F 0 "U25" H 3750 1547 60  0000 C CNN
-F 1 "33k" H 3750 1441 60  0000 C CNN
-F 2 "Resistor_SMD:R_Array_Convex_4x0603" H 3750 1450 60  0001 C CNN
-F 3 "" H 3750 1450 60  0001 C CNN
-	1    3750 1450
-	1    0    0    -1
-$EndComp
-$Comp
-L BOSCH_154_PIN:RESISTOR_ARRAY U23
-U 1 1 5DC064E8
-P 3300 2150
-F 0 "U23" V 3247 2088 60  0000 L CNN
-F 1 "2.15K" V 3353 2088 60  0000 L CNN
-F 2 "Resistor_SMD:R_Array_Convex_4x0603" H 3300 2150 60  0001 C CNN
-F 3 "" H 3300 2150 60  0001 C CNN
-	1    3300 2150
-	0    1    1    0
-$EndComp
-$Comp
-L BOSCH_154_PIN:RESISTOR_ARRAY U27
-U 1 1 5DC06DCD
-P 4700 2150
-F 0 "U27" V 4647 2088 60  0000 L CNN
-F 1 "1NF" V 4753 2088 60  0000 L CNN
-F 2 "Resistor_SMD:R_Array_Convex_4x0603" H 4700 2150 60  0001 C CNN
-F 3 "" H 4700 2150 60  0001 C CNN
-	1    4700 2150
-	0    1    1    0
-$EndComp
-Wire Wire Line
-	3900 1900 4250 1900
-Wire Wire Line
-	3900 1800 4350 1800
-Wire Wire Line
-	3900 1700 4450 1700
-Wire Wire Line
-	3900 1600 4550 1600
-Wire Wire Line
-	4550 2000 4550 1600
-Connection ~ 4550 1600
-Wire Wire Line
-	4550 1600 4950 1600
-Wire Wire Line
-	4450 2000 4450 1700
-Connection ~ 4450 1700
-Wire Wire Line
-	4450 1700 4950 1700
-Wire Wire Line
-	4350 2000 4350 1800
-Connection ~ 4350 1800
-Wire Wire Line
-	4350 1800 4950 1800
-Wire Wire Line
-	4250 2000 4250 1900
-Connection ~ 4250 1900
-Wire Wire Line
-	4250 1900 4950 1900
-Wire Wire Line
-	4550 2300 4450 2300
-Connection ~ 4350 2300
-Wire Wire Line
-	4350 2300 4250 2300
-Connection ~ 4450 2300
-Wire Wire Line
-	4450 2300 4350 2300
-Wire Wire Line
-	2850 2300 2950 2300
-Connection ~ 2950 2300
-Wire Wire Line
-	2950 2300 3050 2300
-Connection ~ 3050 2300
-Wire Wire Line
-	3050 2300 3150 2300
+P 3050 2400
+F 0 "#PWR095" H 3050 2150 50  0001 C CNN
+F 1 "GND" H 3055 2227 50  0000 C CNN
+F 2 "" H 3050 2400 50  0001 C CNN
+F 3 "" H 3050 2400 50  0001 C CNN
+	1    3050 2400
+	1    0    0    -1
+$EndComp
+Wire Wire Line
+	4000 1900 4350 1900
+Wire Wire Line
+	4000 1800 4450 1800
+Wire Wire Line
+	4000 1700 4550 1700
+Wire Wire Line
+	4000 1600 4650 1600
+Wire Wire Line
+	4650 2000 4650 1600
+Connection ~ 4650 1600
+Wire Wire Line
+	4650 1600 5050 1600
+Wire Wire Line
+	4550 2000 4550 1700
+Connection ~ 4550 1700
+Wire Wire Line
+	4550 1700 5050 1700
+Wire Wire Line
+	4450 2000 4450 1800
+Connection ~ 4450 1800
+Wire Wire Line
+	4450 1800 5050 1800
+Wire Wire Line
+	4350 2000 4350 1900
+Connection ~ 4350 1900
+Wire Wire Line
+	4350 1900 5050 1900
+Wire Wire Line
+	4650 2400 4550 2400
+Connection ~ 4550 2400
+Connection ~ 3050 2400
+Wire Wire Line
+	3050 2400 3150 2400
 $Comp
 L power:GND #PWR098
 U 1 1 5DC53ED2
-P 4450 2300
-F 0 "#PWR098" H 4450 2050 50  0001 C CNN
-F 1 "GND" H 4455 2127 50  0000 C CNN
-F 2 "" H 4450 2300 50  0001 C CNN
-F 3 "" H 4450 2300 50  0001 C CNN
-	1    4450 2300
+P 4550 2400
+F 0 "#PWR098" H 4550 2150 50  0001 C CNN
+F 1 "GND" H 4555 2227 50  0000 C CNN
+F 2 "" H 4550 2400 50  0001 C CNN
+F 3 "" H 4550 2400 50  0001 C CNN
+	1    4550 2400
 	1    0    0    -1
 $EndComp
@@
 Text HLabel 2300 1900 0    50   Input ~ 0
 DIGITAL_4
-Text HLabel 4950 1600 2    50   Input ~ 0
+Text HLabel 5050 1600 2    50   Input ~ 0
 DIGITAL_1_MCU
-Text HLabel 4950 1700 2    50   Input ~ 0
+Text HLabel 5050 1700 2    50   Input ~ 0
 DIGITAL_2_MCU
-Text HLabel 4950 1800 2    50   Input ~ 0
+Text HLabel 5050 1800 2    50   Input ~ 0
 DIGITAL_3_MCU
-Text HLabel 4950 1900 2    50   Input ~ 0
+Text HLabel 5050 1900 2    50   Input ~ 0
 DIGITAL_4_MCU
+Wire Wire Line
+	4350 2400 4450 2400
+Wire Wire Line
+	2850 2400 2950 2400
+$Comp
+L Device:R_Pack04 U23
+U 1 1 5CDEE3A2
+P 2950 2200
+F 0 "U23" H 2670 2154 50  0000 R CNN
+F 1 "2.15k" H 2670 2245 50  0000 R CNN
+F 2 "" V 3225 2200 50  0001 C CNN
+F 3 "~" H 2950 2200 50  0001 C CNN
+	1    2950 2200
+	-1   0    0    1
+$EndComp
+$Comp
+L Device:R_Pack04 U27
+U 1 1 5CDEF221
+P 4450 2200
+F 0 "U27" H 4170 2154 50  0000 R CNN
+F 1 "1nF" H 4170 2245 50  0000 R CNN
+F 2 "" V 4725 2200 50  0001 C CNN
+F 3 "~" H 4450 2200 50  0001 C CNN
+	1    4450 2200
+	-1   0    0    1
+$EndComp
+$Comp
+L Device:R_Pack04 U25
+U 1 1 5CDEFC0B
+P 3800 1800
+F 0 "U25" V 3383 1800 50  0000 C CNN
+F 1 "33k" V 3474 1800 50  0000 C CNN
+F 2 "" V 4075 1800 50  0001 C CNN
+F 3 "~" H 3800 1800 50  0001 C CNN
+	1    3800 1800
+	0    1    1    0
+$EndComp
+Connection ~ 2950 2400
+Wire Wire Line
+	2950 2400 3050 2400
+Connection ~ 4450 2400
+Wire Wire Line
+	4450 2400 4550 2400
 $EndSCHEMATC
