File: TLE8888-1QK.sch (KiCad schematic (older format))
At the start: 37 parts, among them Q1 IPD30N06S2L-23, U2 TLE8888QK

Commit message: fix 8888
Parts:
- U2: symbol BOSCH_154_PIN:TLE8888QK -> rusefi_tle8888:TLE8888QK
Changed lines of the file:
@@
 $EndDescr
 $Comp
-L BOSCH_154_PIN:TLE8888QK U2
+L rusefi_tle8888:TLE8888QK U2
 U 1 1 5C5DF903
 P 10150 6950

Commit message: fix 9201, 4427, digital resistors
Parts:
- D2: symbol BOSCH_154_PIN:PESD1CAN-UX -> rusefi_pesd1can:PESD1CAN-UX
Changed lines of the file:
@@
 	14325 7250 14325 7500
 $Comp
-L BOSCH_154_PIN:PESD1CAN-UX D?
+L rusefi_pesd1can:PESD1CAN-UX D?
 U 1 1 5C984DE7
 P 14825 7600

Commit message: latest updates
Parts:
- Q1: footprint Package_TO_SOT_SMD:TO-252-2_THERMAL -> Package_TO_SOT_SMD:TO-252-2
Connections:
- net UBR renamed 12V-SWITCH
Changed lines of the file:
@@
 $Descr User 19685 15748
 encoding utf-8
-Sheet 2 7
+Sheet 2 6
 Title "ME7 ECU"
 Date "2019-01-31"
@@
 Wire Wire Line
 	8000 8900 8000 8800
-Text HLabel 8000 8900 0    60   Input ~ 12
+Text HLabel 6650 7950 0    60   Input ~ 12
 OUT_6
-Text HLabel 8000 8000 0    60   Input ~ 12
+Text HLabel 6650 7650 0    60   Input ~ 12
 OUT_5
 Wire Wire Line
@@
 Wire Wire Line
 	6900 8300 8100 8300
-Wire Wire Line
-	9850 10100 9950 10100
-Wire Wire Line
-	10050 10100 9950 10100
-Connection ~ 9950 10100
 Text HLabel 9950 10100 3    60   Input ~ 12
 OUT_7
@@
 F 0 "Q1" H 9875 11075 50  0000 C CNN
 F 1 "IPD30N06S2L-23" V 10175 11075 50  0000 C CNN
-F 2 "Package_TO_SOT_SMD:TO-252-2_THERMAL" H 10200 11125 50  0001 L CIN
+F 2 "Package_TO_SOT_SMD:TO-252-2" H 10200 11125 50  0001 L CIN
 F 3 "http://www.fairchildsemi.com/ds/BU/BUZ11.pdf" H 9950 11200 50  0001 L CNN
 F 4 "MOUSER" H 0   0   50  0001 C CNN "VEND"
@@
 MAIN_RELAY
 Text HLabel 5550 8600 0    60   Input ~ 12
-UBR
+12V-SWITCH
 Text HLabel 8000 8700 0    60   Input ~ 12
 OUT_21
@@
 Text Label 8650 6650 0    60   ~ 12
 GND
-Text Label 5550 8600 0    60   ~ 12
-UBR
 Wire Wire Line
 	6900 9100 8100 9100
@@
 	0    -1   -1   0
 $EndComp
-Text Label 10500 10850 0    60   ~ 12
-UBR
 Wire Wire Line
 	11150 11650 11150 10725
@@
 $EndComp
 Text Label 10750 5550 0    60   ~ 12
-UBR
+12V-SWITCH
 Wire Wire Line
 	10750 5550 10750 6700
@@
 Wire Wire Line
 	13475 7150 13725 7150
-Text Label 13725 7150 0    60   ~ 12
-UBR
 Wire Notes Line
 	14500 5650 11800 5650
@@
 Text Notes 12550 6800 0    50   ~ 0
 -
+Text Label 13675 7150 0    60   ~ 12
+12V-SWITCH
+Text Label 10500 10850 0    60   ~ 12
+12V-SWITCH
+Text Label 6375 8600 0    60   ~ 12
+12V-SWITCH
+Wire Wire Line
+	8000 8900 7200 8900
+Wire Wire Line
+	7200 8900 7200 7950
+Wire Wire Line
+	7200 7950 6650 7950
+Wire Wire Line
+	8000 8000 7450 8000
+Wire Wire Line
+	7450 8000 7450 7650
+Wire Wire Line
+	7450 7650 6650 7650
+Wire Wire Line
+	9850 10100 10050 10100
 $EndSCHEMATC

Commit message: manual sync with 960
Parts:
- removed R16: 0, Resistor_SMD:R_0603_1608Metric_Pad1.05x0.95mm_HandSolder, symbol Device:R
- added C35: 1nF, Capacitor_SMD:C_0603_1608Metric_Pad1.05x0.95mm_HandSolder, symbol Device:C
- added R15: 15K, Resistor_SMD:R_0603_1608Metric_Pad1.05x0.95mm_HandSolder, symbol Device:R
- added TP3, TP4: TestPoint, symbol Connector:TestPoint
- C1, C10, C13, C14, C16, C4, C5, C6: Manufacturer WURTH -> (none); Part # 885012208087 -> (none); VEND MOUSER -> (none); VEND# 710-885012208087 -> (none)
- C11: Manufacturer WURTH -> (none); Part # 885012208079 -> (none); VEND# 710-885012208079 -> (none)
- C12: value C -> 1nF; Manufacturer WURTH -> (none); Part # 885012208087 -> (none); VEND MOUSER -> (none); VEND# 710-885012208087 -> (none)
- C3: Manufacturer WURTH -> (none); Part # 885012208050 -> (none); VEND# 710-885012208050 -> (none)
- C7, C8, C9: Manufacturer MURATA -> (none); Part # GRT31CR61H106KE01L -> (none); VEND MOUSER -> (none); VEND# 81-GRT31CR61H106KE1L -> (none)
- D2: Status Active -> (none)
- R12, R13: value 0 -> 10K
- R17, R18, R19: value 0 -> DNP
- R9: value 0 -> 5.11K
- U2: Manufacturer INFINEON -> (none)
Connections:
- net CRNK+: now also C35.1, R15.1
- net CRNK-: now also C35.2, R15.2
- net at C12.2, R13.2, R9.2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: now also TP4.1
- net at C12.1, R12.2, R9.1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: now also TP3.1
Other:
- note added: "SEE DATASHEET \nFOR HALL SENSOR USE"
- note removed: "+"
- note removed: "-"

Commit message: Latest (#43)
Parts:
- removed TP3, TP4: TestPoint, symbol Connector:TestPoint
Changed lines of the file:
@@
 $Descr User 19685 15748
 encoding utf-8
-Sheet 2 6
+Sheet 2 7
 Title "microRusEfi"
 Date "2019-01-31"
@@
 U 1 1 5C88CC5C
 P 12000 6400
-F 0 "C12" H 11925 6300 50  0000 C CNN
-F 1 "1nF" V 11900 6500 50  0000 C CNN
+F 0 "C12" H 11975 6175 50  0000 C CNN
+F 1 "1nF" H 11925 6625 50  0000 C CNN
 F 2 "Capacitor_SMD:C_0603_1608Metric_Pad1.05x0.95mm_HandSolder" H 12038 6250 50  0001 C CNN
 F 3 "~" H 12000 6400 50  0001 C CNN
@@
 	11900 6350 11900 6250
 Wire Wire Line
-	11900 6250 11925 6250
-Wire Wire Line
 	11050 6350 11900 6350
 Connection ~ 12000 6250
@@
 Wire Wire Line
 	11900 6450 11900 6550
-Wire Wire Line
-	11900 6550 11925 6550
 Wire Wire Line
 	11150 6450 11900 6450
@@
 Text Notes 13750 6050 0    50   ~ 0
 TRIGGER CONFIG\nAS SEEN\nAT PCB
-Text Label 13350 6800 0    60   ~ 12
+Text Label 13475 6800 0    60   ~ 12
 V5V
-Text Label 13350 6700 0    60   ~ 12
+Text Label 13475 6700 0    60   ~ 12
 GND
 Text Label 13350 5900 0    60   ~ 12
@@
 U 1 1 5D394376
 P 12975 6400
-F 0 "C35" H 12900 6300 50  0000 C CNN
-F 1 "1nF" V 12875 6500 50  0000 C CNN
+F 0 "C35" H 12800 6400 50  0000 C CNN
+F 1 "1nF" H 12950 6625 50  0000 C CNN
 F 2 "Capacitor_SMD:C_0603_1608Metric_Pad1.05x0.95mm_HandSolder" H 13013 6250 50  0001 C CNN
 F 3 "~" H 12975 6400 50  0001 C CNN
@@
 Text Notes 13575 6450 0    50   ~ 0
 SEE DATASHEET \nFOR HALL SENSOR USE
-$Comp
-L Connector:TestPoint TP3
-U 1 1 5D084DE4
-P 11925 6250
-F 0 "TP3" H 11983 6368 50  0000 L CNN
-F 1 "TestPoint" H 11983 6277 50  0000 L CNN
-F 2 "" H 12125 6250 50  0001 C CNN
-F 3 "~" H 12125 6250 50  0001 C CNN
-	1    11925 6250
-	1    0    0    -1
-$EndComp
-Connection ~ 11925 6250
-Wire Wire Line
-	11925 6250 12000 6250
-$Comp
-L Connector:TestPoint TP4
-U 1 1 5D085A43
-P 11925 6550
-F 0 "TP4" H 11867 6576 50  0000 R CNN
-F 1 "TestPoint" H 11867 6667 50  0000 R CNN
-F 2 "" H 12125 6550 50  0001 C CNN
-F 3 "~" H 12125 6550 50  0001 C CNN
-	1    11925 6550
-	-1   0    0    1
-$EndComp
-Connection ~ 11925 6550
-Wire Wire Line
-	11925 6550 12000 6550
+Wire Wire Line
+	11900 6550 12000 6550
+Wire Wire Line
+	11900 6250 12000 6250
+Wire Wire Line
+	13475 6700 13350 6700
+Wire Wire Line
+	13475 6800 13350 6800
 $EndSCHEMATC

Commit message: Latest
Parts:
- C4, C5: value 100nF -> 400nF
Connections:
- net CRNK+: no longer R17.2
Other:
- moved on the sheet: C35, R15, R17
Changed lines of the file:
@@
 P 8000 11800
 F 0 "C4" V 8050 11850 50  0000 L CNN
-F 1 "100nF" V 7875 11800 50  0000 C CNN
+F 1 "400nF" V 7875 11800 50  0000 C CNN
 F 2 "Capacitor_SMD:C_0603_1608Metric_Pad1.05x0.95mm_HandSolder" H 8038 11650 50  0001 C CNN
 F 3 "~" H 8000 11800 50  0001 C CNN
@@
 P 8300 11800
 F 0 "C5" V 8350 11850 50  0000 L CNN
-F 1 "100nF" V 8175 11800 50  0000 C CNN
+F 1 "400nF" V 8175 11800 50  0000 C CNN
 F 2 "Capacitor_SMD:C_0603_1608Metric_Pad1.05x0.95mm_HandSolder" H 8338 11650 50  0001 C CNN
 F 3 "~" H 8300 11800 50  0001 C CNN
@@
 L Device:R R17
 U 1 1 5C8A0B54
-P 13200 5900
-F 0 "R17" V 13250 6075 50  0000 C CNN
-F 1 "DNP" V 13200 5900 50  0000 C CNN
-F 2 "Resistor_SMD:R_0603_1608Metric_Pad1.05x0.95mm_HandSolder" V 13130 5900 50  0001 C CNN
-F 3 "~" H 13200 5900 50  0001 C CNN
-F 4 "MOUSER" H -1250 -450 50  0001 C CNN "VEND"
-	1    13200 5900
+P 11425 5850
+F 0 "R17" V 11475 6025 50  0000 C CNN
+F 1 "DNP" V 11425 5850 50  0000 C CNN
+F 2 "Resistor_SMD:R_0603_1608Metric_Pad1.05x0.95mm_HandSolder" V 11355 5850 50  0001 C CNN
+F 3 "~" H 11425 5850 50  0001 C CNN
+F 4 "MOUSER" H -3025 -500 50  0001 C CNN "VEND"
+	1    11425 5850
 	0    1    1    0
 $EndComp
@@
 	12175 6550 12300 6550
 Wire Wire Line
-	12600 6550 12850 6550
+	12600 6550 12675 6550
 Connection ~ 12850 6550
 Wire Wire Line
-	12600 6250 12850 6250
-Connection ~ 12850 6250
-Wire Wire Line
-	13050 5950 12850 5950
-Wire Wire Line
-	13050 5950 13050 5900
+	11275 5900 11075 5900
+Wire Wire Line
+	11275 5900 11275 5850
 Wire Wire Line
 	13000 6800 13050 6800
@@
 	11150 6500 11150 6450
 Wire Wire Line
-	12850 5950 12850 6250
+	11075 5900 11075 6200
 Wire Wire Line
 	12850 6550 12850 6750
-Wire Wire Line
-	12850 6250 12975 6250
-Wire Wire Line
-	12850 6550 12975 6550
 Connection ~ 12800 7150
 Wire Wire Line
@@
 Text Label 13475 6700 0    60   ~ 12
 GND
-Text Label 13350 5900 0    60   ~ 12
+Text Label 11575 5850 0    60   ~ 12
 V5V
 Text Label 13675 7150 0    60   ~ 12
@@
 L Device:C C35
 U 1 1 5D394376
-P 12975 6400
-F 0 "C35" H 12800 6400 50  0000 C CNN
-F 1 "1nF" H 12950 6625 50  0000 C CNN
-F 2 "Capacitor_SMD:C_0603_1608Metric_Pad1.05x0.95mm_HandSolder" H 13013 6250 50  0001 C CNN
-F 3 "~" H 12975 6400 50  0001 C CNN
-	1    12975 6400
-	1    0    0    -1
-$EndComp
-Connection ~ 12975 6250
-Wire Wire Line
-	12975 6250 13100 6250
-Connection ~ 12975 6550
-Wire Wire Line
-	12975 6550 13100 6550
+P 12675 6400
+F 0 "C35" H 12500 6400 50  0000 C CNN
+F 1 "1nF" H 12650 6625 50  0000 C CNN
+F 2 "Capacitor_SMD:C_0603_1608Metric_Pad1.05x0.95mm_HandSolder" H 12713 6250 50  0001 C CNN
+F 3 "~" H 12675 6400 50  0001 C CNN
+	1    12675 6400
+	1    0    0    -1
+$EndComp
 $Comp
 L Device:R R15
 U 1 1 5D394E3F
-P 13100 6400
-F 0 "R15" V 13175 6400 50  0000 C CNN
-F 1 "15K" V 13100 6400 50  0000 C CNN
-F 2 "Resistor_SMD:R_0603_1608Metric_Pad1.05x0.95mm_HandSolder" V 13030 6400 50  0001 C CNN
-F 3 "~" H 13100 6400 50  0001 C CNN
-F 4 "MOUSER" H -900 -250 50  0001 C CNN "VEND"
-	1    13100 6400
-	1    0    0    -1
-$EndComp
-Connection ~ 13100 6250
-Wire Wire Line
-	13100 6250 13175 6250
-Connection ~ 13100 6550
-Wire Wire Line
-	13100 6550 13175 6550
+P 12800 6400
+F 0 "R15" V 12875 6400 50  0000 C CNN
+F 1 "15K" V 12800 6400 50  0000 C CNN
+F 2 "Resistor_SMD:R_0603_1608Metric_Pad1.05x0.95mm_HandSolder" V 12730 6400 50  0001 C CNN
+F 3 "~" H 12800 6400 50  0001 C CNN
+F 4 "MOUSER" H -1200 -250 50  0001 C CNN "VEND"
+	1    12800 6400
+	1    0    0    -1
+$EndComp
 Text Notes 13575 6450 0    50   ~ 0
 SEE DATASHEET \nFOR HALL SENSOR USE
@@
 Wire Wire Line
 	13475 6800 13350 6800
+Wire Wire Line
+	12600 6250 12675 6250
+Connection ~ 12675 6250
+Wire Wire Line
+	12675 6250 12800 6250
+Connection ~ 12675 6550
+Wire Wire Line
+	12675 6550 12800 6550
+Connection ~ 12800 6250
+Connection ~ 12800 6550
+Wire Wire Line
+	12800 6550 12850 6550
+Wire Wire Line
+	12850 6550 13175 6550
+Wire Wire Line
+	12800 6250 13175 6250
 $EndSCHEMATC
