File: TLE8888-1QK.sch (KiCad schematic (older format))
At the start: 40 parts, among them Q1 IPD30N06S2L-23, U2 TLE8888QK

Commit message: manual sync from jharvey
Other:
- note added: "rusEFI MRE was measured to consume 235mA from the 12V battery, for 2.9 watts"
- moved on the sheet: R12, R13, R15
Changed lines of the file:
@@
 Text HLabel 11500 8350 2    60   Input ~ 12
 IN_12
-Text HLabel 7350 9200 0    60   Input ~ 12
+Text HLabel 8100 9200 0    60   Input ~ 12
 IGN_OUT_1
 Text HLabel 8100 9300 0    60   Input ~ 12
@@
 Wire Wire Line
 	8000 8900 8000 8800
-Text HLabel 6650 7950 0    60   Input ~ 12
+Text HLabel 8000 8900 0    60   Input ~ 12
 OUT_6
-Text HLabel 6650 7650 0    60   Input ~ 12
+Text HLabel 8000 8000 0    60   Input ~ 12
 OUT_5
 Wire Wire Line
@@
 Wire Wire Line
 	10150 10100 10150 10650
-Text HLabel 11150 10575 2    60   Input ~ 12
+Text HLabel 10600 10575 2    60   Input ~ 12
 OUT_19
-Text HLabel 11150 10650 2    60   Input ~ 12
+Text HLabel 10600 10650 2    60   Input ~ 12
 OUT_20
 Text HLabel 9350 6700 1    60   Input ~ 12
@@
 L Device:R R12
 U 1 1 5C89FE8C
-P 12450 6250
-F 0 "R12" V 12500 6425 50  0000 C CNN
-F 1 "10K" V 12450 6250 50  0000 C CNN
-F 2 "Resistor_SMD:R_0603_1608Metric" V 12380 6250 50  0001 C CNN
-F 3 "~" H 12450 6250 50  0001 C CNN
-F 4 "RMCF0603JT10K0" H 0   0   50  0001 C CNN "Part #"
-F 5 "DIGI" H 0   0   50  0001 C CNN "VEND"
-F 6 "RMCF0603JT10K0CT-ND" H 0   0   50  0001 C CNN "VEND#"
-F 7 "StackPole" H 0   0   50  0001 C CNN "Manufacturer"
-	1    12450 6250
+P 12350 6250
+F 0 "R12" V 12400 6425 50  0000 C CNN
+F 1 "10K" V 12350 6250 50  0000 C CNN
+F 2 "Resistor_SMD:R_0603_1608Metric" V 12280 6250 50  0001 C CNN
+F 3 "~" H 12350 6250 50  0001 C CNN
+F 4 "RMCF0603JT10K0" H -100 0   50  0001 C CNN "Part #"
+F 5 "DIGI" H -100 0   50  0001 C CNN "VEND"
+F 6 "RMCF0603JT10K0CT-ND" H -100 0   50  0001 C CNN "VEND#"
+F 7 "StackPole" H -100 0   50  0001 C CNN "Manufacturer"
+	1    12350 6250
 	0    1    1    0
 $EndComp
@@
 L Device:R R13
 U 1 1 5C8A058E
-P 12450 6550
-F 0 "R13" V 12500 6725 50  0000 C CNN
-F 1 "10K" V 12450 6550 50  0000 C CNN
-F 2 "Resistor_SMD:R_0603_1608Metric" V 12380 6550 50  0001 C CNN
-F 3 "~" H 12450 6550 50  0001 C CNN
-F 4 "RMCF0603JT10K0" H 0   0   50  0001 C CNN "Part #"
-F 5 "DIGI" H 0   0   50  0001 C CNN "VEND"
-F 6 "RMCF0603JT10K0CT-ND" H 0   0   50  0001 C CNN "VEND#"
-F 7 "StackPole" H 0   0   50  0001 C CNN "Manufacturer"
-	1    12450 6550
+P 12350 6550
+F 0 "R13" V 12400 6725 50  0000 C CNN
+F 1 "10K" V 12350 6550 50  0000 C CNN
+F 2 "Resistor_SMD:R_0603_1608Metric" V 12280 6550 50  0001 C CNN
+F 3 "~" H 12350 6550 50  0001 C CNN
+F 4 "RMCF0603JT10K0" H -100 0   50  0001 C CNN "Part #"
+F 5 "DIGI" H -100 0   50  0001 C CNN "VEND"
+F 6 "RMCF0603JT10K0CT-ND" H -100 0   50  0001 C CNN "VEND#"
+F 7 "StackPole" H -100 0   50  0001 C CNN "Manufacturer"
+	1    12350 6550
 	0    1    1    0
 $EndComp
@@
 CRNK-
 Wire Wire Line
-	11500 7550 14100 7550
-Wire Wire Line
-	11500 7650 14100 7650
+	11500 7550 14025 7550
+Wire Wire Line
+	11500 7650 14025 7650
 Text HLabel 11500 7850 2    60   Input ~ 12
 CAN_TX
@@
 CAN_RX
 Wire Wire Line
-	14100 7250 14100 7550
-Wire Wire Line
-	14100 7650 14100 7950
-Wire Wire Line
-	14100 7950 14200 7950
+	14025 7250 14025 7550
+Wire Wire Line
+	14025 7650 14025 7950
+Wire Wire Line
+	14025 7950 14200 7950
 Wire Wire Line
 	14325 7950 14325 7700
 Wire Wire Line
-	14100 7250 14200 7250
+	14025 7250 14200 7250
 Wire Wire Line
 	14325 7250 14325 7500
@@
 Text HLabel 9150 10100 3    60   Input ~ 12
 FCLP
-Text HLabel 11150 10375 2    60   Input ~ 12
-CRNK_IN
-Wire Wire Line
-	10550 10375 11150 10375
 Wire Wire Line
 	10850 10100 10850 10300
@@
 	9750 10725 11150 10725
 Wire Wire Line
-	10150 10650 11150 10650
+	10150 10650 10600 10650
 Text Label 11250 10500 0    60   ~ 12
 VDDIO
 Wire Wire Line
-	10550 10100 10550 10375
-Wire Wire Line
-	10250 10575 11150 10575
+	10250 10575 10600 10575
 Wire Wire Line
 	10050 10850 10200 10850
@@
 Text Label 11600 7450 0    60   ~ 12
 WAKE
-Text Label 11800 9550 0    60   ~ 12
+Text Label 12025 9550 0    60   ~ 12
 IGN_EN
 Text Label 11550 10300 0    60   ~ 12
@@
 P 10950 10100
 F 0 "#PWR014" H 10950 9850 50  0001 C CNN
-F 1 "GND" V 10950 9925 50  0000 C CNN
+F 1 "GND" H 10950 9950 50  0000 C CNN
 F 2 "" H 10950 10100 50  0001 C CNN
 F 3 "" H 10950 10100 50  0001 C CNN
@@
 P 10350 10100
 F 0 "#PWR012" H 10350 9850 50  0001 C CNN
-F 1 "GND" V 10350 9925 50  0000 C CNN
+F 1 "GND" H 10350 9950 50  0000 C CNN
 F 2 "" H 10350 10100 50  0001 C CNN
 F 3 "" H 10350 10100 50  0001 C CNN
@@
 P 9050 10350
 F 0 "#PWR08" H 9050 10100 50  0001 C CNN
-F 1 "GND" V 9050 10175 50  0000 C CNN
+F 1 "GND" H 9050 10200 50  0000 C CNN
 F 2 "" H 9050 10350 50  0001 C CNN
 F 3 "" H 9050 10350 50  0001 C CNN
@@
 P 13300 7450
 F 0 "#PWR021" H 13300 7200 50  0001 C CNN
-F 1 "GND" V 13350 7350 50  0000 C CNN
+F 1 "GND" H 13300 7325 50  0000 C CNN
 F 2 "" H 13300 7450 50  0001 C CNN
 F 3 "" H 13300 7450 50  0001 C CNN
@@
 	13025 7450 13300 7450
 Connection ~ 13300 7450
-Wire Wire Line
-	8100 9200 7350 9200
 $Comp
 L Device:R R7
@@
 Connection ~ 12175 6250
 Wire Wire Line
-	12175 6250 12300 6250
+	12175 6250 12200 6250
 Wire Wire Line
 	11900 6450 11900 6550
@@
 Connection ~ 12175 6550
 Wire Wire Line
-	12175 6550 12300 6550
-Wire Wire Line
-	12600 6550 12675 6550
+	12175 6550 12200 6550
+Wire Wire Line
+	12500 6550 12675 6550
 Connection ~ 12850 6550
 Wire Wire Line
@@
 Text Label 10500 10850 0    60   ~ 12
 12V-SWITCH
-Text Label 6375 8600 0    60   ~ 12
+Text Label 6250 8600 0    60   ~ 12
 12V-SWITCH
-Wire Wire Line
-	8000 8900 7200 8900
-Wire Wire Line
-	7200 8900 7200 7950
-Wire Wire Line
-	7200 7950 6650 7950
-Wire Wire Line
-	8000 8000 7450 8000
-Wire Wire Line
-	7450 8000 7450 7650
-Wire Wire Line
-	7450 7650 6650 7650
 Wire Wire Line
 	9850 10100 10050 10100
@@
 L Device:R R15
 U 1 1 5D394E3F
-P 12800 6400
-F 0 "R15" V 12875 6400 50  0000 C CNN
-F 1 "15K" V 12800 6400 50  0000 C CNN
-F 2 "Resistor_SMD:R_0603_1608Metric" V 12730 6400 50  0001 C CNN
-F 3 "~" H 12800 6400 50  0001 C CNN
-F 4 "DIGI" H -1200 -250 50  0001 C CNN "VEND"
-F 5 "RMCF0603JG15K0" H 0   0   50  0001 C CNN "Part #"
-F 6 "RMCF0603JG15K0CT-ND" H 0   0   50  0001 C CNN "VEND#"
-F 7 "StackPole" H 0   0   50  0001 C CNN "Manufacturer"
-	1    12800 6400
+P 12850 6400
+F 0 "R15" V 12925 6400 50  0000 C CNN
+F 1 "15K" V 12850 6400 50  0000 C CNN
+F 2 "Resistor_SMD:R_0603_1608Metric" V 12780 6400 50  0001 C CNN
+F 3 "~" H 12850 6400 50  0001 C CNN
+F 4 "DIGI" H -1150 -250 50  0001 C CNN "VEND"
+F 5 "RMCF0603JG15K0" H 50  0   50  0001 C CNN "Part #"
+F 6 "RMCF0603JG15K0CT-ND" H 50  0   50  0001 C CNN "VEND#"
+F 7 "StackPole" H 50  0   50  0001 C CNN "Manufacturer"
+	1    12850 6400
 	1    0    0    -1
 $EndComp
@@
 	13475 6800 13350 6800
 Wire Wire Line
-	12600 6250 12675 6250
+	12500 6250 12675 6250
 Connection ~ 12675 6250
 Wire Wire Line
@@
 Connection ~ 12675 6550
 Wire Wire Line
-	12675 6550 12800 6550
-Connection ~ 12800 6250
-Connection ~ 12800 6550
-Wire Wire Line
-	12800 6550 12850 6550
+	12675 6550 12850 6550
+Connection ~ 12850 6250
 Wire Wire Line
 	12850 6550 13175 6550
 Wire Wire Line
-	12800 6250 13175 6250
+	12850 6250 13175 6250
 Connection ~ 12725 6250
 Wire Wire Line
-	12725 6250 12800 6250
+	12725 6250 12850 6250
 $Comp
 L Mechanical:Fiducial FID3
@@
 	1    0    0    -1
 $EndComp
+Text Notes 8250 5175 0    50   ~ 0
+rusEFI MRE was measured to consume 235mA from the 12V battery, for 2.9 watts
+Text HLabel 10600 10375 2    60   Input ~ 12
+CRNK_IN
+Wire Wire Line
+	10550 10100 10550 10375
+Wire Wire Line
+	10550 10375 10600 10375
 $EndSCHEMATC
