File: TLE9201SG.sch (KiCad schematic (older format))
At the start: 6 parts, among them U4 TLE9201SG

Commit message: fix 9201, 4427, digital resistors
Parts:
- U4: symbol BOSCH_154_PIN:TLE9201SG -> rusefi_tle9201:TLE9201SG
Changed lines of the file:
@@
 	7400 3750 7600 3750
 $Comp
-L BOSCH_154_PIN:TLE9201SG U4
+L rusefi_tle9201:TLE9201SG U4
 U 1 1 5DE44E83
 P 5525 3100

Commit message: Latest schematics
Connections:
- net UBR renamed 12V
Changed lines of the file:
@@
 $Descr A4 11693 8268
 encoding utf-8
-Sheet 7 7
+Sheet 4 6
 Title ""
 Date ""
@@
 OUT1
 Text HLabel 4675 3550 0    50   Input ~ 0
-UBR
+12V
 Text HLabel 4675 3350 0    50   Input ~ 0
 VDD

Commit message: Update of returning faults each pull (#21)
Parts:
- C19: footprint Capacitor_SMD:C_0805_2012Metric_Pad1.15x1.40mm_HandSolder -> Capacitor_SMD:C_0603_1608Metric_Pad1.05x0.95mm_HandSolder
- R42: footprint Resistor_SMD:R_0805_2012Metric_Pad1.15x1.40mm_HandSolder -> Resistor_SMD:R_0603_1608Metric_Pad1.05x0.95mm_HandSolder
Changed lines of the file:
@@
-EESchema Schematic File Version 5
+EESchema Schematic File Version 4
 LIBS:microRusEfi-cache
 EELAYER 29 0
@@
 encoding utf-8
 Sheet 4 6
-Title ""
+Title "microRusEfi"
 Date ""
 Rev ""
@@
 F 0 "R42" H 7200 4150 50  0000 C CNN
 F 1 "4.7K" V 7100 4000 50  0000 C CNN
-F 2 "Resistor_SMD:R_0805_2012Metric_Pad1.15x1.40mm_HandSolder" H 7100 4000 50  0001 C CNN
+F 2 "Resistor_SMD:R_0603_1608Metric_Pad1.05x0.95mm_HandSolder" H 7100 4000 50  0001 C CNN
 F 3 "~" H 7100 4000 50  0001 C CNN
 F 4 "MOUSER" H 1800 450 50  0001 C CNN "VEND"
@@
 F 0 "C19" H 7500 4100 50  0000 C CNN
 F 1 "10nF" H 7500 3900 50  0000 C CNN
-F 2 "Capacitor_SMD:C_0805_2012Metric_Pad1.15x1.40mm_HandSolder" H 7400 4000 50  0001 C CNN
+F 2 "Capacitor_SMD:C_0603_1608Metric_Pad1.05x0.95mm_HandSolder" H 7400 4000 50  0001 C CNN
 F 3 "~" H 7400 4000 50  0001 C CNN
 F 4 "WURTH" H 1800 450 50  0001 C CNN "Manufacturer"

Commit message: manual sync with 960
Parts:
- C19: Manufacturer WURTH -> (none); Part # 885012208052 -> (none); VEND MOUSER -> (none); VEND# 710-885012208052 -> (none)
- U4: Part # (none) -> 726-TLE9201SG
Changed lines of the file:
@@
 F 2 "Capacitor_SMD:C_0603_1608Metric_Pad1.05x0.95mm_HandSolder" H 7400 4000 50  0001 C CNN
 F 3 "~" H 7400 4000 50  0001 C CNN
-F 4 "WURTH" H 1800 450 50  0001 C CNN "Manufacturer"
-F 5 "885012208052" H 1800 450 50  0001 C CNN "Part #"
-F 6 "MOUSER" H 1800 450 50  0001 C CNN "VEND"
-F 7 "710-885012208052" H 1800 450 50  0001 C CNN "VEND#"
 	1    7400 4000
 	1    0    0    -1
@@
 F 2 "Package_SO:Infineon_PG-DSO-12-11" H 5525 3100 50  0001 C CNN
 F 3 "" H 5525 3100 50  0001 C CNN
+F 4 "726-TLE9201SG" H 0   0   50  0001 C CNN "Part #"
 	1    5525 3100
 	1    0    0    -1

Commit message: Update (#46)
Changed lines of the file:
@@
 Comment4 ""
 $EndDescr
-Text HLabel 7600 3750 2    50   Input ~ 0
+Text HLabel 7600 3750 2    50   Input ~ 6
 OUT2
-Text HLabel 7600 4250 2    50   Input ~ 0
+Text HLabel 7600 4250 2    50   Input ~ 6
 OUT1
-Text HLabel 4675 3550 0    50   Input ~ 0
+Text HLabel 4675 3550 0    50   Input ~ 6
 12V
-Text HLabel 4675 3350 0    50   Input ~ 0
+Text HLabel 4675 3350 0    50   Input ~ 6
 VDD
-Text HLabel 4675 3250 0    50   Input ~ 0
+Text HLabel 4675 3250 0    50   Input ~ 6
 DIR
-Text HLabel 4675 3450 0    50   Input ~ 0
+Text HLabel 4675 3450 0    50   Input ~ 6
 SO
-Text HLabel 6750 3250 2    50   Input ~ 0
+Text HLabel 6750 3250 2    50   Input ~ 6
 PWM
-Text HLabel 6750 3350 2    50   Input ~ 0
+Text HLabel 6750 3350 2    50   Input ~ 6
 DIS
-Text HLabel 6750 3450 2    50   Input ~ 0
+Text HLabel 6750 3450 2    50   Input ~ 6
 SCK
-Text HLabel 6750 3550 2    50   Input ~ 0
+Text HLabel 6750 3550 2    50   Input ~ 6
 CS
-Text HLabel 6750 3650 2    50   Input ~ 0
+Text HLabel 6750 3650 2    50   Input ~ 6
 SI
-Text HLabel 4675 3750 0    50   Input ~ 0
+Text HLabel 4675 3750 0    50   Input ~ 6
 GND
 Wire Wire Line
@@
 Wire Wire Line
 	6125 3750 7100 3750
-Text Label 5325 3650 2    50   ~ 0
+Text Label 5325 3650 2    50   ~ 6
 OUT1
-Text Label 7100 4250 2    50   ~ 0
+Text Label 7100 4250 2    50   ~ 6
 OUT1
 Connection ~ 5150 3350
