File: TLE9201SG.sch (KiCad schematic (older format))
At the start: 7 parts, among them U4 TLE9201SG

Commit message: ETB part number should be C112633? #133
Parts:
- U4: LCSC (none) -> C112633
Changed lines of the file:
@@
 EESchema Schematic File Version 4
-EELAYER 30 0
+LIBS:microRusEfi-cache
+EELAYER 29 0
 EELAYER END
 $Descr A 11000 8500
@@
 F 6 "TLE9201SGAUMA1CT-ND" H 0   0   50  0001 C CNN "VEND#"
 F 7 "Infineon " H 0   0   50  0001 C CNN "Manufacturer"
+F 8 "C112633" H 5525 3100 50  0001 C CNN "LCSC"
 	1    5525 3100
 	1    0    0    -1
