File: hi-lo.sch (KiCad schematic (older format))
At the start: 25 parts, among them P1 CONN_3, P2 CONN_3, U31 TC4427, U32 TC4427, U33 TC4427

Commit message: Fix kicad libs (#14)
* gitignore

* fix tc4427

* fix cache name

* fix 8888

* update lib

* add molex

* fix adc

* update lib

* fix 9201, 4427, digital resistors

* fix usb
Parts:
- U31, U32, U33: symbol tc4427:TC4427 -> rusefi_tc4427:TC4427
Changed lines of the file:
@@
 EESchema Schematic File Version 4
-LIBS:MicroRusefi-cache
+LIBS:microRusEfi-cache
 EELAYER 29 0
 EELAYER END
@@
 $EndComp
 $Comp
-L tc4427:TC4427 U33
+L rusefi_tc4427:TC4427 U33
 U 1 1 5D14ADC4
 P 6500 7950
@@
 $EndComp
 $Comp
-L tc4427:TC4427 U32
+L rusefi_tc4427:TC4427 U32
 U 1 1 5D14F506
 P 6450 6750
@@
 $EndComp
 $Comp
-L tc4427:TC4427 U31
+L rusefi_tc4427:TC4427 U31
 U 1 1 5D15756C
 P 6400 5400

Commit message: Latest schematics
Connections:
- net IGN_5 renamed HS1
- net IGN_5_MCU renamed HS1_MCU
- net IGN_6 renamed HS2
- net IGN_6_MCU renamed HS2_MCU
Changed lines of the file:
@@
 $Descr B 17000 11000
 encoding utf-8
-Sheet 3 7
+Sheet 3 6
 Title "frankenso"
 Date "2019-04-12"
@@
 IGN_4
 Text HLabel 7800 7700 2    60   Input ~ 0
-IGN_5
+HS1
 Text HLabel 7800 8300 2    60   Input ~ 0
-IGN_6
+HS2
 Text HLabel 5150 5350 0    60   Input ~ 0
 IGN_1_MCU
@@
 IGN_4_MCU
 Text HLabel 5250 7900 0    60   Input ~ 0
-IGN_5_MCU
+HS1_MCU
 Text HLabel 5250 8100 0    60   Input ~ 0
-IGN_6_MCU
+HS2_MCU
 Wire Wire Line
 	4350 6300 4350 6800

Commit message: manual sync with 960
Parts:
- C17, C78: value 0.1uF -> 10nF; MFG,MFG# AVX,08055C104KAT2A -> (none); VEND1,VEND1# DIGI,478-1395-1-ND -> (none)
- P1, P2: MFG,MFG# DNP,DNP -> (none); VEND1,VEND1# DNP,DNP -> (none); VEND2,VEND2# , -> (none)
- R104, R105, R106, R107, R108, R109: MFG,MFG# Panasonic,ECG ERJ-6ENF20R0V -> (none); VEND1,VEND1# DIGI,ERJ-6ENF20R0V -> (none)
- R112, R113, R114, R115, R116, R117: MFG,MFG# Panasonic,ERA-6AEB102V -> (none); VEND1,VEND1# DIGI,P1.0KDACT-ND -> (none)
- R120, R121, R122, R123, R124, R125: MFG,MFG# PANASONIC,ERJ-6ENF1000V -> (none); VEND1,VEND1# DIGI,P100CTR-ND -> (none)
- U31, U32, U33: MFG,MFG# MICROCHIP,TC4427AVOA -> (none); Part # (none) -> 579-TC4427EOA; VEND# (none) -> 579-TC4427EOA; VEND1,VEND1# MOUSER,579-TC4427AVOA -> (none)
Changed lines of the file:
@@
 F 2 "Resistor_SMD:R_0603_1608Metric_Pad1.05x0.95mm_HandSolder" V 980 3050 60  0001 C CNN
 F 3 "" H 7650 8300 60  0001 C CNN
-F 4 "PANASONIC,ERJ-6ENF1000V" V 980 3050 60  0001 C CNN "MFG,MFG#"
-F 5 "DIGI,P100CTR-ND" V 980 3050 60  0001 C CNN "VEND1,VEND1#"
 	1    7650 8300
 	0    1    1    0
@@
 F 2 "Resistor_SMD:R_0603_1608Metric_Pad1.05x0.95mm_HandSolder" V 980 3050 60  0001 C CNN
 F 3 "" H 7650 7700 60  0001 C CNN
-F 4 "PANASONIC,ERJ-6ENF1000V" V 980 3050 60  0001 C CNN "MFG,MFG#"
-F 5 "DIGI,P100CTR-ND" V 980 3050 60  0001 C CNN "VEND1,VEND1#"
 	1    7650 7700
 	0    1    -1   0
@@
 F 2 "Package_SO:SO-8_3.9x4.9mm_P1.27mm" H 6500 7950 60  0001 C CNN
 F 3 "" H 6500 7950 60  0000 C CNN
-F 4 "MICROCHIP,TC4427AVOA" H 6500 7950 60  0001 C CNN "MFG,MFG#"
-F 5 "MOUSER,579-TC4427AVOA" H 6500 7950 60  0001 C CNN "VEND1,VEND1#"
+F 4 "579-TC4427EOA" H 0   0   50  0001 C CNN "Part #"
+F 5 "579-TC4427EOA" H 0   0   50  0001 C CNN "VEND#"
 	1    6500 7950
 	1    0    0    -1
@@
 F 2 "Resistor_SMD:R_0603_1608Metric_Pad1.05x0.95mm_HandSolder" V -770 5150 60  0001 C CNN
 F 3 "" H 5900 8000 60  0001 C CNN
-F 4 "Panasonic,ERA-6AEB102V" V -770 5150 60  0001 C CNN "MFG,MFG#"
-F 5 "DIGI,P1.0KDACT-ND" V -770 5150 60  0001 C CNN "VEND1,VEND1#"
 	1    5900 8000
 	0    1    -1   0
@@
 F 2 "Resistor_SMD:R_0603_1608Metric_Pad1.05x0.95mm_HandSolder" V -1270 5050 60  0001 C CNN
 F 3 "" H 5400 7900 60  0001 C CNN
-F 4 "Panasonic,ECG ERJ-6ENF20R0V" V -1270 5050 60  0001 C CNN "MFG,MFG#"
-F 5 "DIGI,ERJ-6ENF20R0V" V -1270 5050 60  0001 C CNN "VEND1,VEND1#"
 	1    5400 7900
 	0    1    -1   0
@@
 F 2 "Resistor_SMD:R_0603_1608Metric_Pad1.05x0.95mm_HandSolder" V -770 5350 60  0001 C CNN
 F 3 "" H 5900 8200 60  0001 C CNN
-F 4 "Panasonic,ERA-6AEB102V" V -770 5350 60  0001 C CNN "MFG,MFG#"
-F 5 "DIGI,P1.0KDACT-ND" V -770 5350 60  0001 C CNN "VEND1,VEND1#"
 	1    5900 8200
 	0    1    -1   0
@@
 F 2 "Resistor_SMD:R_0603_1608Metric_Pad1.05x0.95mm_HandSolder" V -1270 5250 60  0001 C CNN
 F 3 "" H 5400 8100 60  0001 C CNN
-F 4 "Panasonic,ECG ERJ-6ENF20R0V" V -1270 5250 60  0001 C CNN "MFG,MFG#"
-F 5 "DIGI,ERJ-6ENF20R0V" V -1270 5250 60  0001 C CNN "VEND1,VEND1#"
 	1    5400 8100
 	0    1    -1   0
@@
 F 2 "Resistor_SMD:R_0603_1608Metric_Pad1.05x0.95mm_HandSolder" V 930 1850 60  0001 C CNN
 F 3 "" H 7600 7100 60  0001 C CNN
-F 4 "PANASONIC,ERJ-6ENF1000V" V 930 1850 60  0001 C CNN "MFG,MFG#"
-F 5 "DIGI,P100CTR-ND" V 930 1850 60  0001 C CNN "VEND1,VEND1#"
 	1    7600 7100
 	0    1    1    0
@@
 F 2 "Resistor_SMD:R_0603_1608Metric_Pad1.05x0.95mm_HandSolder" V 930 1850 60  0001 C CNN
 F 3 "" H 7600 6500 60  0001 C CNN
-F 4 "PANASONIC,ERJ-6ENF1000V" V 930 1850 60  0001 C CNN "MFG,MFG#"
-F 5 "DIGI,P100CTR-ND" V 930 1850 60  0001 C CNN "VEND1,VEND1#"
 	1    7600 6500
 	0    1    -1   0
@@
 F 2 "Package_SO:SO-8_3.9x4.9mm_P1.27mm" H 6450 6750 60  0001 C CNN
 F 3 "" H 6450 6750 60  0000 C CNN
-F 4 "MICROCHIP,TC4427AVOA" H 6450 6750 60  0001 C CNN "MFG,MFG#"
-F 5 "MOUSER,579-TC4427AVOA" H 6450 6750 60  0001 C CNN "VEND1,VEND1#"
+F 4 "579-TC4427EOA" H 0   0   50  0001 C CNN "Part #"
+F 5 "579-TC4427EOA" H 0   0   50  0001 C CNN "VEND#"
 	1    6450 6750
 	1    0    0    -1
@@
 F 2 "Resistor_SMD:R_0603_1608Metric_Pad1.05x0.95mm_HandSolder" V -820 3950 60  0001 C CNN
 F 3 "" H 5850 6800 60  0001 C CNN
-F 4 "Panasonic,ERA-6AEB102V" V -820 3950 60  0001 C CNN "MFG,MFG#"
-F 5 "DIGI,P1.0KDACT-ND" V -820 3950 60  0001 C CNN "VEND1,VEND1#"
 	1    5850 6800
 	0    1    -1   0
@@
 F 2 "Resistor_SMD:R_0603_1608Metric_Pad1.05x0.95mm_HandSolder" V -1320 3850 60  0001 C CNN
 F 3 "" H 5350 6700 60  0001 C CNN
-F 4 "Panasonic,ECG ERJ-6ENF20R0V" V -1320 3850 60  0001 C CNN "MFG,MFG#"
-F 5 "DIGI,ERJ-6ENF20R0V" V -1320 3850 60  0001 C CNN "VEND1,VEND1#"
 	1    5350 6700
 	0    1    -1   0
@@
 F 2 "Resistor_SMD:R_0603_1608Metric_Pad1.05x0.95mm_HandSolder" V -820 4150 60  0001 C CNN
 F 3 "" H 5850 7000 60  0001 C CNN
-F 4 "Panasonic,ERA-6AEB102V" V -820 4150 60  0001 C CNN "MFG,MFG#"
-F 5 "DIGI,P1.0KDACT-ND" V -820 4150 60  0001 C CNN "VEND1,VEND1#"
 	1    5850 7000
 	0    1    -1   0
@@
 F 2 "Resistor_SMD:R_0603_1608Metric_Pad1.05x0.95mm_HandSolder" V -1320 4050 60  0001 C CNN
 F 3 "" H 5350 6900 60  0001 C CNN
-F 4 "Panasonic,ECG ERJ-6ENF20R0V" V -1320 4050 60  0001 C CNN "MFG,MFG#"
-F 5 "DIGI,ERJ-6ENF20R0V" V -1320 4050 60  0001 C CNN "VEND1,VEND1#"
 	1    5350 6900
 	0    1    -1   0
@@
 P 4200 6800
 F 0 "C78" V 4250 6850 40  0000 L CNN
-F 1 "0.1uF" V 4250 6550 40  0000 L CNN
+F 1 "10nF" V 4250 6550 40  0000 L CNN
 F 2 "Capacitor_SMD:C_0603_1608Metric_Pad1.05x0.95mm_HandSolder" V -2120 1850 60  0001 C CNN
 F 3 "" H 4200 6800 60  0001 C CNN
-F 4 "AVX,08055C104KAT2A" V -2120 1850 60  0001 C CNN "MFG,MFG#"
-F 5 "DIGI,478-1395-1-ND" V -2120 1850 60  0001 C CNN "VEND1,VEND1#"
 	1    4200 6800
 	0    1    -1   0
@@
 F 2 "Resistor_SMD:R_0603_1608Metric_Pad1.05x0.95mm_HandSolder" V 880 500 60  0001 C CNN
 F 3 "" H 7550 5750 60  0001 C CNN
-F 4 "PANASONIC,ERJ-6ENF1000V" V 880 500 60  0001 C CNN "MFG,MFG#"
-F 5 "DIGI,P100CTR-ND" V 880 500 60  0001 C CNN "VEND1,VEND1#"
 	1    7550 5750
 	0    1    1    0
@@
 F 2 "Resistor_SMD:R_0603_1608Metric_Pad1.05x0.95mm_HandSolder" V 880 500 60  0001 C CNN
 F 3 "" H 7550 5150 60  0001 C CNN
-F 4 "PANASONIC,ERJ-6ENF1000V" V 880 500 60  0001 C CNN "MFG,MFG#"
-F 5 "DIGI,P100CTR-ND" V 880 500 60  0001 C CNN "VEND1,VEND1#"
 	1    7550 5150
 	0    1    -1   0
@@
 F 2 "Package_SO:SO-8_3.9x4.9mm_P1.27mm" H 6400 5400 60  0001 C CNN
 F 3 "" H 6400 5400 60  0000 C CNN
-F 4 "MICROCHIP,TC4427AVOA" H 6400 5400 60  0001 C CNN "MFG,MFG#"
-F 5 "MOUSER,579-TC4427AVOA" H 6400 5400 60  0001 C CNN "VEND1,VEND1#"
+F 4 "579-TC4427EOA" H 0   0   50  0001 C CNN "Part #"
+F 5 "579-TC4427EOA" H 0   0   50  0001 C CNN "VEND#"
 	1    6400 5400
 	1    0    0    -1
@@
 F 2 "Jumper:SolderJumper-3_P1.3mm_Open_RoundedPad1.0x1.5mm" V 1055 3200 60  0001 C CNN
 F 3 "" H 4575 3225 60  0001 C CNN
-F 4 "DNP,DNP" V 1055 3200 60  0001 C CNN "MFG,MFG#"
-F 5 "DNP,DNP" V 1055 3200 60  0001 C CNN "VEND1,VEND1#"
-F 6 "," H 4575 3225 60  0001 C CNN "VEND2,VEND2#"
 	1    3150 7300
 	0    -1   -1   0
@@
 F 2 "Resistor_SMD:R_0603_1608Metric_Pad1.05x0.95mm_HandSolder" V -870 2600 60  0001 C CNN
 F 3 "" H 5800 5450 60  0001 C CNN
-F 4 "Panasonic,ERA-6AEB102V" V -870 2600 60  0001 C CNN "MFG,MFG#"
-F 5 "DIGI,P1.0KDACT-ND" V -870 2600 60  0001 C CNN "VEND1,VEND1#"
 	1    5800 5450
 	0    1    -1   0
@@
 F 2 "Resistor_SMD:R_0603_1608Metric_Pad1.05x0.95mm_HandSolder" V -1370 2500 60  0001 C CNN
 F 3 "" H 5300 5350 60  0001 C CNN
-F 4 "Panasonic,ECG ERJ-6ENF20R0V" V -1370 2500 60  0001 C CNN "MFG,MFG#"
-F 5 "DIGI,ERJ-6ENF20R0V" V -1370 2500 60  0001 C CNN "VEND1,VEND1#"
 	1    5300 5350
 	0    1    -1   0
@@
 F 2 "Resistor_SMD:R_0603_1608Metric_Pad1.05x0.95mm_HandSolder" V -870 2800 60  0001 C CNN
 F 3 "" H 5800 5650 60  0001 C CNN
-F 4 "Panasonic,ERA-6AEB102V" V -870 2800 60  0001 C CNN "MFG,MFG#"
-F 5 "DIGI,P1.0KDACT-ND" V -870 2800 60  0001 C CNN "VEND1,VEND1#"
 	1    5800 5650
 	0    1    -1   0
@@
 F 2 "Resistor_SMD:R_0603_1608Metric_Pad1.05x0.95mm_HandSolder" V -1370 2700 60  0001 C CNN
 F 3 "" H 5300 5550 60  0001 C CNN
-F 4 "Panasonic,ECG ERJ-6ENF20R0V" V -1370 2700 60  0001 C CNN "MFG,MFG#"
-F 5 "DIGI,ERJ-6ENF20R0V" V -1370 2700 60  0001 C CNN "VEND1,VEND1#"
 	1    5300 5550
 	0    1    -1   0
@@
 F 2 "Jumper:SolderJumper-3_P1.3mm_Open_RoundedPad1.0x1.5mm" V 1055 850 60  0001 C CNN
 F 3 "" H 4575 875 60  0001 C CNN
-F 4 "DNP,DNP" V 1055 850 60  0001 C CNN "MFG,MFG#"
-F 5 "DNP,DNP" V 1055 850 60  0001 C CNN "VEND1,VEND1#"
-F 6 "," H 4575 875 60  0001 C CNN "VEND2,VEND2#"
 	1    3150 4950
 	0    -1   -1   0
@@
 P 4000 5100
 F 0 "C17" V 4050 5150 40  0000 L CNN
-F 1 "0.1uF" V 4050 4850 40  0000 L CNN
+F 1 "10nF" V 4050 4850 40  0000 L CNN
 F 2 "Capacitor_SMD:C_0603_1608Metric_Pad1.05x0.95mm_HandSolder" V -2320 150 60  0001 C CNN
 F 3 "" H 4000 5100 60  0001 C CNN
-F 4 "AVX,08055C104KAT2A" V -2320 150 60  0001 C CNN "MFG,MFG#"
-F 5 "DIGI,478-1395-1-ND" V -2320 150 60  0001 C CNN "VEND1,VEND1#"
 	1    4000 5100
 	-1   0    0    -1

Commit message: Latest
Parts:
- removed P1, P2: CONN_3, Jumper:SolderJumper-3_P1.3mm_Open_RoundedPad1.0x1.5mm, symbol Jumper:Jumper_3_Open
- added R57: DNP, Resistor_SMD:R_0603_1608Metric_Pad1.05x0.95mm_HandSolder, symbol Device:R
- added R59: 0R, Resistor_SMD:R_0603_1608Metric_Pad1.05x0.95mm_HandSolder, symbol Device:R
Connections:
- net 12V: now also R59.1
- net 5V: now also C78.1, U32.6 (VDD), U33.6 (VDD), R57.2
- net at C17.1, U31.6 (VDD): now also R57.1, R59.2
Changed lines of the file:
@@
 $Descr B 17000 11000
 encoding utf-8
-Sheet 3 6
+Sheet 3 7
 Title "microRusEfi"
 Date "2019-04-12"
@@
 	1    0    0    -1
 $EndComp
-Text HLabel 3150 7550 2    60   Input ~ 0
-12V
-Text HLabel 3150 7050 2    60   Input ~ 0
+Text HLabel 4350 7150 2    60   Input ~ 0
 5V
-$Comp
-L Jumper:Jumper_3_Open P1
-U 1 1 5D157586
-P 3150 7300
-F 0 "P1" V 3100 7300 50  0000 C CNN
-F 1 "CONN_3" V 3200 7300 40  0000 C CNN
-F 2 "Jumper:SolderJumper-3_P1.3mm_Open_RoundedPad1.0x1.5mm" V 1055 3200 60  0001 C CNN
-F 3 "" H 4575 3225 60  0001 C CNN
-	1    3150 7300
-	0    -1   -1   0
-$EndComp
 $Comp
 L Device:R R112
@@
 Wire Wire Line
 	7400 5150 7300 5150
-Wire Wire Line
-	3300 7300 4350 7300
 Wire Wire Line
 	5450 5350 5550 5350
@@
 Wire Wire Line
 	4350 6300 6900 6300
-Connection ~ 4350 7300
-Wire Wire Line
-	4350 7300 4350 7500
 Connection ~ 4350 6800
-Wire Wire Line
-	4350 6800 4350 7300
-$Comp
-L Jumper:Jumper_3_Open P2
-U 1 1 5DFEE1CB
-P 3150 4950
-F 0 "P2" V 3100 4950 50  0000 C CNN
-F 1 "CONN_3" V 3200 4950 40  0000 C CNN
-F 2 "Jumper:SolderJumper-3_P1.3mm_Open_RoundedPad1.0x1.5mm" V 1055 850 60  0001 C CNN
-F 3 "" H 4575 875 60  0001 C CNN
-	1    3150 4950
-	0    -1   -1   0
-$EndComp
-Wire Wire Line
-	3300 4950 4000 4950
-Text Label 3150 4700 0    50   ~ 0
+Text Label 3100 4650 0    50   ~ 0
 5V
-Text Label 3150 5200 0    50   ~ 0
-12V
 $Comp
 L Device:C C17
@@
 Wire Wire Line
 	4000 4950 6850 4950
+Wire Wire Line
+	4350 6800 4350 7500
+$Comp
+L Device:R R59
+U 1 1 5D2B3D8E
+P 3100 5100
+F 0 "R59" V 3175 5100 40  0000 C CNN
+F 1 "0R" V 3107 5101 40  0000 C CNN
+F 2 "Resistor_SMD:R_0603_1608Metric_Pad1.05x0.95mm_HandSolder" V -3570 2250 60  0001 C CNN
+F 3 "" H 3100 5100 60  0001 C CNN
+	1    3100 5100
+	1    0    0    1
+$EndComp
+$Comp
+L Device:R R57
+U 1 1 5D2B6FCF
+P 3100 4800
+F 0 "R57" V 3175 4800 40  0000 C CNN
+F 1 "DNP" V 3107 4801 40  0000 C CNN
+F 2 "Resistor_SMD:R_0603_1608Metric_Pad1.05x0.95mm_HandSolder" V -3570 1950 60  0001 C CNN
+F 3 "" H 3100 4800 60  0001 C CNN
+	1    3100 4800
+	1    0    0    1
+$EndComp
+Wire Wire Line
+	3100 4950 4000 4950
+Connection ~ 3100 4950
+Text HLabel 3100 5250 0    50   Input ~ 10
+12V
 $EndSCHEMATC

Commit message: Update (#46)
Changed lines of the file:
@@
 Comment4 ""
 $EndDescr
-Text Notes 6250 3300 0    160  ~ 0
+Text Notes 6250 3300 0    160  ~ 6
 8 channel high / low side driver
 NoConn ~ 6150 7800
@@
 	1    0    0    -1
 $EndComp
-Text HLabel 4350 7150 2    60   Input ~ 0
+Text HLabel 4350 7150 2    60   Input ~ 6
 5V
 $Comp
@@
 Wire Wire Line
 	6850 4950 6850 5450
-Text HLabel 7700 5150 2    60   Input ~ 0
+Text HLabel 7700 5150 2    60   Input ~ 6
 IGN_1
-Text HLabel 7700 5750 2    60   Input ~ 0
+Text HLabel 7700 5750 2    60   Input ~ 6
 IGN_2
-Text HLabel 7750 6500 2    60   Input ~ 0
+Text HLabel 7750 6500 2    60   Input ~ 6
 IGN_3
-Text HLabel 7750 7100 2    60   Input ~ 0
+Text HLabel 7750 7100 2    60   Input ~ 6
 IGN_4
-Text HLabel 7800 7700 2    60   Input ~ 0
+Text HLabel 7800 7700 2    60   Input ~ 6
 HS1
-Text HLabel 7800 8300 2    60   Input ~ 0
+Text HLabel 7800 8300 2    60   Input ~ 6
 HS2
-Text HLabel 5150 5350 0    60   Input ~ 0
+Text HLabel 5150 5350 0    60   Input ~ 6
 IGN_1_MCU
-Text HLabel 5150 5550 0    60   Input ~ 0
+Text HLabel 5150 5550 0    60   Input ~ 6
 IGN_2_MCU
-Text HLabel 5200 6700 0    60   Input ~ 0
+Text HLabel 5200 6700 0    60   Input ~ 6
 IGN_3_MCU
-Text HLabel 5200 6900 0    60   Input ~ 0
+Text HLabel 5200 6900 0    60   Input ~ 6
 IGN_4_MCU
-Text HLabel 5250 7900 0    60   Input ~ 0
+Text HLabel 5250 7900 0    60   Input ~ 6
 HS1_MCU
-Text HLabel 5250 8100 0    60   Input ~ 0
+Text HLabel 5250 8100 0    60   Input ~ 6
 HS2_MCU
 Wire Wire Line
@@
 	4350 6300 6900 6300
 Connection ~ 4350 6800
-Text Label 3100 4650 0    50   ~ 0
+Text Label 3100 4650 0    50   ~ 6
 5V
 $Comp
