File: hi-lo.sch (KiCad schematic (older format))
At the start: 14 parts, among them U31 MIC4427, U32 MIC4427, U33 MIC4427

Commit message: Updated JP2 removing default bridge. https://github.com/rusefi/hw_microRusEfi/issues/126
Parts:
- JP2: footprint Jumper:SolderJumper-3_P1.3mm_Bridged2Bar12_Pad1.0x1.5mm -> Jumper:SolderJumper-3_P1.3mm_Open_Pad1.0x1.5mm; symbol Jumper:SolderJumper_3_Bridged12 -> Jumper:SolderJumper_3_Open
Changed lines of the file:
@@
 $EndComp
 $Comp
-L Jumper:SolderJumper_3_Bridged12 JP2
+L Jumper:SolderJumper_3_Open JP2
 U 1 1 5DAB9BDF
 P 3550 4700
 F 0 "JP2" H 3550 4950 50  0000 C CNN
 F 1 "High side voltage 5V 12V" H 3550 4850 50  0000 C CNN
-F 2 "Jumper:SolderJumper-3_P1.3mm_Bridged2Bar12_Pad1.0x1.5mm" H 3550 4700 50  0001 C CNN
+F 2 "Jumper:SolderJumper-3_P1.3mm_Open_Pad1.0x1.5mm" H 3550 4700 50  0001 C CNN
 F 3 "~" H 3550 4700 50  0001 C CNN
 	1    3550 4700

Commit message: Added 4X low sides now 4 channels are either low side or analog.
Parts:
- RN5, RN6: Manufacturer (none) -> Yageo; Part # (none) -> YC164-JR-0710KL; VEND (none) -> DIGI; VEND# (none) -> YC164J-10KCT-ND
Changed lines of the file:
@@
 $Descr B 17000 11000
 encoding utf-8
-Sheet 2 7
+Sheet 2 9
 Title "microRusEfi-2L"
 Date "2020-02-12"
@@
 F 3 "~" H 5950 8500 50  0001 C CNN
 F 4 "C29718" H 5950 8500 50  0001 C CNN "LCSC"
+F 5 "Yageo" H 5950 8500 50  0001 C CNN "Manufacturer"
+F 6 "YC164-JR-0710KL" H 5950 8500 50  0001 C CNN "Part #"
+F 7 "DIGI" H 5950 8500 50  0001 C CNN "VEND"
+F 8 "YC164J-10KCT-ND" H 5950 8500 50  0001 C CNN "VEND#"
 	1    5950 8500
 	1    0    0    -1
@@
 F 3 "~" H 5850 5975 50  0001 C CNN
 F 4 "C29718" H 5850 5975 50  0001 C CNN "LCSC"
+F 5 "Yageo" H 5850 5975 50  0001 C CNN "Manufacturer"
+F 6 "YC164-JR-0710KL" H 5850 5975 50  0001 C CNN "Part #"
+F 7 "DIGI" H 5850 5975 50  0001 C CNN "VEND"
+F 8 "YC164J-10KCT-ND" H 5850 5975 50  0001 C CNN "VEND#"
 	1    5850 5975
 	1    0    0    -1
