File: microRusEfi.sch (KiCad schematic (older format))
At the start: 11 parts, among them U3 Molex_48_pin

Commit message: latest updates
Connections:
- net labels removed: UBR
Changed lines of the file:
@@
 Wire Wire Line
 	11275 4425 11700 4425
-Text Label 11275 4725 3    50   ~ 0
-UBR
-Text Label 10975 4825 3    50   ~ 0
-UBR
 $Comp
 L Device:LED D21
@@
 Text Label 5150 1575 3    60   ~ 12
 12V-SWITCH
+Text Label 10975 4825 3    60   ~ 12
+12V-SWITCH
+Text Label 11275 4725 3    60   ~ 12
+12V-SWITCH
 $EndSCHEMATC

Commit message: manual sync with 960
Parts:
- removed D21: LED, LED_SMD:LED_0603_1608Metric_Pad1.05x0.95mm_HandSolder, symbol Device:LED
- removed R28: 1K, Resistor_SMD:R_0603_1608Metric_Pad1.05x0.95mm_HandSolder, symbol Device:R
- added R16: DNP, modules:Logo, symbol Device:R
- D15, D20: Part # (none) -> NSR0530HT
Connections:
- net labels added: AN-TEMP-1, AN-TEMP-2, AN-TEMP-3, AN-TEMP-4, AN-VOLT-4, AN-VOLT-5, AN-VOLT-6, AN-VOLT-7, AN-VOLT-8, AN-VOLT-9
- net labels removed: ACC-PEDAL, BRAKE-PEDAL, CLUTCH-PEDAL, DIGITAL_IN_1, DIGITAL_IN_2, ECT-SENSOR, IAT-SENSOR, MAF-SENSOR, MAP-SENSOR, TPS
Changed lines of the file:
@@
 Text Label 8350 1575 3    60   ~ 12
 FUEL-PUMP
-Text Label 7650 1575 3    60   ~ 12
-TPS
 Text Label 7150 1575 3    60   ~ 12
-ECT-SENSOR
+AN-TEMP-2
 Text Label 8050 1575 3    60   ~ 12
-AN-VOLT-1
+AN-VOLT-3
 Text Label 8250 1575 3    60   ~ 12
 RPM-OUT
@@
 Text Label 5300 1575 3    60   ~ 12
 GND
+Text Label 8900 1575 3    60   ~ 12
+5V2
 Text Label 8150 1575 3    60   ~ 12
-5V2
-Text Label 7550 1575 3    60   ~ 12
-ACC-PEDAL
-Text Label 8900 1575 3    60   ~ 12
-CLUTCH-PEDAL
-Text Label 9000 1575 3    60   ~ 12
-BRAKE-PEDAL
+AN-VOLT-6
 Text Label 9300 1575 3    60   ~ 12
 ALTERNATOR
-Text Label 7050 1575 3    60   ~ 12
-MAF-SENSOR
 Text Label 8450 1575 3    60   ~ 12
 WASTEGATE
 Text Label 6600 1575 3    60   ~ 12
-IAT-SENSOR
+AN-TEMP-1
 Text Label 7250 1575 3    60   ~ 12
-MAP-SENSOR
-Text Label 9800 1575 3    60   ~ 12
+AN-TEMP-3
+Text Label 9900 1575 3    60   ~ 12
 CANH
 Text Label 4850 1575 3    60   ~ 12
 GND
-Text Label 9900 1575 3    60   ~ 12
+Text Label 9800 1575 3    60   ~ 12
 CANL
 Text Label 5900 1575 3    60   ~ 12
@@
 GND
 Text Label 6700 1575 3    60   ~ 12
-AN-VOLT-2
+AN-VOLT-4
 Text Label 6250 1575 3    50   ~ 0
 USB_D-
@@
 Text Label 4725 6325 2    60   ~ 0
 VDD
-Text Label 7450 1575 3    50   ~ 0
+Text Label 7650 1575 3    50   ~ 10
 CAM_SENSOR
-Text Label 3425 3975 2    60   ~ 12
-TPS
 Text Label 3425 3575 2    60   ~ 12
-ECT-SENSOR
+AN-TEMP-2
 Text Label 3425 4175 2    60   ~ 12
-AN-VOLT-1
-Text Label 3425 3875 2    60   ~ 12
-ACC-PEDAL
-Text Label 3425 3775 2    60   ~ 12
-MAF-SENSOR
+AN-VOLT-3
 Text Label 3425 3475 2    60   ~ 12
-IAT-SENSOR
+AN-TEMP-1
 Text Label 3425 3675 2    60   ~ 12
-MAP-SENSOR
+AN-TEMP-3
 Text Label 3425 4275 2    60   ~ 12
-AN-VOLT-2
+AN-VOLT-4
 Text Label 3425 4375 2    60   ~ 12
-AN-VOLT-3
+AN-VOLT-5
 Text Label 6800 1575 3    60   ~ 12
-AN-VOLT-3
+AN-VOLT-5
+Text Label 3425 4475 2    60   ~ 12
+AN-VOLT-6
 Text Label 3425 4775 2    60   ~ 12
-CLUTCH-PEDAL
-Text Label 3425 4675 2    60   ~ 12
-BRAKE-PEDAL
-Text Label 3425 4575 2    50   ~ 0
-DIGITAL_IN_1
-Text Label 3425 4475 2    50   ~ 0
-DIGITAL_IN_2
-Text Label 8600 1575 3    50   ~ 0
-DIGITAL_IN_1
-Text Label 7900 1575 3    50   ~ 0
-DIGITAL_IN_2
+AN-VOLT-9
+Text Label 3425 4675 2    50   ~ 10
+AN-VOLT-8
+Text Label 3425 4575 2    50   ~ 10
+AN-VOLT-7
 $Comp
 L Device:D_Schottky D15
@@
 F 2 "Diode_SMD:D_SOD-323" H 10975 4675 50  0001 C CNN
 F 3 "~" H 10975 4675 50  0001 C CNN
+F 4 "NSR0530HT" H 0   0   50  0001 C CNN "Part #"
 	1    10975 4675
 	0    -1   -1   0
@@
 F 2 "Diode_SMD:D_SOD-323" H 11275 4575 50  0001 C CNN
 F 3 "~" H 11275 4575 50  0001 C CNN
+F 4 "NSR0530HT" H 0   0   50  0001 C CNN "Part #"
 	1    11275 4575
 	0    -1   -1   0
@@
 Wire Wire Line
 	11275 4425 11700 4425
-$Comp
-L Device:LED D21
-U 1 1 5E75E63B
-P 14125 5500
-F 0 "D21" H 14118 5245 50  0000 C CNN
-F 1 "LED" H 14118 5336 50  0000 C CNN
-F 2 "LED_SMD:LED_0603_1608Metric_Pad1.05x0.95mm_HandSolder" H 14125 5500 50  0001 C CNN
-F 3 "~" H 14125 5500 50  0001 C CNN
-	1    14125 5500
-	-1   0    0    1
-$EndComp
-$Comp
-L Device:R R28
-U 1 1 5E75E8AF
-P 14425 5500
-F 0 "R28" V 14218 5500 50  0000 C CNN
-F 1 "1K" V 14309 5500 50  0000 C CNN
-F 2 "Resistor_SMD:R_0603_1608Metric_Pad1.05x0.95mm_HandSolder" V 14355 5500 50  0001 C CNN
-F 3 "~" H 14425 5500 50  0001 C CNN
-	1    14425 5500
-	0    1    1    0
-$EndComp
-Text Label 13975 5500 2    60   ~ 12
-INJECTOR-1
-Text Label 14575 5500 0    60   ~ 12
-5V
 $Comp
 L Device:LED D22
@@
 Text Label 7750 1575 3    60   ~ 12
 MAIN_RELAY
-Text Label 3425 4075 2    50   ~ 0
+Text Label 3425 3975 2    50   ~ 10
 CAM_SENSOR
 Wire Wire Line
@@
 Text Label 11275 4725 3    60   ~ 12
 12V-SWITCH
+$Comp
+L Device:R R16
+U 1 1 5D002597
+P 14750 2275
+F 0 "R16" H 14820 2321 50  0000 L CNN
+F 1 "DNP" H 14820 2230 50  0000 L CNN
+F 2 "modules:Logo" V 14680 2275 50  0001 C CNN
+F 3 "~" H 14750 2275 50  0001 C CNN
+	1    14750 2275
+	1    0    0    -1
+$EndComp
+Text Label 7450 1575 3    60   ~ 12
+AN-VOLT-2
+Text Label 3425 4075 2    60   ~ 12
+AN-VOLT-2
+Text Label 7550 1575 3    60   ~ 12
+AN-VOLT-1
+Text Label 3425 3875 2    60   ~ 12
+AN-VOLT-1
+Text Label 7050 1575 3    60   ~ 12
+AN-TEMP-4
+Text Label 3425 3775 2    60   ~ 12
+AN-TEMP-4
+Text Label 7900 1575 3    50   ~ 10
+AN-VOLT-7
+Text Label 8600 1575 3    50   ~ 10
+AN-VOLT-8
+Text Label 9000 1575 3    60   ~ 12
+AN-VOLT-9
 $EndSCHEMATC

Commit message: Update (#40)
Parts:
- removed D23: LED, LED_SMD:LED_0603_1608Metric_Pad1.05x0.95mm_HandSolder, symbol Device:LED
- removed R30: 1K, Resistor_SMD:R_0603_1608Metric_Pad1.05x0.95mm_HandSolder, symbol Device:R
- added TP6: TP, TestPoint:TestPoint_Pad_D2.0mm, symbol Connector:TestPoint
Connections:
- net labels added: AN-VOLT-10
- wire segments 82 -> 84
Changed lines of the file:
@@
 	6700 3875 5600 3875
-Wire Wire Line
-	6700 3975 5600 3975
 Wire Wire Line
 	6700 4175 5600 4175
@@
 VDD
 Wire Wire Line
-	9000 5475 7950 5475
+	9000 5475 8100 5475
 $Sheet
 S 8300 7125 1050 1200
@@
 Text Label 4725 6325 2    60   ~ 0
 VDD
-Text Label 7650 1575 3    50   ~ 10
+Text Label 7350 1575 3    50   ~ 10
 CAM_SENSOR
 Text Label 3425 3575 2    60   ~ 12
@@
 	0    1    1    0
 $EndComp
-$Comp
-L Device:LED D23
-U 1 1 5E766AEA
-P 14125 6400
-F 0 "D23" H 14118 6145 50  0000 C CNN
-F 1 "LED" H 14118 6236 50  0000 C CNN
-F 2 "LED_SMD:LED_0603_1608Metric_Pad1.05x0.95mm_HandSolder" H 14125 6400 50  0001 C CNN
-F 3 "~" H 14125 6400 50  0001 C CNN
-	1    14125 6400
-	-1   0    0    1
-$EndComp
-$Comp
-L Device:R R30
-U 1 1 5E766AF4
-P 14425 6400
-F 0 "R30" V 14218 6400 50  0000 C CNN
-F 1 "1K" V 14309 6400 50  0000 C CNN
-F 2 "Resistor_SMD:R_0603_1608Metric_Pad1.05x0.95mm_HandSolder" V 14355 6400 50  0001 C CNN
-F 3 "~" H 14425 6400 50  0001 C CNN
-	1    14425 6400
-	0    1    1    0
-$EndComp
 Text Label 14575 5950 0    60   ~ 12
-5V
-Text Label 13975 6400 2    60   ~ 12
-CRANK
-Text Label 14575 6400 0    60   ~ 12
 5V
 $Comp
@@
 Text Label 7750 1575 3    60   ~ 12
 MAIN_RELAY
-Text Label 3425 3975 2    50   ~ 10
+Text Label 4050 4925 2    50   ~ 10
 CAM_SENSOR
 Wire Wire Line
@@
 F32 "ADC_13_MCU" I R 5600 4675 50
 F33 "ADC_14_MCU" I R 5600 4775 50
+F34 "CAM" I L 4050 4925 50
+F35 "CAM_MCU" I R 5600 4925 50
 $EndSheet
 Wire Wire Line
@@
 F5 "PA1" I L 6700 3575 60
 F6 "PA3" I L 6700 3775 60
-F7 "PA5" I L 6700 3975 60
+F7 "PA5" I L 6700 4925 60
 F8 "PA7" I L 6700 4175 60
 F9 "PC5" I L 6700 4575 60
@@
 F21 "PD13" I L 6700 7825 60
 F22 "PD15" I L 6700 8025 60
-F23 "PC0" I L 6700 5625 60
+F23 "PC0" I L 6700 3975 60
 F24 "PC2" I L 6700 4275 60
 F25 "PA0" I L 6700 3475 60
@@
 Text Label 9000 1575 3    60   ~ 12
 AN-VOLT-9
+$Comp
+L Connector:TestPoint TP6
+U 1 1 5CFB23FC
+P 8100 5475
+F 0 "TP6" H 8158 5593 50  0001 L CNN
+F 1 "TP" H 8158 5502 50  0000 L CNN
+F 2 "TestPoint:TestPoint_Pad_D2.0mm" H 8300 5475 50  0001 C CNN
+F 3 "~" H 8300 5475 50  0001 C CNN
+	1    8100 5475
+	1    0    0    -1
+$EndComp
+Connection ~ 8100 5475
+Wire Wire Line
+	8100 5475 7950 5475
+Wire Wire Line
+	6700 4925 5600 4925
+Text Label 3425 3975 2    50   ~ 10
+AN-VOLT-10
+Text Label 7650 1575 3    50   ~ 10
+AN-VOLT-10
+Wire Wire Line
+	5600 3975 6700 3975
 $EndSCHEMATC

Commit message: Latest (#43)
Parts:
- removed TP6: TP, TestPoint:TestPoint_Pad_D2.0mm, symbol Connector:TestPoint
- added TP4: TP, TestPoint:TestPoint_Pad_D2.0mm, symbol Connector:TestPoint
- D22: footprint LED_SMD:LED_0603_1608Metric_Pad1.05x0.95mm_HandSolder -> LED_SMD:LED_0402_1005Metric
- R29: footprint Resistor_SMD:R_0603_1608Metric_Pad1.05x0.95mm_HandSolder -> Resistor_SMD:R_0402_1005Metric
Connections:
- net labels added: GP_OUT_1, GP_OUT_2, GP_OUT_3, GP_OUT_4, GP_OUT_5, GP_OUT_6, PE1, PE2, PE3, PE4
- net labels removed: ALTERNATOR, FUEL-PUMP, HS_1, HS_2, RPM-OUT, RUNNING_LED, WASTEGATE
- wire segments 84 -> 88
Other:
- note added: "GP OUT 5 AND 6 ARE HIGH SIDE DRIVEN"
- note removed: "ALL PINS ARE SHOWN AS DEFAULT PINOUT\nANY UNUSED PINS CAN BE USED FOR OTHER PURPOSES"
- moved on the sheet: D22, R29
Changed lines of the file:
@@
 $Descr User 17000 12598
 encoding utf-8
-Sheet 1 6
+Sheet 1 7
 Title "microRusEfi"
 Date "2019-01-31"
@@
 Text Label 10750 6675 0    60   ~ 0
 VDD
-Wire Wire Line
-	9000 5475 8100 5475
 $Sheet
 S 8300 7125 1050 1200
@@
 5V
 Text Label 11450 5925 0    60   ~ 12
-ALTERNATOR
+GP_OUT_4
 Wire Wire Line
 	6700 5175 5600 5175
@@
 $EndComp
 Text Label 8350 1575 3    60   ~ 12
-FUEL-PUMP
+GP_OUT_2
 Text Label 7150 1575 3    60   ~ 12
 AN-TEMP-2
@@
 AN-VOLT-3
 Text Label 8250 1575 3    60   ~ 12
-RPM-OUT
+GP_OUT_3
 Text Label 9550 1575 3    60   ~ 12
 CRNK+
@@
 AN-VOLT-6
 Text Label 9300 1575 3    60   ~ 12
-ALTERNATOR
+GP_OUT_4
 Text Label 8450 1575 3    60   ~ 12
-WASTEGATE
+GP_OUT_1
 Text Label 6600 1575 3    60   ~ 12
 AN-TEMP-1
@@
 Text Label 6700 1575 3    60   ~ 12
 AN-VOLT-4
-Text Label 6250 1575 3    50   ~ 0
+Text Label 6250 1575 3    50   ~ 10
 USB_D-
-Text Label 6400 1575 3    50   ~ 0
+Text Label 6400 1575 3    50   ~ 10
 USB_D+
 $Sheet
@@
 Text Label 4475 6025 2    50   ~ 0
 E-THROTTLE-
-Text Label 5050 1575 3    50   ~ 0
+Text Label 5050 1575 3    50   ~ 10
 E-THROTTLE+
-Text Label 5500 1575 3    50   ~ 0
+Text Label 5500 1575 3    50   ~ 10
 E-THROTTLE-
-Text Label 5400 1575 3    50   ~ 0
+Text Label 5400 1575 3    50   ~ 10
 VVT-1
-Text Label 4950 1575 3    50   ~ 0
+Text Label 4950 1575 3    50   ~ 10
 VVT-2
 Text Label 11700 4525 0    50   ~ 0
@@
 	11275 4425 11700 4425
 $Comp
-L Device:LED D22
-U 1 1 5E7651E5
-P 14125 5950
-F 0 "D22" H 14118 5695 50  0000 C CNN
-F 1 "LED" H 14118 5786 50  0000 C CNN
-F 2 "LED_SMD:LED_0603_1608Metric_Pad1.05x0.95mm_HandSolder" H 14125 5950 50  0001 C CNN
-F 3 "~" H 14125 5950 50  0001 C CNN
-	1    14125 5950
-	-1   0    0    1
-$EndComp
-$Comp
-L Device:R R29
-U 1 1 5E7651EF
-P 14425 5950
-F 0 "R29" V 14218 5950 50  0000 C CNN
-F 1 "1K" V 14309 5950 50  0000 C CNN
-F 2 "Resistor_SMD:R_0603_1608Metric_Pad1.05x0.95mm_HandSolder" V 14355 5950 50  0001 C CNN
-F 3 "~" H 14425 5950 50  0001 C CNN
-	1    14425 5950
-	0    1    1    0
-$EndComp
-Text Label 14575 5950 0    60   ~ 12
-5V
-$Comp
 L power:GND #PWR0162
 U 1 1 5E774BC6
@@
 	5800 6500 5800 6600
 Connection ~ 5800 6600
-Text Label 7950 6175 0    50   ~ 0
-RUNNING_LED
-Text Label 13975 5950 2    50   ~ 0
-RUNNING_LED
 Wire Wire Line
 	10750 4225 11425 4225
@@
 	10750 3925 11425 3925
 Text Label 11450 5725 0    60   ~ 12
-FUEL-PUMP
+GP_OUT_2
 Text Label 11450 5625 0    60   ~ 12
-WASTEGATE
+GP_OUT_1
 Text Label 11450 5825 0    60   ~ 12
-RPM-OUT
+GP_OUT_3
 Text Notes 11575 3725 0    50   ~ 0
 LOW SIDE OUTPUTS\n
@@
 Text Label 8300 5875 2    60   ~ 12
 GND
-Text Label 6000 1575 3    50   ~ 0
-HS_1
+Text Label 6000 1575 3    50   ~ 10
+GP_OUT_6
 Text Label 7750 1575 3    60   ~ 12
 MAIN_RELAY
@@
 Wire Wire Line
 	10750 5925 11450 5925
-Text Label 6100 1575 3    50   ~ 0
-HS_2
-Text Label 9725 7325 0    50   ~ 0
-HS_1
-Text Label 9725 7225 0    50   ~ 0
-HS_2
+Text Label 6100 1575 3    50   ~ 10
+GP_OUT_5
+Text Label 9725 7325 0    50   ~ 10
+GP_OUT_6
+Text Label 9725 7225 0    50   ~ 10
+GP_OUT_5
 Wire Notes Line
 	11300 3550 11300 4800
@@
 Wire Wire Line
 	5600 4775 6700 4775
-Text Notes 6325 2750 0    50   ~ 0
-ALL PINS ARE SHOWN AS DEFAULT PINOUT\nANY UNUSED PINS CAN BE USED FOR OTHER PURPOSES
+Text Notes 6675 2750 0    50   ~ 0
+GP OUT 5 AND 6 ARE HIGH SIDE DRIVEN
 NoConn ~ 10750 3425
 NoConn ~ 10750 3525
@@
 F13 "PE11" I R 7950 4125 60
 F14 "PE13" I R 7950 3925 60
-F15 "PE15" I R 7950 5900 60
+F15 "PE15" I L 6700 7625 60
 F16 "PB11" I R 7950 8925 60
-F17 "PB13" I L 6700 8325 60
-F18 "PB15" I L 6700 8925 60
+F17 "PB13" I L 6700 7550 60
+F18 "PB15" I L 6700 7475 60
 F19 "PD9" I R 7950 8525 60
 F20 "PD11" I R 7950 9525 60
 F21 "PD13" I L 6700 7825 60
 F22 "PD15" I L 6700 8025 60
-F23 "PC0" I L 6700 3975 60
+F23 "PC0" I L 6700 3875 60
 F24 "PC2" I L 6700 4275 60
 F25 "PA0" I L 6700 3475 60
 F26 "PA2" I L 6700 3675 60
-F27 "PA4" I L 6700 3875 60
+F27 "PA4" I L 6700 3975 60
 F28 "PA6" I L 6700 4075 60
 F29 "PC4" I L 6700 4475 60
@@
 F35 "PB10" I L 6700 8425 60
 F36 "PB12" I R 7950 4925 60
-F37 "PB14" I R 7950 8325 60
+F37 "PB14" I L 6700 7400 60
 F38 "PD8" I L 6700 9025 60
 F39 "PD10" I R 7950 8825 60
@@
 Text Label 9000 1575 3    60   ~ 12
 AN-VOLT-9
-$Comp
-L Connector:TestPoint TP6
-U 1 1 5CFB23FC
-P 8100 5475
-F 0 "TP6" H 8158 5593 50  0001 L CNN
-F 1 "TP" H 8158 5502 50  0000 L CNN
-F 2 "TestPoint:TestPoint_Pad_D2.0mm" H 8300 5475 50  0001 C CNN
-F 3 "~" H 8300 5475 50  0001 C CNN
-	1    8100 5475
-	1    0    0    -1
-$EndComp
-Connection ~ 8100 5475
-Wire Wire Line
-	8100 5475 7950 5475
-Wire Wire Line
-	6700 4925 5600 4925
 Text Label 3425 3975 2    50   ~ 10
 AN-VOLT-10
@@
 Wire Wire Line
 	5600 3975 6700 3975
+Text Label 7950 6175 0    50   ~ 10
+PE1
+Text Label 6700 8125 2    50   ~ 10
+PE2
+Text Label 6700 8625 2    50   ~ 10
+PE3
+Text Label 6700 8525 2    50   ~ 10
+PE4
+Text Label 13975 6025 2    50   ~ 10
+PE1
+Text Label 14575 6025 0    60   ~ 12
+5V
+$Comp
+L Device:R R29
+U 1 1 5E7651EF
+P 14425 6025
+F 0 "R29" V 14218 6025 50  0000 C CNN
+F 1 "1K" V 14309 6025 50  0000 C CNN
+F 2 "Resistor_SMD:R_0402_1005Metric" V 14355 6025 50  0001 C CNN
+F 3 "~" H 14425 6025 50  0001 C CNN
+	1    14425 6025
+	0    1    1    0
+$EndComp
+$Comp
+L Device:LED D22
+U 1 1 5E7651E5
+P 14125 6025
+F 0 "D22" H 14118 5770 50  0000 C CNN
+F 1 "LED" H 14118 5861 50  0000 C CNN
+F 2 "LED_SMD:LED_0402_1005Metric" H 14125 6025 50  0001 C CNN
+F 3 "~" H 14125 6025 50  0001 C CNN
+	1    14125 6025
+	-1   0    0    1
+$EndComp
+$Sheet
+S 5500 7325 725  375
+U 5D2F23B4
+F0 "FlashMemory" 50
+F1 "FlashMemory.sch" 50
+F2 "SI" I R 6225 7475 50
+F3 "SCK" I R 6225 7550 50
+F4 "CS" I R 6225 7625 50
+F5 "SO" I R 6225 7400 50
+F6 "VDD" I L 5500 7625 50
+$EndSheet
+Wire Wire Line
+	6700 7475 6225 7475
+Wire Wire Line
+	6700 7400 6225 7400
+Wire Wire Line
+	6700 7550 6225 7550
+Text Label 5500 7625 2    50   ~ 10
+VDD
+Wire Wire Line
+	6225 7625 6700 7625
+Wire Wire Line
+	7950 5475 8125 5475
+$Comp
+L Connector:TestPoint TP4
+U 1 1 5D358BCF
+P 8125 5475
+F 0 "TP4" H 8183 5593 50  0001 L CNN
+F 1 "TP" H 8183 5502 50  0000 L CNN
+F 2 "TestPoint:TestPoint_Pad_D2.0mm" H 8325 5475 50  0001 C CNN
+F 3 "~" H 8325 5475 50  0001 C CNN
+	1    8125 5475
+	1    0    0    -1
+$EndComp
+Connection ~ 8125 5475
+Wire Wire Line
+	8125 5475 9000 5475
+Wire Wire Line
+	5600 4925 6700 4925
 $EndSCHEMATC

Commit message: Latest
Parts:
- added TP3: TP, TestPoint:TestPoint_Pad_D2.0mm, symbol Connector:TestPoint
- D22: footprint LED_SMD:LED_0402_1005Metric -> LED_SMD:LED_0603_1608Metric_Pad1.05x0.95mm_HandSolder
- R29: footprint Resistor_SMD:R_0402_1005Metric -> Resistor_SMD:R_0603_1608Metric_Pad1.05x0.95mm_HandSolder
Connections:
- wire segments 88 -> 89
Changed lines of the file:
@@
 F 0 "R29" V 14218 6025 50  0000 C CNN
 F 1 "1K" V 14309 6025 50  0000 C CNN
-F 2 "Resistor_SMD:R_0402_1005Metric" V 14355 6025 50  0001 C CNN
+F 2 "Resistor_SMD:R_0603_1608Metric_Pad1.05x0.95mm_HandSolder" V 14355 6025 50  0001 C CNN
 F 3 "~" H 14425 6025 50  0001 C CNN
 	1    14425 6025
@@
 F 0 "D22" H 14118 5770 50  0000 C CNN
 F 1 "LED" H 14118 5861 50  0000 C CNN
-F 2 "LED_SMD:LED_0402_1005Metric" H 14125 6025 50  0001 C CNN
+F 2 "LED_SMD:LED_0603_1608Metric_Pad1.05x0.95mm_HandSolder" H 14125 6025 50  0001 C CNN
 F 3 "~" H 14125 6025 50  0001 C CNN
 	1    14125 6025
@@
 	8125 5475 9000 5475
 Wire Wire Line
-	5600 4925 6700 4925
+	5600 4925 6150 4925
+$Comp
+L Connector:TestPoint TP3
+U 1 1 5D08B37F
+P 6150 4925
+F 0 "TP3" H 6208 5043 50  0001 L CNN
+F 1 "TP" H 6208 4952 50  0000 L CNN
+F 2 "TestPoint:TestPoint_Pad_D2.0mm" H 6350 4925 50  0001 C CNN
+F 3 "~" H 6350 4925 50  0001 C CNN
+	1    6150 4925
+	1    0    0    -1
+$EndComp
+Connection ~ 6150 4925
+Wire Wire Line
+	6150 4925 6700 4925
 $EndSCHEMATC
