File: microRusEfi.sch (KiCad schematic (older format))
At the start: 10 parts, among them U3 Molex_48_pin

Commit message: Update (#46)
Parts:
- added D21, D23, D27: LED, LED_SMD:LED_0402_1005Metric, symbol Device:LED
- added R36, R49, R51: 1K, Resistor_SMD:R_0402_1005Metric, symbol Device:R
- D22: footprint LED_SMD:LED_0603_1608Metric_Pad1.05x0.95mm_HandSolder -> LED_SMD:LED_0402_1005Metric
- R29: footprint Resistor_SMD:R_0603_1608Metric_Pad1.05x0.95mm_HandSolder -> Resistor_SMD:R_0402_1005Metric
Connections:
- wire segments 89 -> 96
- no-connect marks 8 -> 4
Changed lines of the file:
@@
 F4 "IN_11" I L 9000 4525 60
 F5 "IN_12" I L 9000 4625 60
-F6 "IGN_IN_1" I L 9000 3375 60
-F7 "IGN_IN_2" I L 9000 3475 60
-F8 "IGN_IN_3" I L 9000 3575 60
-F9 "IGN_IN_4" I L 9000 3675 60
+F6 "IGN_IN_1" I L 9000 3400 60
+F7 "IGN_IN_2" I L 9000 3500 60
+F8 "IGN_IN_3" I L 9000 3600 60
+F9 "IGN_IN_4" I L 9000 3700 60
 F10 "IGN_OUT_1" I R 10750 3425 60
 F11 "IGN_OUT_2" I R 10750 3525 60
@@
 	1    0    0    -1
 $EndComp
-Text Label 10750 6675 0    60   ~ 0
+Text Label 10750 6675 0    60   ~ 6
 VDD
 $Sheet
@@
 Wire Wire Line
 	6700 5175 5600 5175
-Text Label 6200 5175 2    60   ~ 0
+Text Label 6200 5175 2    60   ~ 6
 Vref
 Text Label 9725 7625 0    60   ~ 12
@@
 F13 "12V" I L 4725 6225 50
 $EndSheet
-Text Label 4475 5925 2    50   ~ 0
+Text Label 4475 5925 2    50   ~ 6
 E-THROTTLE+
-Text Label 4475 6025 2    50   ~ 0
+Text Label 4475 6025 2    50   ~ 6
 E-THROTTLE-
 Text Label 5050 1575 3    50   ~ 10
@@
 Text Label 4950 1575 3    50   ~ 10
 VVT-2
-Text Label 11700 4525 0    50   ~ 0
+Text Label 11700 4525 0    50   ~ 6
 VVT-1
-Text Label 11700 4425 0    50   ~ 0
+Text Label 11700 4425 0    50   ~ 6
 VVT-2
 Text Label 4725 6425 2    60   ~ 12
 GND
-Text Label 4725 6325 2    60   ~ 0
+Text Label 4725 6325 2    60   ~ 6
 VDD
 Text Label 7350 1575 3    50   ~ 10
@@
 Text Label 11450 5825 0    60   ~ 12
 GP_OUT_3
-Text Notes 11575 3725 0    50   ~ 0
+Text Notes 11575 3725 0    50   ~ 6
 LOW SIDE OUTPUTS\n
-Text Notes 12100 4475 0    50   ~ 0
+Text Notes 12100 4475 0    50   ~ 6
 4.5A
-Text Notes 12050 5700 0    50   ~ 0
+Text Notes 12050 5700 0    50   ~ 6
 0.6A
 Wire Wire Line
@@
 Wire Wire Line
 	10750 5825 11450 5825
-Text Notes 12100 4050 0    50   ~ 0
+Text Notes 12100 4050 0    50   ~ 6
 2.2A
 Wire Wire Line
@@
 Wire Notes Line
 	9625 8100 9625 7000
-Text Notes 10625 7925 2    50   ~ 0
+Text Notes 10625 7925 2    50   ~ 6
 HIGH-SIDE OUTPUTS \n
-Text Notes 2550 3300 0    50   ~ 0
+Text Notes 2550 3300 0    50   ~ 6
 ANALOG INPUTS.\nADC 1-4 HAS BIAS RESISTORS \nFOR TEMP SENSORS\n\nCAN ALSO BE USED \nAS DIGITAL INPUTS
 Wire Notes Line
@@
 Wire Notes Line
 	11300 5225 12475 5225
-Text Notes 11375 5450 0    50   ~ 0
+Text Notes 11375 5450 0    50   ~ 6
 CAN BE USED AS LOW-SIDE \nOR HIGH-SIDE
 Wire Notes Line
@@
 Wire Wire Line
 	5600 4775 6700 4775
-Text Notes 6675 2750 0    50   ~ 0
+Text Notes 6675 2750 0    50   ~ 6
 GP OUT 5 AND 6 ARE HIGH SIDE DRIVEN
 NoConn ~ 10750 3425
@@
 NoConn ~ 10750 3625
 NoConn ~ 10750 3725
-NoConn ~ 9000 3375
-NoConn ~ 9000 3475
-NoConn ~ 9000 3575
-NoConn ~ 9000 3675
 Wire Wire Line
 	5675 5925 6700 5925
@@
 Wire Wire Line
 	5675 6400 6700 6400
-Text Notes 3950 5750 0    50   ~ 0
+Text Notes 3950 5750 0    50   ~ 6
 6A H-BRIDGE
 Wire Wire Line
@@
 Wire Wire Line
 	3425 4775 4050 4775
-Text Label 6700 5400 2    50   ~ 0
+Text Label 6700 5400 2    50   ~ 6
 USB_D-
-Text Label 6700 5475 2    50   ~ 0
+Text Label 6700 5475 2    50   ~ 6
 USB_D+
-Text Label 5975 5075 0    50   ~ 0
+Text Label 5975 5075 0    50   ~ 6
 Vbat_MCU
-Text Label 5625 4475 0    50   ~ 0
+Text Label 5625 4475 0    50   ~ 6
 AnOut11
-Text Label 5625 4575 0    50   ~ 0
+Text Label 5625 4575 0    50   ~ 6
 AnOut12
-Text Label 5625 4675 0    50   ~ 0
+Text Label 5625 4675 0    50   ~ 6
 AnOut13
-Text Label 5625 4775 0    50   ~ 0
+Text Label 5625 4775 0    50   ~ 6
 AnOut14
 $Sheet
@@
 F 0 "R29" V 14218 6025 50  0000 C CNN
 F 1 "1K" V 14309 6025 50  0000 C CNN
-F 2 "Resistor_SMD:R_0603_1608Metric_Pad1.05x0.95mm_HandSolder" V 14355 6025 50  0001 C CNN
+F 2 "Resistor_SMD:R_0402_1005Metric" V 14355 6025 50  0001 C CNN
 F 3 "~" H 14425 6025 50  0001 C CNN
 	1    14425 6025
@@
 F 0 "D22" H 14118 5770 50  0000 C CNN
 F 1 "LED" H 14118 5861 50  0000 C CNN
-F 2 "LED_SMD:LED_0603_1608Metric_Pad1.05x0.95mm_HandSolder" H 14125 6025 50  0001 C CNN
+F 2 "LED_SMD:LED_0402_1005Metric" H 14125 6025 50  0001 C CNN
 F 3 "~" H 14125 6025 50  0001 C CNN
 	1    14125 6025
@@
 Wire Wire Line
 	6150 4925 6700 4925
+$Comp
+L power:GND #PWR0183
+U 1 1 5D16B569
+P 8500 3500
+F 0 "#PWR0183" H 8500 3250 50  0001 C CNN
+F 1 "GND" H 8505 3327 50  0000 C CNN
+F 2 "" H 8500 3500 50  0001 C CNN
+F 3 "" H 8500 3500 50  0001 C CNN
+	1    8500 3500
+	0    1    1    0
+$EndComp
+Wire Wire Line
+	8500 3400 9000 3400
+Wire Wire Line
+	8500 3400 8500 3500
+Wire Wire Line
+	9000 3500 8500 3500
+Wire Wire Line
+	9000 3600 8500 3600
+Connection ~ 8500 3500
+Wire Wire Line
+	9000 3700 8500 3700
+Wire Wire Line
+	8500 3500 8500 3600
+Wire Wire Line
+	8500 3700 8500 3600
+Connection ~ 8500 3600
+Text Label 14550 6425 0    60   ~ 12
+5V
+$Comp
+L Device:R R36
+U 1 1 5D1B59DE
+P 14400 6425
+F 0 "R36" V 14193 6425 50  0000 C CNN
+F 1 "1K" V 14284 6425 50  0000 C CNN
+F 2 "Resistor_SMD:R_0402_1005Metric" V 14330 6425 50  0001 C CNN
+F 3 "~" H 14400 6425 50  0001 C CNN
+	1    14400 6425
+	0    1    1    0
+$EndComp
+$Comp
+L Device:LED D21
+U 1 1 5D1B59E8
+P 14100 6425
+F 0 "D21" H 14093 6170 50  0000 C CNN
+F 1 "LED" H 14093 6261 50  0000 C CNN
+F 2 "LED_SMD:LED_0402_1005Metric" H 14100 6425 50  0001 C CNN
+F 3 "~" H 14100 6425 50  0001 C CNN
+	1    14100 6425
+	-1   0    0    1
+$EndComp
+Text Label 14550 6900 0    60   ~ 12
+5V
+$Comp
+L Device:R R49
+U 1 1 5D1BAEA8
+P 14400 6900
+F 0 "R49" V 14193 6900 50  0000 C CNN
+F 1 "1K" V 14284 6900 50  0000 C CNN
+F 2 "Resistor_SMD:R_0402_1005Metric" V 14330 6900 50  0001 C CNN
+F 3 "~" H 14400 6900 50  0001 C CNN
+	1    14400 6900
+	0    1    1    0
+$EndComp
+$Comp
+L Device:LED D23
+U 1 1 5D1BAEB2
+P 14100 6900
+F 0 "D23" H 14093 6645 50  0000 C CNN
+F 1 "LED" H 14093 6736 50  0000 C CNN
+F 2 "LED_SMD:LED_0402_1005Metric" H 14100 6900 50  0001 C CNN
+F 3 "~" H 14100 6900 50  0001 C CNN
+	1    14100 6900
+	-1   0    0    1
+$EndComp
+Text Label 14550 7375 0    60   ~ 12
+5V
+$Comp
+L Device:R R51
+U 1 1 5D1C01BF
+P 14400 7375
+F 0 "R51" V 14193 7375 50  0000 C CNN
+F 1 "1K" V 14284 7375 50  0000 C CNN
+F 2 "Resistor_SMD:R_0402_1005Metric" V 14330 7375 50  0001 C CNN
+F 3 "~" H 14400 7375 50  0001 C CNN
+	1    14400 7375
+	0    1    1    0
+$EndComp
+$Comp
+L Device:LED D27
+U 1 1 5D1C01C9
+P 14100 7375
+F 0 "D27" H 14093 7120 50  0000 C CNN
+F 1 "LED" H 14093 7211 50  0000 C CNN
+F 2 "LED_SMD:LED_0402_1005Metric" H 14100 7375 50  0001 C CNN
+F 3 "~" H 14100 7375 50  0001 C CNN
+	1    14100 7375
+	-1   0    0    1
+$EndComp
+Text Label 13950 6425 2    50   ~ 10
+PE2
+Text Label 13950 6900 2    50   ~ 10
+PE3
+Text Label 13950 7375 2    50   ~ 10
+PE4
 $EndSCHEMATC

Commit message: Small fix (#52)
Parts:
- removed R29, R36, R49, R51: 1K, Resistor_SMD:R_0402_1005Metric, symbol Device:R
- added RN1: R_Pack04, Resistor_SMD:R_Array_Convex_4x0603, symbol Device:R_Pack04
Connections:
- wire segments 96 -> 99
Other:
- moved on the sheet: D21, D23, D27
Changed lines of the file:
@@
 	1    0    0    -1
 $EndComp
-Text Label 10750 6675 0    60   ~ 6
+Text Label 10750 6675 0    60   ~ 12
 VDD
 $Sheet
@@
 Wire Wire Line
 	6700 5175 5600 5175
-Text Label 6200 5175 2    60   ~ 6
+Text Label 6200 5175 2    60   ~ 12
 Vref
 Text Label 9725 7625 0    60   ~ 12
@@
 F13 "12V" I L 4725 6225 50
 $EndSheet
-Text Label 4475 5925 2    50   ~ 6
+Text Label 4475 5925 2    50   ~ 10
 E-THROTTLE+
-Text Label 4475 6025 2    50   ~ 6
+Text Label 4475 6025 2    50   ~ 10
 E-THROTTLE-
 Text Label 5050 1575 3    50   ~ 10
@@
 Text Label 4950 1575 3    50   ~ 10
 VVT-2
-Text Label 11700 4525 0    50   ~ 6
+Text Label 11700 4525 0    50   ~ 10
 VVT-1
-Text Label 11700 4425 0    50   ~ 6
+Text Label 11700 4425 0    50   ~ 10
 VVT-2
 Text Label 4725 6425 2    60   ~ 12
 GND
-Text Label 4725 6325 2    60   ~ 6
+Text Label 4725 6325 2    60   ~ 12
 VDD
 Text Label 7350 1575 3    50   ~ 10
@@
 Text Label 11450 5825 0    60   ~ 12
 GP_OUT_3
-Text Notes 11575 3725 0    50   ~ 6
+Text Notes 11575 3725 0    50   ~ 10
 LOW SIDE OUTPUTS\n
-Text Notes 12100 4475 0    50   ~ 6
+Text Notes 12100 4475 0    50   ~ 10
 4.5A
-Text Notes 12050 5700 0    50   ~ 6
+Text Notes 12050 5700 0    50   ~ 10
 0.6A
 Wire Wire Line
@@
 Wire Wire Line
 	10750 5825 11450 5825
-Text Notes 12100 4050 0    50   ~ 6
+Text Notes 12100 4050 0    50   ~ 10
 2.2A
 Wire Wire Line
@@
 Wire Notes Line
 	9625 8100 9625 7000
-Text Notes 10625 7925 2    50   ~ 6
+Text Notes 10625 7925 2    50   ~ 10
 HIGH-SIDE OUTPUTS \n
-Text Notes 2550 3300 0    50   ~ 6
+Text Notes 2550 3300 0    50   ~ 10
 ANALOG INPUTS.\nADC 1-4 HAS BIAS RESISTORS \nFOR TEMP SENSORS\n\nCAN ALSO BE USED \nAS DIGITAL INPUTS
 Wire Notes Line
@@
 Wire Notes Line
 	11300 5225 12475 5225
-Text Notes 11375 5450 0    50   ~ 6
+Text Notes 11375 5450 0    50   ~ 10
 CAN BE USED AS LOW-SIDE \nOR HIGH-SIDE
 Wire Notes Line
@@
 Wire Wire Line
 	5600 4775 6700 4775
-Text Notes 6675 2750 0    50   ~ 6
+Text Notes 6675 2750 0    50   ~ 10
 GP OUT 5 AND 6 ARE HIGH SIDE DRIVEN
 NoConn ~ 10750 3425
@@
 Wire Wire Line
 	5675 6400 6700 6400
-Text Notes 3950 5750 0    50   ~ 6
+Text Notes 3950 5750 0    50   ~ 10
 6A H-BRIDGE
 Wire Wire Line
@@
 Wire Wire Line
 	3425 4775 4050 4775
-Text Label 6700 5400 2    50   ~ 6
+Text Label 6700 5400 2    50   ~ 10
 USB_D-
-Text Label 6700 5475 2    50   ~ 6
+Text Label 6700 5475 2    50   ~ 10
 USB_D+
-Text Label 5975 5075 0    50   ~ 6
+Text Label 5975 5075 0    50   ~ 10
 Vbat_MCU
-Text Label 5625 4475 0    50   ~ 6
+Text Label 5625 4475 0    50   ~ 10
 AnOut11
-Text Label 5625 4575 0    50   ~ 6
+Text Label 5625 4575 0    50   ~ 10
 AnOut12
-Text Label 5625 4675 0    50   ~ 6
+Text Label 5625 4675 0    50   ~ 10
 AnOut13
-Text Label 5625 4775 0    50   ~ 6
+Text Label 5625 4775 0    50   ~ 10
 AnOut14
 $Sheet
@@
 Text Label 13975 6025 2    50   ~ 10
 PE1
-Text Label 14575 6025 0    60   ~ 12
+Text Label 14675 6175 0    60   ~ 12
 5V
-$Comp
-L Device:R R29
-U 1 1 5E7651EF
-P 14425 6025
-F 0 "R29" V 14218 6025 50  0000 C CNN
-F 1 "1K" V 14309 6025 50  0000 C CNN
-F 2 "Resistor_SMD:R_0402_1005Metric" V 14355 6025 50  0001 C CNN
-F 3 "~" H 14425 6025 50  0001 C CNN
-	1    14425 6025
-	0    1    1    0
-$EndComp
 $Comp
 L Device:LED D22
@@
 	8500 3700 8500 3600
 Connection ~ 8500 3600
-Text Label 14550 6425 0    60   ~ 12
-5V
-$Comp
-L Device:R R36
-U 1 1 5D1B59DE
-P 14400 6425
-F 0 "R36" V 14193 6425 50  0000 C CNN
-F 1 "1K" V 14284 6425 50  0000 C CNN
-F 2 "Resistor_SMD:R_0402_1005Metric" V 14330 6425 50  0001 C CNN
-F 3 "~" H 14400 6425 50  0001 C CNN
-	1    14400 6425
-	0    1    1    0
-$EndComp
 $Comp
 L Device:LED D21
 U 1 1 5D1B59E8
-P 14100 6425
-F 0 "D21" H 14093 6170 50  0000 C CNN
-F 1 "LED" H 14093 6261 50  0000 C CNN
-F 2 "LED_SMD:LED_0402_1005Metric" H 14100 6425 50  0001 C CNN
-F 3 "~" H 14100 6425 50  0001 C CNN
-	1    14100 6425
+P 14125 6125
+F 0 "D21" H 14118 5870 50  0000 C CNN
+F 1 "LED" H 14118 5961 50  0000 C CNN
+F 2 "LED_SMD:LED_0402_1005Metric" H 14125 6125 50  0001 C CNN
+F 3 "~" H 14125 6125 50  0001 C CNN
+	1    14125 6125
 	-1   0    0    1
-$EndComp
-Text Label 14550 6900 0    60   ~ 12
-5V
-$Comp
-L Device:R R49
-U 1 1 5D1BAEA8
-P 14400 6900
-F 0 "R49" V 14193 6900 50  0000 C CNN
-F 1 "1K" V 14284 6900 50  0000 C CNN
-F 2 "Resistor_SMD:R_0402_1005Metric" V 14330 6900 50  0001 C CNN
-F 3 "~" H 14400 6900 50  0001 C CNN
-	1    14400 6900
-	0    1    1    0
 $EndComp
 $Comp
 L Device:LED D23
 U 1 1 5D1BAEB2
-P 14100 6900
-F 0 "D23" H 14093 6645 50  0000 C CNN
-F 1 "LED" H 14093 6736 50  0000 C CNN
-F 2 "LED_SMD:LED_0402_1005Metric" H 14100 6900 50  0001 C CNN
-F 3 "~" H 14100 6900 50  0001 C CNN
-	1    14100 6900
+P 14125 6225
+F 0 "D23" H 14118 5970 50  0000 C CNN
+F 1 "LED" H 14118 6061 50  0000 C CNN
+F 2 "LED_SMD:LED_0402_1005Metric" H 14125 6225 50  0001 C CNN
+F 3 "~" H 14125 6225 50  0001 C CNN
+	1    14125 6225
 	-1   0    0    1
-$EndComp
-Text Label 14550 7375 0    60   ~ 12
-5V
-$Comp
-L Device:R R51
-U 1 1 5D1C01BF
-P 14400 7375
-F 0 "R51" V 14193 7375 50  0000 C CNN
-F 1 "1K" V 14284 7375 50  0000 C CNN
-F 2 "Resistor_SMD:R_0402_1005Metric" V 14330 7375 50  0001 C CNN
-F 3 "~" H 14400 7375 50  0001 C CNN
-	1    14400 7375
-	0    1    1    0
 $EndComp
 $Comp
 L Device:LED D27
 U 1 1 5D1C01C9
-P 14100 7375
-F 0 "D27" H 14093 7120 50  0000 C CNN
-F 1 "LED" H 14093 7211 50  0000 C CNN
-F 2 "LED_SMD:LED_0402_1005Metric" H 14100 7375 50  0001 C CNN
-F 3 "~" H 14100 7375 50  0001 C CNN
-	1    14100 7375
+P 14125 6325
+F 0 "D27" H 14118 6070 50  0000 C CNN
+F 1 "LED" H 14118 6161 50  0000 C CNN
+F 2 "LED_SMD:LED_0402_1005Metric" H 14125 6325 50  0001 C CNN
+F 3 "~" H 14125 6325 50  0001 C CNN
+	1    14125 6325
 	-1   0    0    1
 $EndComp
-Text Label 13950 6425 2    50   ~ 10
+Text Label 13975 6125 2    50   ~ 10
 PE2
-Text Label 13950 6900 2    50   ~ 10
+Text Label 13975 6225 2    50   ~ 10
 PE3
-Text Label 13950 7375 2    50   ~ 10
+Text Label 13975 6325 2    50   ~ 10
 PE4
+$Comp
+L Device:R_Pack04 RN1
+U 1 1 5CF9A0A2
+P 14475 6125
+F 0 "RN1" V 14058 6125 50  0000 C CNN
+F 1 "R_Pack04" V 14149 6125 50  0000 C CNN
+F 2 "Resistor_SMD:R_Array_Convex_4x0603" V 14750 6125 50  0001 C CNN
+F 3 "~" H 14475 6125 50  0001 C CNN
+	1    14475 6125
+	0    1    -1   0
+$EndComp
+Wire Wire Line
+	14675 6325 14675 6225
+Connection ~ 14675 6225
+Wire Wire Line
+	14675 6225 14675 6125
+Connection ~ 14675 6125
+Wire Wire Line
+	14675 6125 14675 6025
 $EndSCHEMATC

Commit message: Ready To Go! (#53)
Parts:
- U3: Manufacturer (none) -> MOLEX; Part # (none) -> 500762-0481
- renumbered R16 to LOGO1
Connections:
- wire segments 99 -> 101
Other:
- moved on the sheet: LOGO1
Changed lines of the file:
@@
 F 2 "rusefi_lib:Molex_48" H 7750 2125 60  0001 C CNN
 F 3 "" H 7750 2125 60  0001 C CNN
+F 4 "MOLEX" H 0   0   50  0001 C CNN "Manufacturer"
+F 5 "500762-0481" H 0   0   50  0001 C CNN "Part #"
 	1    7750 2125
 	0    -1   -1   0
@@
 F13 "PE11" I R 7950 4125 60
 F14 "PE13" I R 7950 3925 60
-F15 "PE15" I L 6700 7625 60
-F16 "PB11" I R 7950 8925 60
-F17 "PB13" I L 6700 7550 60
-F18 "PB15" I L 6700 7475 60
+F15 "PE15" I L 6700 7700 60
+F16 "PB11" I L 6700 7800 60
+F17 "PB13" I L 6700 7600 60
+F18 "PB15" I L 6700 7500 60
 F19 "PD9" I R 7950 8525 60
 F20 "PD11" I R 7950 9525 60
-F21 "PD13" I L 6700 7825 60
-F22 "PD15" I L 6700 8025 60
+F21 "PD13" I R 7950 8100 60
+F22 "PD15" I L 6700 8150 60
 F23 "PC0" I L 6700 3875 60
 F24 "PC2" I L 6700 4275 60
@@
 F33 "PE12" I R 7950 4025 60
 F34 "PE14" I R 7950 3825 60
-F35 "PB10" I L 6700 8425 60
+F35 "PB10" I L 6700 7900 60
 F36 "PB12" I R 7950 4925 60
 F37 "PB14" I L 6700 7400 60
 F38 "PD8" I L 6700 9025 60
 F39 "PD10" I R 7950 8825 60
-F40 "PD12" I L 6700 7725 60
-F41 "PD14" I L 6700 7925 60
+F40 "PD12" I R 7950 8000 60
+F41 "PD14" I R 7950 8200 60
 F42 "5V" I R 7950 6775 60
 F43 "PE6" I R 7950 9225 60
 F44 "PE4" I L 6700 8525 60
-F45 "PE2" I L 6700 8125 60
-F46 "PE0" I L 6700 8225 60
+F45 "PE2" I L 6700 8250 60
+F46 "PE0" I L 6700 8350 60
 F47 "PB8" I L 6700 8725 60
 F48 "PB6" I R 7950 4825 60
@@
 12V-SWITCH
 $Comp
-L Device:R R16
+L Device:R LOGO1
 U 1 1 5D002597
-P 14750 2275
-F 0 "R16" H 14820 2321 50  0000 L CNN
-F 1 "DNP" H 14820 2230 50  0000 L CNN
-F 2 "modules:Logo" V 14680 2275 50  0001 C CNN
-F 3 "~" H 14750 2275 50  0001 C CNN
-	1    14750 2275
+P 15800 825
+F 0 "LOGO1" H 15870 871 50  0000 L CNN
+F 1 "DNP" H 15870 780 50  0000 L CNN
+F 2 "modules:Logo" V 15730 825 50  0001 C CNN
+F 3 "~" H 15800 825 50  0001 C CNN
+	1    15800 825
 	1    0    0    -1
 $EndComp
@@
 Text Label 7950 6175 0    50   ~ 10
 PE1
-Text Label 6700 8125 2    50   ~ 10
+Text Label 6700 8250 2    50   ~ 10
 PE2
 Text Label 6700 8625 2    50   ~ 10
@@
 $EndComp
 $Sheet
-S 5500 7325 725  375
+S 5500 7325 700  625
 U 5D2F23B4
 F0 "FlashMemory" 50
 F1 "FlashMemory.sch" 50
-F2 "SI" I R 6225 7475 50
-F3 "SCK" I R 6225 7550 50
-F4 "CS" I R 6225 7625 50
-F5 "SO" I R 6225 7400 50
+F2 "SI" I R 6200 7500 50
+F3 "SCK" I R 6200 7600 50
+F4 "CS" I R 6200 7700 50
+F5 "SO" I R 6200 7400 50
 F6 "VDD" I L 5500 7625 50
+F7 "HOLD" I R 6200 7800 50
+F8 "WP" I R 6200 7900 50
 $EndSheet
-Wire Wire Line
-	6700 7475 6225 7475
-Wire Wire Line
-	6700 7400 6225 7400
-Wire Wire Line
-	6700 7550 6225 7550
 Text Label 5500 7625 2    50   ~ 10
 VDD
-Wire Wire Line
-	6225 7625 6700 7625
 Wire Wire Line
 	7950 5475 8125 5475
@@
 Wire Wire Line
 	14675 6125 14675 6025
+Wire Wire Line
+	6200 7400 6700 7400
+Wire Wire Line
+	6700 7500 6200 7500
+Wire Wire Line
+	6200 7600 6700 7600
+Wire Wire Line
+	6700 7700 6200 7700
+Wire Wire Line
+	6700 7900 6200 7900
+Wire Wire Line
+	6200 7800 6700 7800
 $EndSCHEMATC
