File: adc.sch (KiCad schematic (older format))
At the start: 54 parts, among them U35 MCP6004, U36 MCP6004, U37 10K, U38 10K, U39 10nF, U40 10nF, U41 1K, U42 1K, U43 1.5K, U44 1.5K, U46 MCP6004, U48 10K, U50 10nF, U52 1K, U54 1.5K

Commit message: fix adc
Parts:
- removed D14: BAS70-04, Package_TO_SOT_SMD:SOT-23, symbol Diode:BAS40-04
- removed U37, U38, U48: 10K, Resistor_SMD:R_Array_Convex_4x0603, symbol BOSCH_154_PIN:RESISTOR_ARRAY
- removed U39, U40, U50: 10nF, Resistor_SMD:R_Array_Convex_4x0603, symbol BOSCH_154_PIN:RESISTOR_ARRAY
- removed U41, U42, U52: 1K, Resistor_SMD:R_Array_Convex_4x0603, symbol BOSCH_154_PIN:RESISTOR_ARRAY
- removed U43, U44, U54: 1.5K, Resistor_SMD:R_Array_Convex_4x0603, symbol BOSCH_154_PIN:RESISTOR_ARRAY
- added U37, U38, U48: 10k, symbol Device:R_Pack04
- added U39, U40, U50: 10nF, symbol Device:R_Pack04
- added U41, U42, U52: 1k, symbol Device:R_Pack04
- added U43, U44, U54: 1.5k, symbol Device:R_Pack04
Connections:
- wire segments 262 -> 258
Other:
- moved on the sheet: D11, D12, D13, R11, R131, R139, R14, R141, R142, R143, R15, R23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

Commit message: Latest schematics
Parts:
- removed R15, R26, R33, R36: DNP, Resistor_SMD:R_0603_1608Metric_Pad1.05x0.95mm_HandSolder, symbol Device:R
- added C40: 0.1uF, Capacitor_SMD:C_0603_1608Metric_Pad1.05x0.95mm_HandSolder, symbol Device:C
- added D18, D24, D25, D26: BAS70-04, Package_TO_SOT_SMD:SOT-23, symbol Diode:BAS40-04
- added R52, R54, R56, R58: 500K, Resistor_SMD:R_0603_1608Metric_Pad1.05x0.95mm_HandSolder, symbol Device:R
- added U10: 1.5k, Resistor_SMD:R_Array_Convex_4x0603, symbol Device:R_Pack04
- added U6: 10k, Resistor_SMD:R_Array_Convex_4x0603, symbol Device:R_Pack04
- added U7: 10nF, Resistor_SMD:R_Array_Convex_4x0603, symbol Device:R_Pack04
- added U8: MCP6004, Package_SO:TSSOP-14_4.4x5mm_P0.65mm, symbol Amplifier_Operational:MCP6004
- added U9: 1k, Resistor_SMD:R_Array_Convex_4x0603, symbol Device:R_Pack04
- U37, U38, U39, U40, U41, U42, U43, U44, U48, U50, U52, U54: footprint (none) -> Resistor_SMD:R_Array_Convex_4x0603
Connections:
- net 5V: now also C40.1, D18.2, D24.2, D25.2, D26.2, U8.4 (V+)
- net GND: now also C40.2, D18.1, D24.1, D25.1, D26.1, R52.2, R54.2, R56.2, R58.2, U10.5 (R4.2), U10.6 (R3.2), U10.7 (R2.2), U10.8 (R1.2), U7.5 (R4.2), U7.6 (R3.2), U7.7 (R2.2), U7.8 (R1.2), U8.11 (V-)
- net UBR renamed 12V-SWITCH
- net UBR_MCU renamed Vbat_MCU
- new net: D24.3, U6.6 (R3.2), U7.2 (R2.1), U8.12 (+)
- new net: U8.13 (-), U8.14, U9.3 (R3.1)
- new net: D18.3, U6.5 (R4.2), U7.1 (R1.1), U8.10 (+)
- new net: U8.8, U8.9 (-), U9.4 (R4.1)
- new net: D26.3, U6.8 (R1.2), U7.4 (R4.1), U8.5 (+)
- new net: U8.6 (-), U8.7, U9.1 (R1.1)
- new net: U8.1, U8.2 (-), U9.2 (R2.1)
- new net: D25.3, U6.7 (R2.2), U7.3 (R3.1), U8.3 (+)
- new net ADC_11: R58.1, U6.1 (R1.1)
- new net ADC_11_MCU: U10.1 (R1.1), U9.8 (R1.2)
- new net ADC_12: R56.1, U6.2 (R2.1)
- new net ADC_12_MCU: U10.2 (R2.1), U9.7 (R2.2)
- new net ADC_13: R54.1, U6.3 (R3.1)
- new net ADC_13_MCU: U10.3 (R3.1), U9.6 (R3.2)
- new net ADC_14: R52.1, U6.4 (R4.1)
- new net ADC_14_MCU: U10.4 (R4.1), U9.5 (R4.2)

Commit message: manual sync with 960
Parts:
- removed D13: BAS70-04, Package_TO_SOT_SMD:SOT-23, symbol Diode:BAS40-04
- C40, C79, C80, C82: value 0.1uF -> 10nF; MFG,MFG# AVX,08055C104KAT2A -> (none); VEND1,VEND1# DIGI,478-1395-1-ND -> (none)
- R11, R139, R14, R142, R23, R25, R27, R40: MFG,MFG# DNP,DNP -> (none); VEND1,VEND1# DNP,DNP -> (none); VEND2,VEND2# , -> (none)
- R131, R141, R143, R24, R31, R32, R34, R35, R37, R38, R39, R41, R52, R54, R56, R58: MFG,MFG# ECG,ERA6AEB4993V -> (none); VEND1,VEND1# DIGI,P499KDACT-ND -> (none); VEND2,VEND2# , -> (none)
- U10, U43, U44, U54: Part # (none) -> 667-EXB-V8V152JV
- U35, U36, U46, U8: MFG,MFG# ADA4096-4ARUZ-R7 -> (none); Part # ADA4096-4ARUZ-R7 -> 579-MCP6004T-I/ST; VEND# 584-ADA4096-4ARUZ-R7 -> 579-MCP6004T-I/ST; VEND1,VEND1# DIGI,MCP6004-E/SL-ND -> (none); VEND2,VEND2# , -> (none)
- U35, U36, U46, U8: MFG,MFG# ADA4096-4ARUZ-R7 -> (none); Part # ADA4096-4ARUZ-R7 -> 579-MCP6004T-I/ST; VEND# 584-ADA4096-4ARUZ-R7 -> 579-MCP6004T-I/ST
- U37, U38, U48, U6: Part # (none) -> 603-YC324-JK-0710KL; VEND# (none) -> 603-YC324-JK-0710KL
- U39, U40, U50, U7: Part # (none) -> 80-CA064X103K2RAUTO
- U41, U42, U52, U9: Part # (none) -> 667-EXB-V8V102JV; VEND# (none) -> 667-EXB-V8V102JV
Connections:
- net at U50.4 (R4.1): now also U46.5 (+), U48.8 (R1.2)

Commit message: Update (#40)
Parts:
- added C41: 1nF, Capacitor_SMD:C_0603_1608Metric_Pad1.05x0.95mm_HandSolder, symbol Device:C
- added R26: DNP, Resistor_SMD:R_0603_1608Metric_Pad1.05x0.95mm_HandSolder, symbol Device:R
- added R28: 2.15K, Resistor_SMD:R_0603_1608Metric_Pad1.05x0.95mm_HandSolder, symbol Device:R
- added R30: 33K, Resistor_SMD:R_0603_1608Metric_Pad1.05x0.95mm_HandSolder, symbol Device:R
Connections:
- net 5V: now also R26.2, R28.2
- net ADC_6: now also R26.1
- net GND: now also C41.2
- new net CAM: R28.1, R30.2
- new net CAM_MCU: C41.1, R30.1
Changed lines of the file:
@@
 Wire Wire Line
 	12600 3350 13050 3350
+Text Label 2525 4250 0    60   ~ 0
+5V
+$Comp
+L Device:R R26
+U 1 1 5CF4D843
+P 2525 4400
+F 0 "R26" V 2605 4400 40  0000 C CNN
+F 1 "DNP" V 2532 4401 40  0000 C CNN
+F 2 "Resistor_SMD:R_0603_1608Metric_Pad1.05x0.95mm_HandSolder" V 4330 4100 60  0001 C CNN
+F 3 "" H 7850 4125 60  0001 C CNN
+	1    2525 4400
+	-1   0    0    1
+$EndComp
+Wire Wire Line
+	2525 4850 2525 4550
+$Comp
+L Device:R R28
+U 1 1 5CFF5765
+P 10500 7075
+F 0 "R28" V 10580 7075 40  0000 C CNN
+F 1 "2.15K" V 10507 7076 40  0000 C CNN
+F 2 "Resistor_SMD:R_0603_1608Metric_Pad1.05x0.95mm_HandSolder" V 12305 6275 60  0001 C CNN
+F 3 "" H 15825 6300 60  0001 C CNN
+	1    10500 7075
+	-1   0    0    1
+$EndComp
+$Comp
+L Device:R R30
+U 1 1 5CFF714D
+P 10775 7225
+F 0 "R30" V 10855 7225 40  0000 C CNN
+F 1 "33K" V 10782 7226 40  0000 C CNN
+F 2 "Resistor_SMD:R_0603_1608Metric_Pad1.05x0.95mm_HandSolder" V 12580 6425 60  0001 C CNN
+F 3 "" H 16100 6450 60  0001 C CNN
+	1    10775 7225
+	0    1    -1   0
+$EndComp
+$Comp
+L Device:C C41
+U 1 1 5CFF8DB5
+P 10975 7375
+F 0 "C41" H 10975 7475 40  0000 L CNN
+F 1 "1nF" H 10981 7290 40  0000 L CNN
+F 2 "Capacitor_SMD:C_0603_1608Metric_Pad1.05x0.95mm_HandSolder" V 7605 1725 60  0001 C CNN
+F 3 "" H 10975 7375 60  0001 C CNN
+	1    10975 7375
+	1    0    0    -1
+$EndComp
+Text HLabel 10050 7225 0    50   Input ~ 0
+CAM
+Text HLabel 11650 7225 2    50   Input ~ 0
+CAM_MCU
+Wire Wire Line
+	10050 7225 10500 7225
+Connection ~ 10500 7225
+Wire Wire Line
+	10500 7225 10625 7225
+Wire Wire Line
+	10925 7225 10975 7225
+Connection ~ 10975 7225
+Wire Wire Line
+	10975 7225 11650 7225
+$Comp
+L power:GND #PWR0139
+U 1 1 5D03EC5A
+P 10975 7525
+F 0 "#PWR0139" H 10975 7525 30  0001 C CNN
+F 1 "GND" H 10975 7455 30  0001 C CNN
+F 2 "" H 10975 7525 60  0000 C CNN
+F 3 "" H 10975 7525 60  0000 C CNN
+	1    10975 7525
+	1    0    0    -1
+$EndComp
+Text Label 10500 6925 0    60   ~ 0
+5V
 $EndSCHEMATC

Commit message: Latest (#43)
Parts:
- added D13: BAS70-04, Package_TO_SOT_SMD:SOT-23, symbol Diode:BAS40-04
Connections:
- net 5V: now also D13.2
- net CAM: now also D13.3
- net GND: now also D13.1
Changed lines of the file:
@@
 $Descr B 17000 11000
 encoding utf-8
-Sheet 5 6
+Sheet 5 7
 Title "frankenso"
 Date "2018-02-24"
@@
 Text HLabel 11650 7225 2    50   Input ~ 0
 CAM_MCU
-Wire Wire Line
-	10050 7225 10500 7225
 Connection ~ 10500 7225
 Wire Wire Line
@@
 Text Label 10500 6925 0    60   ~ 0
 5V
+$Comp
+L Diode:BAS40-04 D13
+U 1 1 5D22D9AA
+P 10400 7225
+F 0 "D13" V 10438 7305 40  0000 L CNN
+F 1 "BAS70-04" V 9850 7125 40  0000 L CNN
+F 2 "Package_TO_SOT_SMD:SOT-23" H 10400 7225 60  0001 C CNN
+F 3 "" H 10400 7225 60  0000 C CNN
+F 4 "BAS70-04" H 6150 2175 50  0001 C CNN "Part #"
+	1    10400 7225
+	0    -1   -1   0
+$EndComp
+Wire Wire Line
+	10050 7225 10500 7225
+$Comp
+L power:GND #PWR0140
+U 1 1 5D251281
+P 10300 7525
+F 0 "#PWR0140" H 10300 7525 30  0001 C CNN
+F 1 "GND" H 10300 7455 30  0001 C CNN
+F 2 "" H 10300 7525 60  0000 C CNN
+F 3 "" H 10300 7525 60  0000 C CNN
+	1    10300 7525
+	1    0    0    -1
+$EndComp
+Text Label 10300 6925 0    60   ~ 0
+5V
 $EndSCHEMATC

Commit message: Latest
Parts:
- removed R142: 1K, Resistor_SMD:R_0603_1608Metric_Pad1.05x0.95mm_HandSolder, symbol Device:R
- removed R143: 500K, Resistor_SMD:R_0603_1608Metric_Pad1.05x0.95mm_HandSolder, symbol Device:R
- removed R26: DNP, Resistor_SMD:R_0603_1608Metric_Pad1.05x0.95mm_HandSolder, symbol Device:R
- R14, R23, R25, R27: value DNP -> 2.7K
Connections:
- net 5V: now also U48.1 (R1.1)
- net CAM: no longer D13.3
- net CAM_MCU: now also D13.3
Other:
- moved on the sheet: D13
Changed lines of the file:
@@
 ADC_10_MCU
-Wire Notes Line
-	9350 2600 9375 2600
 Wire Notes Line
 	9800 3325 9825 3325
@@
 Wire Notes Line
 	9775 3525 9800 3525
-Text Label 9150 2350 0    60   ~ 0
-5V
-$Comp
-L Device:R R142
-U 1 1 5D0E7EF2
-P 9150 2500
-F 0 "R142" V 9230 2500 40  0000 C CNN
-F 1 "1K" V 9157 2501 40  0000 C CNN
-F 2 "Resistor_SMD:R_0603_1608Metric_Pad1.05x0.95mm_HandSolder" V 10955 2200 60  0001 C CNN
-F 3 "" H 14475 2225 60  0001 C CNN
-	1    9150 2500
-	-1   0    0    1
-$EndComp
-$Comp
-L power:GND #PWR0183
-U 1 1 5D0E7EFC
-P 9350 2350
-F 0 "#PWR0183" H 9350 2350 30  0001 C CNN
-F 1 "GND" H 9350 2280 30  0001 C CNN
-F 2 "" H 9350 2350 60  0000 C CNN
-F 3 "" H 9350 2350 60  0000 C CNN
-	1    9350 2350
-	-1   0    0    1
-$EndComp
-$Comp
-L Device:R R143
-U 1 1 5D0E7F09
-P 9350 2500
-F 0 "R143" V 9430 2500 40  0000 C CNN
-F 1 "500K" V 9357 2501 40  0000 C CNN
-F 2 "Resistor_SMD:R_0603_1608Metric_Pad1.05x0.95mm_HandSolder" V 11155 1700 60  0001 C CNN
-F 3 "" H 14675 1725 60  0001 C CNN
-	1    9350 2500
-	-1   0    0    1
-$EndComp
+Text Label 9350 3400 0    60   ~ 0
+5V
 Wire Notes Line
 	9375 3525 9400 3525
@@
 P 2500 1450
 F 0 "R14" V 2580 1450 40  0000 C CNN
-F 1 "DNP" V 2507 1451 40  0000 C CNN
+F 1 "2.7K" V 2507 1451 40  0000 C CNN
 F 2 "Resistor_SMD:R_0603_1608Metric_Pad1.05x0.95mm_HandSolder" V 4305 1150 60  0001 C CNN
 F 3 "" H 7825 1175 60  0001 C CNN
@@
 P 2675 1450
 F 0 "R23" V 2755 1450 40  0000 C CNN
-F 1 "DNP" V 2682 1451 40  0000 C CNN
+F 1 "2.7K" V 2682 1451 40  0000 C CNN
 F 2 "Resistor_SMD:R_0603_1608Metric_Pad1.05x0.95mm_HandSolder" V 4480 1150 60  0001 C CNN
 F 3 "" H 8000 1175 60  0001 C CNN
@@
 P 2850 1450
 F 0 "R25" V 2930 1450 40  0000 C CNN
-F 1 "DNP" V 2857 1451 40  0000 C CNN
+F 1 "2.7K" V 2857 1451 40  0000 C CNN
 F 2 "Resistor_SMD:R_0603_1608Metric_Pad1.05x0.95mm_HandSolder" V 4655 1150 60  0001 C CNN
 F 3 "" H 8175 1175 60  0001 C CNN
@@
 P 3025 1450
 F 0 "R27" V 3105 1450 40  0000 C CNN
-F 1 "DNP" V 3032 1451 40  0000 C CNN
+F 1 "2.7K" V 3032 1451 40  0000 C CNN
 F 2 "Resistor_SMD:R_0603_1608Metric_Pad1.05x0.95mm_HandSolder" V 4830 1150 60  0001 C CNN
 F 3 "" H 8350 1175 60  0001 C CNN
@@
 	11100 3350 12600 3350
 Wire Wire Line
-	9350 2650 9350 3400
-Wire Wire Line
 	9350 3400 10650 3400
 Wire Wire Line
@@
 	9750 3500 10650 3500
 Connection ~ 9750 2850
-Wire Wire Line
-	9150 2650 9350 2650
-Connection ~ 9350 2650
 $Comp
 L Device:C C40
@@
 Wire Wire Line
 	12600 3350 13050 3350
-Text Label 2525 4250 0    60   ~ 0
-5V
-$Comp
-L Device:R R26
-U 1 1 5CF4D843
-P 2525 4400
-F 0 "R26" V 2605 4400 40  0000 C CNN
-F 1 "DNP" V 2532 4401 40  0000 C CNN
-F 2 "Resistor_SMD:R_0603_1608Metric_Pad1.05x0.95mm_HandSolder" V 4330 4100 60  0001 C CNN
-F 3 "" H 7850 4125 60  0001 C CNN
-	1    2525 4400
-	-1   0    0    1
-$EndComp
-Wire Wire Line
-	2525 4850 2525 4550
 $Comp
 L Device:R R28
@@
 Connection ~ 10975 7225
 Wire Wire Line
-	10975 7225 11650 7225
+	10975 7225 11500 7225
 $Comp
 L power:GND #PWR0139
@@
 L Diode:BAS40-04 D13
 U 1 1 5D22D9AA
-P 10400 7225
-F 0 "D13" V 10438 7305 40  0000 L CNN
-F 1 "BAS70-04" V 9850 7125 40  0000 L CNN
-F 2 "Package_TO_SOT_SMD:SOT-23" H 10400 7225 60  0001 C CNN
-F 3 "" H 10400 7225 60  0000 C CNN
-F 4 "BAS70-04" H 6150 2175 50  0001 C CNN "Part #"
-	1    10400 7225
+P 11400 7225
+F 0 "D13" V 11438 7305 40  0000 L CNN
+F 1 "BAS70-04" V 10850 7125 40  0000 L CNN
+F 2 "Package_TO_SOT_SMD:SOT-23" H 11400 7225 60  0001 C CNN
+F 3 "" H 11400 7225 60  0000 C CNN
+F 4 "BAS70-04" H 7150 2175 50  0001 C CNN "Part #"
+	1    11400 7225
 	0    -1   -1   0
 $EndComp
@@
 L power:GND #PWR0140
 U 1 1 5D251281
-P 10300 7525
-F 0 "#PWR0140" H 10300 7525 30  0001 C CNN
-F 1 "GND" H 10300 7455 30  0001 C CNN
-F 2 "" H 10300 7525 60  0000 C CNN
-F 3 "" H 10300 7525 60  0000 C CNN
-	1    10300 7525
-	1    0    0    -1
-$EndComp
-Text Label 10300 6925 0    60   ~ 0
-5V
+P 11300 7525
+F 0 "#PWR0140" H 11300 7525 30  0001 C CNN
+F 1 "GND" H 11300 7455 30  0001 C CNN
+F 2 "" H 11300 7525 60  0000 C CNN
+F 3 "" H 11300 7525 60  0000 C CNN
+	1    11300 7525
+	1    0    0    -1
+$EndComp
+Text Label 11300 6925 0    60   ~ 0
+5V
+Connection ~ 11500 7225
+Wire Wire Line
+	11500 7225 11650 7225
 $EndSCHEMATC
