File: zMRETestFixture.kicad_pcb (KiCad board)
At the start: 2 copper layers, 80.6 x 93.7 mm, 40 parts, among them J12 Conn_01x01, J13 Conn_01x01, J3 Conn_01x01, J4 Conn_02x05_Counter_Clockwise, J5 Conn_01x01, U3 molex_48pin_MRE

Commit message: draft
Parts:
- removed the D28 at (64.4, 74.4)
- removed RN1: 1k, Resistor_SMD:R_Array_Convex_4x0603
- added D10: 1N4148WS, rusefi_lib:SM0805_jumper, F.Cu at (139.0, 32.5)
- added D11: BLU, rusefi_lib:SM0805_jumper, F.Cu at (170.4, 49.5)
- added D12: 1N4148WS, rusefi_lib:SM0805_jumper, F.Cu at (128.9, 46.4)
- added D13: BLU, rusefi_lib:SM0805_jumper, F.Cu at (178.7, 41.2)
- added D14: 1N4148WS, rusefi_lib:SM0805_jumper, F.Cu at (139.0, 35.2)
- added D16: 1N4148WS, rusefi_lib:SM0805_jumper, F.Cu at (145.3, 29.7)
- added D17: BLU, rusefi_lib:SM0805_jumper, F.Cu at (182.4, 35.7)
- added D18: 1N4148WS, rusefi_lib:SM0805_jumper, F.Cu at (135.3, 43.7)
- added D19: BLU, rusefi_lib:SM0805_jumper, F.Cu at (166.0, 52.2)
- added D2: 1N4148WS, rusefi_lib:SM0805_jumper, F.Cu at (145.3, 38.0)
- added D23: BLU, rusefi_lib:SM0805_jumper, F.Cu at (166.0, 49.2)
- added D24: 1N4148WS, rusefi_lib:SM0805_jumper, F.Cu at (128.9, 49.2)
- added D25: BLU, rusefi_lib:SM0805_jumper, F.Cu at (182.4, 32.7)
- added D26: 1N4148WS, rusefi_lib:SM0805_jumper, F.Cu at (151.6, 27.0)
- added D30: RED, rusefi_lib:SM0805_jumper, F.Cu at (128.9, 54.7)
- added D31: 1N4148WS, rusefi_lib:SM0805_jumper, F.Cu at (151.6, 32.5)
- added D36: RED, rusefi_lib:SM0805_jumper, F.Cu at (135.3, 51.9)
- added D37: 1N4148WS, rusefi_lib:SM0805_jumper, F.Cu at (151.6, 35.2)
- added D38: RED, rusefi_lib:SM0805_jumper, F.Cu at (128.9, 57.4)
- added D39: 1N4148WS, rusefi_lib:SM0805_jumper, F.Cu at (145.3, 40.7)
- added D40: RED, rusefi_lib:SM0805_jumper, F.Cu at (145.3, 32.5)
- added D41: 1N4148WS, rusefi_lib:SM0805_jumper, F.Cu at (151.6, 38.0)
- added D42: RED, rusefi_lib:SM0805_jumper, F.Cu at (135.3, 54.7)
- added D43: 1N4148WS, rusefi_lib:SM0805_jumper, F.Cu at (158.0, 32.5)
- added D8: 1N4148WS, rusefi_lib:SM0805_jumper, F.Cu at (139.0, 29.7)
- added J5: Conn_01x01, Connector_Pin:Pin_D0.7mm_L6.5mm_W1.8mm_FlatFork, F.Cu at (170.1, 52.7)
- added J6: Conn_01x01, Connector_Pin:Pin_D0.7mm_L6.5mm_W1.8mm_FlatFork, F.Cu at (182.8, 39.0)
- added R10: 1k, rusefi_lib:SM0805_jumper, F.Cu at (154.3, 43.5)
- added R11: 1k, rusefi_lib:SM0805_jumper, F.Cu at (158.0, 38.0)
- added R12: 1k, rusefi_lib:SM0805_jumper, F.Cu at (141.6, 54.5)
- added R13: 1k, rusefi_lib:SM0805_jumper, F.Cu at (164.3, 32.5)
- added R14: 1k, rusefi_lib:SM0805_jumper, F.Cu at (147.9, 49.0)
- added R15: 5k, rusefi_lib:SM0805_jumper, F.Cu at (187.3, 76.8)
- added R16: 1k, rusefi_lib:SM0805_jumper, F.Cu at (184.8, 74.9)
- added R17: 5k, rusefi_lib:SM0805_jumper, F.Cu at (181.0, 76.8)
- added R18: 1k, rusefi_lib:SM0805_jumper, F.Cu at (178.4, 74.9)
- added R19: 5k, rusefi_lib:SM0805_jumper, F.Cu at (174.6, 76.8)
- added R2: 5k, rusefi_lib:SM0805_jumper, F.Cu at (141.6, 49.0)
- added R20: 1k, rusefi_lib:SM0805_jumper, F.Cu at (172.1, 74.9)
- added R21: 5k, rusefi_lib:SM0805_jumper, F.Cu at (168.3, 76.8)
- added R22: 1k, rusefi_lib:SM0805_jumper, F.Cu at (165.7, 74.9)
- added R23: 5k, rusefi_lib:SM0805_jumper, F.Cu at (161.9, 76.8)
- added R24: 1k, rusefi_lib:SM0805_jumper, F.Cu at (158.8, 74.9)
- added R25: 5k, rusefi_lib:SM0805_jumper, F.Cu at (152.4, 81.9)
- added R26: 1k, rusefi_lib:SM0805_jumper, F.Cu at (152.4, 85.1)
- added R27: 5k, rusefi_lib:SM0805_jumper, F.Cu at (146.7, 76.8)
- added R28: 1k, rusefi_lib:SM0805_jumper, F.Cu at (144.1, 74.9)
- added R3: 5k, rusefi_lib:SM0805_jumper, F.Cu at (164.3, 27.0)
- added R30: 1k, rusefi_lib:SM0805_jumper, F.Cu at (154.3, 51.7)
- added R31: 5k, rusefi_lib:SM0805_jumper, F.Cu at (170.6, 35.2)
- added R32: 1k, rusefi_lib:SM0805_jumper, F.Cu at (135.3, 57.4)
- added R33: 5k, rusefi_lib:SM0805_jumper, F.Cu at (147.9, 43.5)
- added R34: 1k, rusefi_lib:SM0805_jumper, F.Cu at (151.6, 29.7)
- added R36: 5k, rusefi_lib:SM0805_jumper, F.Cu at (128.9, 51.9)
- added R37: 1k, rusefi_lib:SM0805_jumper, F.Cu at (139.0, 40.7)
- added R38: 5k, rusefi_lib:SM0805_jumper, F.Cu at (145.3, 35.2)
- added R39: 1k, rusefi_lib:SM0805_jumper, F.Cu at (152.4, 74.9)
- added R4: 5k, rusefi_lib:SM0805_jumper, F.Cu at (147.9, 46.2)
- added R40: 5k, rusefi_lib:SM0805_jumper, F.Cu at (152.4, 78.1)
- added R41: 1k, rusefi_lib:SM0805_jumper, F.Cu at (135.3, 74.9)
- added R42: 5k, rusefi_lib:SM0805_jumper, F.Cu at (137.8, 76.2)
- added R43: 1k, rusefi_lib:SM0805_jumper, F.Cu at (160.6, 51.7)
- added R44: 5k, rusefi_lib:SM0805_jumper, F.Cu at (166.9, 46.2)
- added R45: 1k, rusefi_lib:SM0805_jumper, F.Cu at (173.2, 43.5)
- added R46: 5k, rusefi_lib:SM0805_jumper, F.Cu at (154.3, 54.5)
- added R47: 1k, rusefi_lib:SM0805_jumper, F.Cu at (130.8, 76.2)
- added R48: 5k, rusefi_lib:SM0805_jumper, F.Cu at (128.3, 74.9)
- added R5: 1k, rusefi_lib:SM0805_jumper, F.Cu at (164.3, 29.7)
- added R50: 5k, rusefi_lib:SM0805_jumper, F.Cu at (177.0, 32.5)
- added R52: 5k, rusefi_lib:SM0805_jumper, F.Cu at (183.3, 27.0)
- added R53: 5k, rusefi_lib:SM0805_jumper, F.Cu at (183.3, 29.7)
- added R54: 5k, rusefi_lib:SM0805_jumper, F.Cu at (170.6, 40.7)
- added R6: 1k, rusefi_lib:SM0805_jumper, F.Cu at (141.6, 51.7)
- added R7: 1k, rusefi_lib:SM0805_jumper, F.Cu at (158.0, 35.2)
- added R8: 1k, rusefi_lib:SM0805_jumper, F.Cu at (147.9, 57.2)
- added R9: 1k, rusefi_lib:SM0805_jumper, F.Cu at (141.6, 57.2)
- added SW1: SW_Push, Button_Switch_SMD:SW_SPST_B3SL-1002P, F.Cu at (130.8, 38.2)
- added SW2: SW_Push, Button_Switch_SMD:SW_SPST_B3SL-1002P, F.Cu at (130.8, 29.9)
- D1: renamed from D43; footprint Diode_SMD:D_SOD-323 -> rusefi_lib:SM0805_jumper
- D15: value SS54 -> BLU; footprint Diode_SMD:D_SMA -> rusefi_lib:SM0805_jumper; moved to F.Cu
- D20, D4, D6: value SS54 -> 1N4148WS; footprint Diode_SMD:D_SMA -> rusefi_lib:SM0805_jumper; moved to F.Cu
- D21: value LED-RED -> BLU; footprint LED_SMD:LED_0805_2012Metric -> rusefi_lib:SM0805_jumper
- D22: value LED-GREEN -> 1N4148WS; footprint LED_SMD:LED_0805_2012Metric -> rusefi_lib:SM0805_jumper
- D27: value LED-YELLOW -> BLU; footprint LED_SMD:LED_0805_2012Metric -> rusefi_lib:SM0805_jumper
- D28: renamed from D31; value LED-RED -> RED; footprint LED_SMD:LED_0603_1608Metric -> rusefi_lib:SM0805_jumper
- D29: renamed from D30; footprint Diode_SMD:D_SOD-323 -> rusefi_lib:SM0805_jumper
- D3: value SS54 -> GRN; footprint Diode_SMD:D_SMA -> rusefi_lib:SM0805_jumper; moved to F.Cu
- D32, D34: value 1N4148WS -> RED; footprint Diode_SMD:D_SOD-323 -> rusefi_lib:SM0805_jumper
- D33, D35: value LED-RED -> 1N4148WS; footprint LED_SMD:LED_0603_1608Metric -> rusefi_lib:SM0805_jumper
- D5: value SS54 -> YEL(593NM); footprint Diode_SMD:D_SMA -> rusefi_lib:SM0805_jumper; moved to F.Cu
- D7: value B5819W -> YEL(570NM); footprint Diode_SMD:D_SOD-123 -> rusefi_lib:SM0805_jumper
- D9: renamed from D23; value LED-BLUE -> BLU; footprint LED_SMD:LED_0805_2012Metric -> rusefi_lib:SM0805_jumper
- R1: renamed from R10; footprint Resistor_SMD:R_1206_3216Metric -> rusefi_lib:SM0805_jumper
- R29: value 1k -> 5k; footprint Resistor_SMD:R_0603_1608Metric -> rusefi_lib:SM0805_jumper
- R35: renamed from R36; footprint Resistor_SMD:R_0603_1608Metric -> rusefi_lib:SM0805_jumper
- R49, R51: footprint Resistor_SMD:R_0603_1608Metric -> rusefi_lib:SM0805_jumper
- moved D21 142.9 mm to (172.3, 46.5)
- moved D5 142.3 mm to (176.8, 46.5), turned to 0 degrees
- moved D7 140.4 mm to (176.0, 38.2), turned to 0 degrees
- moved R51 136.6 mm to (160.6, 49.0), turned to 0 degrees
- moved D35 131.8 mm to (158.0, 29.7), turned to 0 degrees
- moved D3 130.7 mm to (164.1, 55.3), turned to 0 degrees
- moved D27 126.1 mm to (159.7, 57.7)
- moved R29 124.0 mm to (177.0, 29.7), turned to 0 degrees
- moved D34 117.5 mm to (141.6, 46.2), turned to 0 degrees
- moved D22 117.4 mm to (139.0, 38.0)
- moved D6 109.7 mm to (145.3, 27.0), turned to 0 degrees
- moved D9 92.9 mm to (125.7, 62.9)
- moved D4 88.5 mm to (128.9, 43.7), turned to 0 degrees
- moved D15 72.7 mm to (159.7, 54.7), turned to 0 degrees
- moved R49 69.5 mm to (166.9, 43.5), turned to 0 degrees
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- renumbered J3 to J1, J5 to J2, J12 to J3, J13 to J4, J4 to J7, LOGO2 to LOGO1, LOGO1 to LOGO2, TP5 to TP1, TP0 to TP2, TP2 to TP3, TP12 to TP5, TP3 to TP6, U3 to U1
Connections:
- D15 pad 1: /12V_MREL -> Net-(D15-Pad1)
- D15 pad 2: (no net) -> Net-(D14-Pad1)
- D20 pad 1: /12V_MREL -> Net-(D20-Pad1)
- D20 pad 2: (no net) -> /GP1
- D21 pad 2: (no net) -> Net-(D20-Pad1)
- D22 pad 2: (no net) -> /GP2
- D27 pad 2: (no net) -> Net-(D26-Pad1)
- D29 pad 2: /5V -> /12V_KEY
- D3 pad 1: /12V_MREL -> Net-(D3-Pad1)
- D3 pad 2: Net-(D3-Pad2) -> Net-(D2-Pad1)
- D32 pad 2: /5V -> Net-(D32-Pad2)
- D33 pad 1: Net-(D33-Pad1) -> Net-(D32-Pad2)
- D33 pad 2: Net-(D32-Pad1) -> /12V_KEY
- D34 pad 2: /5V -> Net-(D34-Pad2)
- D35 pad 1: Net-(D35-Pad1) -> Net-(D34-Pad2)
- D35 pad 2: Net-(D34-Pad1) -> /12V_KEY
- D4 pad 1: /12V_MREL -> Net-(D4-Pad1)
- D4 pad 2: Net-(D4-Pad2) -> /E-THROTTLE+
- D5 pad 1: /12V_MREL -> Net-(D5-Pad1)
- D5 pad 2: Net-(D5-Pad2) -> Net-(D4-Pad1)
- D6 pad 1: /12V_MREL -> /E-THROTTLE+
- D7 pad 1: (no net) -> Net-(D6-Pad2)
- D7 pad 2: (no net) -> Net-(D7-Pad2)
- D9 pad 2: (no net) -> Net-(D8-Pad1)
- J1 pad 1: Net-(D4-Pad2) -> /12V_KEY
- J2 pad 1: Net-(D3-Pad2) -> GND
- J3 pad 1: Net-(D6-Pad2) -> /CRNK+
- J4 pad 1: Net-(D5-Pad2) -> /CRNK-
- J7 pad 2: /12V_MREL -> /12V_KEY
- R29 pad 1: Net-(D28-Pad1) (its old number) -> /12V_KEY
- R29 pad 2: GND -> /AT1
- R35 pad 2: /LS2 -> /AV10
- R49 pad 1: Net-(D33-Pad1) -> Net-(D40-Pad1)
- R49 pad 2: /INJECTOR-1 -> /INJECTOR-3
- R51 pad 1: Net-(D35-Pad1) -> Net-(D42-Pad1)
- R51 pad 2: /GP5 -> /INJECTOR-4
- TP5 pad 1: /12V_MREL -> /12V_KEY
- U1 pad 1: /12V_MREL -> /12V_KEY
- U1 pad 10: (no net) -> /Ign2
- U1 pad 11: (no net) -> /Ign3
- U1 pad 12: (no net) -> /Ign4
- U1 pad 13: (no net) -> /GP6
- U1 pad 18: (no net) -> /AT1
- U1 pad 19: (no net) -> /AV4
- U1 pad 20: (no net) -> /AV5
- U1 pad 22: (no net) -> /AT4
- U1 pad 23: (no net) -> /AT2
- U1 pad 24: (no net) -> /AT3
- U1 pad 25: (no net) -> /CAM_SENSOR
- U1 pad 26: (no net) -> /AV2
- U1 pad 27: (no net) -> /AV1
- U1 pad 28: (no net) -> /AV10
- U1 pad 3: /LS2 -> (no net)
- U1 pad 30: (no net) -> /AV7
- U1 pad 31: (no net) -> /AV3
- U1 pad 32: (no net) -> /AV6
- U1 pad 33: (no net) -> /GP3
- U1 pad 34: (no net) -> /GP2
- U1 pad 35: (no net) -> /GP1
- U1 pad 36: (no net) -> /AV8
- U1 pad 38: (no net) -> /INJECTOR-2
- U1 pad 39: (no net) -> /5V2
- U1 pad 4: (no net) -> /E-THROTTLE+
- U1 pad 40: (no net) -> /AV9
- U1 pad 41: (no net) -> /INJECTOR-3
- U1 pad 42: (no net) -> /INJECTOR-4
- U1 pad 43: (no net) -> /GP4
- U1 pad 44: (no net) -> /5V1
- U1 pad 45: (no net) -> /CRNK+
- U1 pad 46: (no net) -> /CRNK-
- U1 pad 5: (no net) -> /12V_KEY
- U1 pad 8: (no net) -> /E-THROTTLE-
- U1 pad 9: (no net) -> /Ign1
- U1 pad J802: /12V_MREL -> /12V_KEY
Other:
- board size 80.6 x 93.7 mm -> 94.6 x 31.1 mm
- board text removed: "1"
- board text removed: "12V-IGN Ignition power use 1A fuse 12V-Relay main relay output use 5A fuse"
- board text removed: "2"
- board text removed: "3"
- board text removed: "4"
- board text removed: "5"
- board text removed: "6"
- board text removed: "7"
- board text removed: "AT1"
- board text removed: "AT4"
- board text removed: "AV1"
- board text removed: "AV10"
- board text removed: "AV11"
- board text removed: "AV4"
- board text removed: "AV5"
- board text removed: "COMS"
- board text removed: "FATAL"
- board text removed: "HIGH-SIDE LEVEL"
- board text removed: "Hall"
- board text removed: "Optional 33V TVS"
- board text removed: "R0.1 PCB DESIGN BY OLA RUUD R0.2 PCB DESIGN BY DAECU R0.3 PCB DESIGN BY DAECU R0.4 PCB DESIGN BY DBECKER R0.5 PCB DESIGN BY COMMUNITY"
- board text removed: "RUN"
- board text removed: "RUSEFI.COM"
- board text removed: "STM32F407VG"
- board text removed: "TC4427"
- board text removed: "TLE8888"
- board text removed: "V5"
- board text removed: "Vbat"
- board text removed: "WARNING"
- board text removed: "fire extinguisher is required"
- board text removed: "micro rusEFI"
- board text removed: "on when hi/lo GP5 is driving low"

Commit message: draft
Parts:
- removed the R19 at (174.6, 76.8)
- removed the R24 at (158.8, 74.9)
- removed the R25 at (152.4, 81.9)
- removed the R26 at (152.4, 85.1)
- removed the R29 at (177.0, 29.7)
- removed the R36 at (128.9, 51.9)
- removed the R37 at (139.0, 40.7)
- added R15: 5k, rusefi_lib:SM0805_jumper, F.Cu at (25.4, 62.2)
- added R21: 5k, rusefi_lib:SM0805_jumper, F.Cu at (40.6, 62.2)
- added R27: 5k, rusefi_lib:SM0805_jumper, F.Cu at (55.9, 62.2)
- added R30: 1k, rusefi_lib:SM0805_jumper, F.Cu at (58.4, 64.1)
- added R32: 1k, rusefi_lib:SM0805_jumper, F.Cu at (63.5, 64.1)
- moved D7 160.3 mm to (15.9, 45.7), turned to 270 degrees
- moved D5 157.7 mm to (19.1, 45.7), turned to 90 degrees
- moved D3 152.1 mm to (21.0, 3.81), turned to 90 degrees
- moved D13 151.0 mm to (32.4, 3.81), turned to 270 degrees
- moved D11 148.4 mm to (29.2, 3.81), turned to 270 degrees
- moved R3 147.4 mm to (19.1, 52.1), turned to 270 degrees
- moved D17 147.1 mm to (38.7, 3.81), turned to 270 degrees
- moved R17 142.7 mm to (30.5, 62.2), turned to 90 degrees
- moved R23 142.4 mm to (45.7, 62.2)
- moved R24 142.0 mm to (43.2, 64.1)
- moved R5 142.0 mm to (26.0, -2.54), turned to 270 degrees
- moved D21 134.2 mm to (45.1, 3.81), turned to 270 degrees
- moved D15 134.1 mm to (35.6, 3.81), turned to 270 degrees
- moved D25 134.1 mm to (51.4, 3.81), turned to 270 degrees
- moved D19 133.2 mm to (41.9, 3.81), turned to 270 degrees
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- renumbered R30 to R16, R31 to R17, R32 to R18, R33 to R19, R34 to R20, R15 to R23, R16 to R24, R17 to R25, R18 to R26, R20 to R28, R21 to R29, R23 to R31, R27 to R36, R28 to R37
Connections:
- D16 pad 2: /GP6 -> /GP1
- D18 pad 2: /GP5 -> /GP2
- D20 pad 2: /GP1 -> /GP3
- D22 pad 2: /GP2 -> /GP4
- D24 pad 2: /GP3 -> /GP5
- D26 pad 2: /GP4 -> /GP6
- R22 pad 2: /AV4 -> /AT4
- R53 pad 2: /5V1 -> /5V2
- R54 pad 2: /5V2 -> /5V1
- U1 pad 13: /GP6 -> (no net)
- U1 pad 14: /GP5 -> (no net)
Routing:
- net /12V_KEY: track 0.00 -> 359.4 mm
- net /E-THROTTLE-: track 0.00 -> 40.9 mm
- net /5V1: track 0.00 -> 35.6 mm
- net /5V2: track 0.00 -> 34.3 mm
- net /E-THROTTLE+: track 0.00 -> 31.9 mm
- net /CRNK-: track 0.00 -> 30.2 mm
- net /CRNK+: track 0.00 -> 29.9 mm
- net /CAM_SENSOR: track 0.00 -> 13.4 mm
- net GND: track 0.00 -> 10.1 mm
- net /AV7: track 0.00 -> 4.71 mm
- net /AV5: track 0.00 -> 4.71 mm
- net /AV4: track 0.00 -> 4.71 mm
- net /AV3: track 0.00 -> 4.71 mm
- net /AV1: track 0.00 -> 4.71 mm
- net /AT4: track 0.00 -> 4.71 mm
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Other:
- board size 94.6 x 31.1 mm -> 106.7 x 124.5 mm
- board text removed: "Freewheel diodes"
- board text removed: "microRusEfi R0.5.1-2L"

Commit message: draft
Parts:
- removed TP3, TP4: TP, TestPoint:TestPoint_Pad_D2.0mm
Connections:
- net /???? renamed Net-(J6-Pad1)
Other:
- outline, holes or cut-outs redrawn
- board text removed: "8"
- board text removed: "9"
- board text removed: "CAM"
- board text removed: "CRANK"

Commit message: draft
Parts:
- added F1: 1A FUSE, rusefi_lib:Blank, F.Cu at (5.08, 38.7)
- added J8: Conn_01x01_Female, rusefi_lib:KeyStone_3557, F.Cu at (17.6, 16.9)
- added J9: Conn_01x01_Female, rusefi_lib:KeyStone_3557, F.Cu at (17.6, 28.8)
- added R53: 5k, rusefi_lib:SM0805_jumper, F.Cu at (108.0, 33.0)
- added R56: 470k, rusefi_lib:SM0805_jumper, F.Cu at (99.7, 42.5)
- R55: renamed from R53; value 5k -> 470k
- moved J1 29.9 mm to (16.5, 11.4)
- moved J5 22.4 mm to (103.5, 21.6)
- moved SW1 16.0 mm to (109.9, 24.8), turned to 270 degrees
- moved R55 14.9 mm to (99.7, 23.5), turned to 90 degrees
- moved R54 13.0 mm to (108.0, 35.6), turned to 0 degrees
- moved SW2 10.3 mm to (109.9, 41.3), turned to 270 degrees
- moved J6 10.0 mm to (103.5, 44.5)
- moved J4 2.62 mm to (102.9, 33.0)
- moved J3 2.54 mm to (102.9, 29.2)
- renumbered TP5 to TP3, TP6 to TP4
Connections:
- J1 pad 1: /12V_KEY -> Net-(J1-Pad1)
- J6 pad 1: Net-(J6-Pad1) -> /CRNK+
- R54 pad 1: Net-(J6-Pad1) -> /5V1
- R54 pad 2: /5V1 -> Net-(R54-Pad2)
- R55 pad 1: /CAM_SENSOR -> GND
- R55 pad 2: /5V2 -> /CAM_SENSOR
- SW1 pad 1: /CAM_SENSOR -> Net-(R53-Pad2)
- SW1 pad 2: GND -> /CAM_SENSOR
- SW2 pad 1: Net-(J6-Pad1) -> Net-(R54-Pad2)
- SW2 pad 2: GND -> /CRNK+
Routing:
- net /CRNK+: track 29.9 -> 54.5 mm
- net Net-(R53-Pad2): track 0.00 -> 13.0 mm
- net Net-(R54-Pad2): track 0.00 -> 9.89 mm
- net Net-(J1-Pad1): track 0.00 -> 9.25 mm
- net /5V2: track 34.3 -> 40.0 mm
- net /12V_KEY: track 359.4 -> 358.2 mm
- net /CRNK-: track 30.2 -> 29.3 mm
- net /CAM_SENSOR: track 13.4 -> 14.0 mm
Other:
- outline, holes or cut-outs redrawn
- board text removed: "INJ1"
- board text removed: "LS2"

Commit message: Draft
Parts:
- removed the R11 at (45.1, -2.54)
- removed the R12 at (48.3, -2.54)
- removed the R13 at (51.4, -2.54)
- removed the R14 at (54.6, -2.54)
- removed the R43 at (85.7, 10.2)
- removed the R44 at (83.2, 10.2)
- removed the R45 at (91.4, 10.2)
- removed the R46 at (88.9, 10.2)
- removed the R51 at (102.9, 10.2)
- removed the R52 at (100.3, 10.2)
- added D44: 1N4148WS, rusefi_lib:SM0805_jumper, F.Cu at (59.7, 45.1)
- added D45: GRN, rusefi_lib:SM0805_jumper, F.Cu at (59.7, 38.7)
- added R17: 1k, rusefi_lib:SM0805_jumper, F.Cu at (65.4, 45.1)
- added R18: 5k, rusefi_lib:SM0805_jumper, F.Cu at (62.9, 45.1)
- added R23: 1k, rusefi_lib:SM0805_jumper, F.Cu at (105.4, 45.1)
- added R24: 5k, rusefi_lib:SM0805_jumper, F.Cu at (102.9, 45.1)
- added R29: 1k, rusefi_lib:SM0805_jumper, F.Cu at (88.3, 45.1)
- added R30: 5k, rusefi_lib:SM0805_jumper, F.Cu at (85.7, 45.1)
- added R35: 1k, rusefi_lib:SM0805_jumper, F.Cu at (71.1, 45.1)
- added R36: 5k, rusefi_lib:SM0805_jumper, F.Cu at (68.6, 45.1)
- added R47: 1k, rusefi_lib:SM0805_jumper, F.Cu at (111.1, 45.1)
- added R48: 5k, rusefi_lib:SM0805_jumper, F.Cu at (108.6, 45.1)
- added R53: 1k, rusefi_lib:SM0805_jumper, F.Cu at (122.6, 45.1)
- added R54: 5k, rusefi_lib:SM0805_jumper, F.Cu at (120.0, 45.1)
- added R55: 1k, rusefi_lib:SM0805_jumper, F.Cu at (128.3, 45.1)
- added R56: 5k, rusefi_lib:SM0805_jumper, F.Cu at (125.7, 45.1)
- added R61: 1k, rusefi_lib:SM0805_jumper, F.Cu at (59.7, 32.4)
- D20, D22, D24, D26: value 1N4148WS -> RED
- D21, D23, D25, D27: value BLU -> 1N4148WS
- moved D22 63.9 mm to (105.4, 38.7), turned to 90 degrees
- moved D23 63.9 mm to (105.4, 32.4), turned to 90 degrees
- moved D24 46.6 mm to (88.3, 38.7), turned to 90 degrees
- moved D25 46.6 mm to (88.3, 32.4), turned to 90 degrees
- moved D34 43.2 mm to (111.1, 38.7)
- moved D35 43.2 mm to (111.1, 32.4)
- moved D36 43.2 mm to (116.8, 38.7)
- moved D37 43.2 mm to (116.8, 32.4)
- moved D40 43.2 mm to (122.6, 38.7)
- moved D41 43.2 mm to (122.6, 32.4)
- moved D42 43.2 mm to (128.3, 38.7)
- moved D43 43.2 mm to (128.3, 32.4)
- moved R2 41.2 mm to (38.1, 47.6)
- moved D2 41.2 mm to (38.0, 35.0)
- moved D3 41.2 mm to (38.1, 41.3)
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- renumbered J8 to J3, J9 to J4, J3 to J5, J4 to J6, J5 to J7, J6 to J8, J7 to J9, R15 to R11, R16 to R12, R17 to R13, R18 to R14, R19 to R15, R20 to R16, R21 to R19, R22 to R20, R23 to R21, R24 to R22, R29 to R31, R30 to R32, R31 to R33, R32 to R34, R35 to R39, R36 to R40, R37 to R41, R38 to R42, R39 to R43, R40 to R44, R41 to R45, R42 to R46, R47 to R51, R48 to R52, R53 to R57, R54 to R58, R55 to R59, R56 to R60
Connections:
- D16 pad 2: /GP1 -> /GP6
- D18 pad 2: /GP2 -> /GP5
- D20 pad 2: /GP3 -> Net-(D20-Pad2)
- D21 pad 1: Net-(D21-Pad1) -> Net-(D20-Pad2)
- D21 pad 2: Net-(D20-Pad1) -> /12V_KEY
- D22 pad 2: /GP4 -> Net-(D22-Pad2)
- D23 pad 1: Net-(D23-Pad1) -> Net-(D22-Pad2)
- D23 pad 2: Net-(D22-Pad1) -> /12V_KEY
- D24 pad 2: /GP5 -> Net-(D24-Pad2)
- D25 pad 1: Net-(D25-Pad1) -> Net-(D24-Pad2)
- D25 pad 2: Net-(D24-Pad1) -> /12V_KEY
- D26 pad 2: /GP6 -> Net-(D26-Pad2)
- D27 pad 1: Net-(D27-Pad1) -> Net-(D26-Pad2)
- D27 pad 2: Net-(D26-Pad1) -> /12V_KEY
- R39 pad 2: /AV10 -> /GP2
- R42 pad 2: /AV10 -> /GP2
- R43 pad 2: /AV6 -> /GP1
- R44 pad 2: /AV6 -> /GP1
- R49 pad 1: Net-(D40-Pad1) -> Net-(D36-Pad1)
- R49 pad 2: /INJECTOR-3 -> /INJECTOR-2
- R50 pad 2: /INJECTOR-3 -> /INJECTOR-2
- U1 pad 13: (no net) -> /GP6
- U1 pad 14: (no net) -> /GP5
- U1 pad 29: (no net) -> /MAIN_RELAY
Routing:
- net /12V_KEY: track 358.2 -> 421.9 mm
- net Net-(D44-Pad1): track 0.00 -> 3.81 mm
- net Net-(D26-Pad2): track 0.00 -> 3.18 mm
- net Net-(D22-Pad2): track 0.00 -> 3.18 mm
- net Net-(D20-Pad2): track 0.00 -> 3.18 mm
- net Net-(D27-Pad1): track 3.17 -> 0.00 mm
- net Net-(D25-Pad1): track 3.17 -> 0.00 mm
- net Net-(D23-Pad1): track 3.17 -> 0.00 mm
- net Net-(D21-Pad1): track 3.17 -> 0.00 mm
- net Net-(D45-Pad1): track 0.00 -> 3.17 mm
- net Net-(D24-Pad2): track 0.00 -> 3.17 mm
- net /AV10: track 2.80 -> 0.00 mm
- net /GP3: track 0.00 -> 2.54 mm
- net /GP4: track 0.00 -> 2.54 mm
- net /GP2: track 0.00 -> 2.54 mm
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- added copper zone on B.Cu, net GND
- added copper zone on F.Cu, net GND
Other:
- outline, holes or cut-outs redrawn

Commit message: Draft
Parts:
- removed the R11 at (45.7, 97.2)
- removed the R13 at (50.8, 97.2)
- removed the R15 at (55.9, 97.2)
- removed the R19 at (61.0, 97.2)
- removed the R31 at (81.3, 97.2)
- removed R33: 5k, rusefi_lib:SM0805_jumper
- added R16: 10k, rusefi_lib:SM0805_jumper, F.Cu at (81.3, 97.2)
- added R22: 10k, rusefi_lib:SM0805_jumper, F.Cu at (86.4, 97.2)
- R13: renamed from R14; value 1k -> 2k2
- R14: renamed from R16; value 1k -> 3k3
- R15: renamed from R20; value 1k -> 4k7
- R17: renamed from R32; value 1k -> 220R
- R21: renamed from R22; value 1k -> 220R
- R23: renamed from R34; value 1k -> 470R
- R27: renamed from R26; value 1k -> 470R
- R28: renamed from R40; value 5k -> 10k
- renumbered D44 to D20, D45 to D21, D20 to D44, D21 to D45, R61 to R11, R23 to R18, R24 to R19, R21 to R20, R29 to R24, R30 to R25, R25 to R26, R41 to R29, R35 to R30, R36 to R31, R39 to R34, R27 to R35, R28 to R36, R42 to R37, R43 to R38, R44 to R39, R45 to R40, R46 to R41, R47 to R42, R48 to R43, R49 to R44, R50 to R45, R51 to R46, R52 to R47, R53 to R48, R54 to R49, R55 to R50, R56 to R51, R17 to R52, R18 to R53, R57 to R54, R58 to R55, R59 to R56, R60 to R57
Connections:
- R17 pad 2: /AV4 -> /AV1
- R20 pad 2: /AV1 -> /AV2
- R21 pad 2: /AV1 -> /AV2
- R23 pad 2: /AV5 -> /AV3
- R26 pad 2: /AV2 -> /AV4
- R27 pad 2: /AV2 -> /AV4
- R28 pad 2: /AV7 -> /AV5
- R29 pad 2: /AV7 -> /AV5
- R35 pad 2: /AV3 -> /AV7
- R36 pad 2: /AV3 -> /AV7
Routing:
- net /AT4: track 4.71 -> 0.00 mm
- net /AT3: track 4.71 -> 0.00 mm
- net /AT1: track 4.71 -> 0.00 mm
- net /AT2: track 4.71 -> 0.00 mm

Commit message: draft
Routing:
- net /AV6: track 2.54 -> 101.0 mm
- net /12V_SAFE: track 0.00 -> 56.8 mm
- net /AT1: track 0.00 -> 49.8 mm
- net /GP4: track 2.54 -> 52.3 mm, vias 0 -> 1
- net /AT4: track 0.00 -> 48.6 mm
- net /AT2: track 0.00 -> 45.8 mm
- net /CAM_SENSOR: track 14.0 -> 58.7 mm
- net /INJECTOR-4: track 2.54 -> 46.6 mm
- net /Ign3: track 0.00 -> 44.0 mm
- net /Ign2: track 0.00 -> 42.9 mm
- net /Ign1: track 0.00 -> 42.2 mm
- net /AT3: track 0.00 -> 41.4 mm
- net /AV10: track 0.00 -> 41.0 mm, vias 0 -> 1
- net /INJECTOR-3: track 2.54 -> 42.6 mm
- net /Ign4: track 0.00 -> 39.6 mm
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Other:
- board text removed: "Program"
- board text removed: "Reset"

Commit message: silk and text progress
Parts:
- moved J2 20.2 mm to (40.6, 63.5)
- moved J4 2.84 mm to (34.1, 67.0)
- moved J3 2.84 mm to (34.1, 55.1)
Routing:
- net Net-(J1-Pad1): vias 0 -> 1
- net GND: vias 209 -> 206
- net /12V_KEY: vias 0 -> 2
Other:
- board text added: "+12v"
- board text added: "1 2 3 4 6 5"
- board text added: "GP4 GP3 GP2 GP1 AV6 AV8 AV9 AV10 IJ1 IJ2 IJ3 IJ4"
- board text added: "microRusEFI text fixture 0.1"
Changed lines of the file:
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@@
   (general
     (thickness 1.6)
-    (drawings 43)
+    (drawings 50)
     (tracks 1136)
     (zones 0)
@@
   )
   (layers
-    (0 F.Cu signal)
-    (31 B.Cu signal)
+    (0 F.Cu signal hide)
+    (31 B.Cu signal hide)
     (32 B.Adhes user)
     (33 F.Adhes user)
@@
     (mod_text_size 0.75 0.75)
     (mod_text_width 0.13)
-    (pad_size 2 3.8)
-    (pad_drill 0)
+    (pad_size 1.6 1.6)
+    (pad_drill 1.2)
     (pad_to_mask_clearance 0.000076)
     (aux_axis_origin 0 0)
@@
   )
   (module rusefi_lib:KeyStone_3557 (layer F.Cu)
-    (at 35.3525 64.4418 90)
-    (fp_text reference J4 (at 4.445 3.2555 90) (layer F.SilkS)
+    (at 34.0825 66.9818 90)
+    (fp_text reference J4 (at 4.445 3.2555 90) (layer F.SilkS) hide
       (effects (font (size 1 1) (thickness 0.15)))
     )
@@
   )
   (module rusefi_lib:KeyStone_3557 (layer F.Cu)
-    (at 35.3568 52.578 270)
-    (fp_text reference J3 (at 4.445 -3.175 90) (layer F.SilkS)
+    (at 34.0868 55.118 270)
+    (fp_text reference J3 (at 4.445 -3.175 90) (layer F.SilkS) hide
       (effects (font (size 1 1) (thickness 0.15)))
     )
@@
   )
   (module Connector_Pin:Pin_D0.7mm_L6.5mm_W1.8mm_FlatFork (layer F.Cu)
-    (at 60.325 67.945 270)
+    (at 40.64 63.5 270)
     (descr "solder Pin_ with flat fork, hole diameter 0.7mm, length 6.5mm, width 1.8mm")
     (tags "solder Pin_ with flat fork")
-    (fp_text reference J2 (at 0 1.8 90) (layer B.SilkS)
+    (fp_text reference J2 (at 0 1.8 90) (layer B.SilkS) hide
       (effects (font (size 1 1) (thickness 0.15)) (justify mirror))
     )
@@
       (effects (font (size 1 1) (thickness 0.15)))
     )
-    (pad 1 thru_hole circle (at 0 0 270) (size 1.4 1.4) (drill 0.7) (layers *.Cu *.Mask)
+    (pad 1 thru_hole circle (at 0 0 270) (size 1.6 1.6) (drill 1.2) (layers *.Cu *.Mask)
       (net 1 GND))
   )
@@
     (descr "solder Pin_ with flat fork, hole diameter 0.7mm, length 6.5mm, width 1.8mm")
     (tags "solder Pin_ with flat fork")
-    (fp_text reference J1 (at 0 1.905 90) (layer B.SilkS)
+    (fp_text reference J1 (at 0 1.905 90) (layer B.SilkS) hide
       (effects (font (size 1 1) (thickness 0.15)) (justify mirror))
     )
@@
       (effects (font (size 1 1) (thickness 0.15)))
     )
-    (pad 1 thru_hole circle (at 0 0 270) (size 1.4 1.4) (drill 0.7) (layers *.Cu *.Mask)
+    (pad 1 thru_hole circle (at 0 0 270) (size 1.6 1.6) (drill 1.2) (layers *.Cu *.Mask)
       (net 87 "Net-(J1-Pad1)"))
   )
@@
       (xy 3.3528 0.39624)) (layer B.SilkS) (width 0.00254))
   )
+  (gr_text "1 2  3 4  6 5" (at 40.64 49.53) (layer F.SilkS)
+    (effects (font (size 1.5 1.5) (thickness 0.13)) (justify left))
+  )
+  (gr_text "GP4  GP3  GP2  GP1  AV6   AV8   AV9  AV10  IJ1   IJ2    IJ3    IJ4" (at 63.5 49.53) (layer F.SilkS)
+    (effects (font (size 1.2 1.2) (thickness 0.13)) (justify left))
+  )
+  (gr_text "microRusEFI text fixture 0.1" (at 127 116.84 90) (layer F.SilkS)
+    (effects (font (size 3 3) (thickness 0.13)))
+  )
+  (gr_text GND (at 40.64 60.96) (layer B.SilkS)
+    (effects (font (size 1.5 1.5) (thickness 0.13)) (justify mirror))
+  )
+  (gr_text GND (at 40.64 60.96) (layer F.SilkS)
+    (effects (font (size 1.5 1.5) (thickness 0.13)))
+  )
+  (gr_text +12v (at 34.29 44.45) (layer F.SilkS)
+    (effects (font (size 1.5 1.5) (thickness 0.13)))
+  )
+  (gr_text +12v (at 34.29 44.45) (layer B.SilkS)
+    (effects (font (size 1.5 1.5) (thickness 0.13)) (justify mirror))
+  )
   (gr_circle (center 50.165 67.945) (end 50.165 66.675) (layer Edge.Cuts) (width 0.2))
   (gr_circle (center 46.355 67.945) (end 46.355 66.675) (layer Edge.Cuts) (width 0.2))
@@
   (via (at 40.894 61.849) (size 0.6) (drill 0.3) (layers F.Cu B.Cu) (net 1))
   (via (at 34.544 61.849) (size 0.6) (drill 0.3) (layers F.Cu B.Cu) (net 1))
-  (via (at 36.195 66.675) (size 0.6) (drill 0.3) (layers F.Cu B.Cu) (net 1))
+  (via (at 36.195 66.675) (size 0.6) (drill 0.3) (layers F.Cu B.Cu) (net 22))
   (via (at 41.529 66.675) (size 0.6) (drill 0.3) (layers F.Cu B.Cu) (net 1))
   (via (at 57.785 66.167) (size 0.6) (drill 0.3) (layers F.Cu B.Cu) (net 1))
   (segment (start 63.3088 66.9932) (end 61.2768 66.9932) (width 1.6764) (layer F.Cu) (net 1))
   (via (at 63.3088 66.9932) (size 0.6) (drill 0.3) (layers F.Cu B.Cu) (net 1))
-  (via (at 33.02 55.118) (size 0.6) (drill 0.3) (layers F.Cu B.Cu) (net 1))
-  (via (at 32.258 66.421) (size 0.6) (drill 0.3) (layers F.Cu B.Cu) (net 1))
+  (via (at 33.02 55.118) (size 0.6) (drill 0.3) (layers F.Cu B.Cu) (net 87))
+  (via (at 32.258 66.421) (size 0.6) (drill 0.3) (layers F.Cu B.Cu) (net 22))
   (via (at 31.75 78.613) (size 0.6) (drill 0.3) (layers F.Cu B.Cu) (net 1))
   (via (at 42.672 80.137) (size 0.6) (drill 0.3) (layers F.Cu B.Cu) (net 1))
