File: zMRETestFixture.kicad_pcb (KiCad board)
At the start: 2 copper layers, 106.7 x 124.5 mm, 120 parts, among them J1 Conn_01x01, J2 Conn_01x01, J3 Conn_01x01_Female, J4 Conn_01x01_Female, J5 Conn_01x01, J6 Conn_01x01, J7 Conn_01x01, J8 Conn_01x01, J9 Conn_02x05_Counter_Clockwise, SW1 SW_Push, SW2 SW_Push, U1 molex_48pin_MRE

Commit message: DRAFT
Parts:
- moved J1 0.65 mm to (34.3, 47.6)
Routing:
- net GND: track 10.1 -> 3.70 mm, vias 206 -> 203
- net /12V_KEY: track 461.1 -> 464.6 mm, vias 2 -> 0
- net Net-(J1-Pad1): track 10.7 -> 11.6 mm, vias 1 -> 0
Other:
- outline, holes or cut-outs redrawn

Commit message: DRAFT`
Parts:
- removed R34: 1k, rusefi_lib:SM0805_jumper
- added D46: 1N4148WS, rusefi_lib:SM0805_jumper, F.Cu at (45.1, 150.5)
- added D47: 1N4148WS, rusefi_lib:SM0805_jumper, F.Cu at (45.1, 148.0)
- added D48: 1N4148WS, rusefi_lib:SM0805_jumper, F.Cu at (45.1, 145.4)
- added D49: 1N4148WS, rusefi_lib:SM0805_jumper, F.Cu at (45.1, 142.9)
- added D50: 1N4148WS, rusefi_lib:SM0805_jumper, F.Cu at (45.1, 140.3)
- added D51: 1N4148WS, rusefi_lib:SM0805_jumper, F.Cu at (45.1, 137.8)
- added D52: 1N4148WS, rusefi_lib:SM0805_jumper, F.Cu at (45.1, 135.3)
- added D53: 1N4148WS, rusefi_lib:SM0805_jumper, F.Cu at (45.1, 132.7)
- added D54: 1N4148WS, rusefi_lib:SM0805_jumper, F.Cu at (45.1, 130.2)
- added D55: 1N4148WS, rusefi_lib:SM0805_jumper, F.Cu at (45.1, 127.6)
- added D56: 1N4148WS, rusefi_lib:SM0805_jumper, F.Cu at (45.1, 125.1)
- added D57: 1N4148WS, rusefi_lib:SM0805_jumper, F.Cu at (45.1, 122.6)
- added D58: 1N4148WS, rusefi_lib:SM0805_jumper, F.Cu at (45.1, 120.0)
- added D59: 1N4148WS, rusefi_lib:SM0805_jumper, F.Cu at (45.1, 117.5)
- added D60: 1N4148WS, rusefi_lib:SM0805_jumper, F.Cu at (45.1, 114.9)
- added D61: GRN, rusefi_lib:SM0805_jumper, F.Cu at (51.4, 153.0)
- added D62: GRN, rusefi_lib:SM0805_jumper, F.Cu at (51.4, 150.5)
- added D63: GRN, rusefi_lib:SM0805_jumper, F.Cu at (51.4, 148.0)
- added D64: GRN, rusefi_lib:SM0805_jumper, F.Cu at (51.4, 145.4)
- added D65: GRN, rusefi_lib:SM0805_jumper, F.Cu at (51.4, 142.9)
- added D66: GRN, rusefi_lib:SM0805_jumper, F.Cu at (51.4, 140.3)
- added D67: GRN, rusefi_lib:SM0805_jumper, F.Cu at (51.4, 137.8)
- added D68: GRN, rusefi_lib:SM0805_jumper, F.Cu at (51.4, 135.3)
- added D69: GRN, rusefi_lib:SM0805_jumper, F.Cu at (51.4, 132.7)
- added D70: GRN, rusefi_lib:SM0805_jumper, F.Cu at (51.4, 130.2)
- added D71: GRN, rusefi_lib:SM0805_jumper, F.Cu at (51.4, 127.6)
- added D72: GRN, rusefi_lib:SM0805_jumper, F.Cu at (51.4, 125.1)
- added D73: GRN, rusefi_lib:SM0805_jumper, F.Cu at (51.4, 122.6)
- added D74: GRN, rusefi_lib:SM0805_jumper, F.Cu at (51.4, 120.0)
- added D75: GRN, rusefi_lib:SM0805_jumper, F.Cu at (51.4, 117.5)
- added D76: GRN, rusefi_lib:SM0805_jumper, F.Cu at (51.4, 114.9)
- added D77: RED, rusefi_lib:SM0805_jumper, F.Cu at (40.6, 73.0)
- added D78: 1N4148WS, rusefi_lib:SM0805_jumper, F.Cu at (34.3, 73.0)
- added D79: RED, rusefi_lib:SM0805_jumper, F.Cu at (40.6, 78.1)
- added D80: 1N4148WS, rusefi_lib:SM0805_jumper, F.Cu at (34.3, 78.1)
- added D81: RED, rusefi_lib:SM0805_jumper, F.Cu at (40.6, 83.2)
- added D82: 1N4148WS, rusefi_lib:SM0805_jumper, F.Cu at (34.3, 83.2)
- added D83: RED, rusefi_lib:SM0805_jumper, F.Cu at (40.6, 88.3)
- added D84: 1N4148WS, rusefi_lib:SM0805_jumper, F.Cu at (34.3, 88.3)
- added D85: RED, rusefi_lib:SM0805_jumper, F.Cu at (40.6, 93.3)
- added D86: 1N4148WS, rusefi_lib:SM0805_jumper, F.Cu at (34.3, 93.3)
- added D87: RED, rusefi_lib:SM0805_jumper, F.Cu at (40.6, 98.4)
- added D88: 1N4148WS, rusefi_lib:SM0805_jumper, F.Cu at (34.3, 98.4)
- added D89: RED, rusefi_lib:SM0805_jumper, F.Cu at (40.6, 103.5)
- added D90: 1N4148WS, rusefi_lib:SM0805_jumper, F.Cu at (34.3, 103.5)
- added D91: 1N4148WS, rusefi_lib:SM0805_jumper, F.Cu at (124.5, 79.4)
- added D92: RED, rusefi_lib:SM0805_jumper, F.Cu at (40.6, 108.6)
- added D93: 1N4148WS, rusefi_lib:SM0805_jumper, F.Cu at (34.3, 108.6)
- added J10: Conn_01x01, Connector_Pin:Pin_D0.7mm_L6.5mm_W1.8mm_FlatFork, F.Cu at (116.2, 123.2)
- added J11: Conn_01x01, Connector_Pin:Pin_D0.7mm_L6.5mm_W1.8mm_FlatFork, F.Cu at (116.2, 120.0)
- added R32: 5k, rusefi_lib:SM0805_jumper, F.Cu at (87.6, 45.1)
- added R58: 470k, rusefi_lib:SM0805_jumper, F.Cu at (142.2, 77.5)
- added R59: 1k, rusefi_lib:SM0805_jumper, F.Cu at (57.8, 153.0)
- added R60: 1k, rusefi_lib:SM0805_jumper, F.Cu at (57.8, 150.5)
- added R61: 1k, rusefi_lib:SM0805_jumper, F.Cu at (57.8, 148.0)
- added R62: 1k, rusefi_lib:SM0805_jumper, F.Cu at (57.8, 145.4)
- added R63: 1k, rusefi_lib:SM0805_jumper, F.Cu at (57.8, 142.9)
- added R64: 1k, rusefi_lib:SM0805_jumper, F.Cu at (57.8, 140.3)
- added R65: 1k, rusefi_lib:SM0805_jumper, F.Cu at (57.8, 137.8)
- added R66: 1k, rusefi_lib:SM0805_jumper, F.Cu at (57.8, 135.3)
- added R67: 1k, rusefi_lib:SM0805_jumper, F.Cu at (57.8, 132.7)
- added R68: 1k, rusefi_lib:SM0805_jumper, F.Cu at (57.8, 130.2)
- added R69: 1k, rusefi_lib:SM0805_jumper, F.Cu at (57.8, 127.6)
- added R70: 1k, rusefi_lib:SM0805_jumper, F.Cu at (57.8, 125.1)
- added R71: 1k, rusefi_lib:SM0805_jumper, F.Cu at (57.8, 122.6)
- added R72: 1k, rusefi_lib:SM0805_jumper, F.Cu at (57.8, 120.0)
- added R73: 1k, rusefi_lib:SM0805_jumper, F.Cu at (57.8, 117.5)
- added R74: 1k, rusefi_lib:SM0805_jumper, F.Cu at (57.8, 114.9)
- added R75: 1k, rusefi_lib:SM0805_jumper, F.Cu at (47.0, 73.0)
- added R76: 5k, rusefi_lib:SM0805_jumper, F.Cu at (47.0, 75.6)
- added R77: 1k, rusefi_lib:SM0805_jumper, F.Cu at (47.0, 78.1)
- added R78: 5k, rusefi_lib:SM0805_jumper, F.Cu at (47.0, 80.6)
- added R79: 1k, rusefi_lib:SM0805_jumper, F.Cu at (47.0, 83.2)
- added R80: 5k, rusefi_lib:SM0805_jumper, F.Cu at (47.0, 85.7)
- added R81: 1k, rusefi_lib:SM0805_jumper, F.Cu at (47.0, 88.3)
- added R82: 5k, rusefi_lib:SM0805_jumper, F.Cu at (47.0, 90.8)
- added R83: 1k, rusefi_lib:SM0805_jumper, F.Cu at (47.0, 93.3)
- added R84: 5k, rusefi_lib:SM0805_jumper, F.Cu at (47.0, 95.9)
- added R85: 1k, rusefi_lib:SM0805_jumper, F.Cu at (47.0, 98.4)
- added R86: 5k, rusefi_lib:SM0805_jumper, F.Cu at (47.0, 101.0)
- added R87: 1k, rusefi_lib:SM0805_jumper, F.Cu at (47.0, 103.5)
- added R88: 1k, rusefi_lib:SM0805_jumper, F.Cu at (121.9, 81.3)
- added R89: 5k, rusefi_lib:SM0805_jumper, F.Cu at (47.0, 106.0)
- added R90: 1k, rusefi_lib:SM0805_jumper, F.Cu at (47.0, 108.6)
- added R91: 5k, rusefi_lib:SM0805_jumper, F.Cu at (47.0, 111.1)
- D10, D12, D14, D16, D18, D8: value 1N4148WS -> BLU
- D11, D13, D15, D17, D9: value BLU -> 1N4148WS
- D19: value BLU -> RED
- D2: value 1N4148WS -> GRN
- D21: value GRN -> RED
- D22, D24, D26, D28, D30, D32, D34, D36, D38, D40, D42, D44: value RED -> 1N4148WS
- D23, D25, D27, D29, D31, D33, D35, D37, D39, D41, D43: value 1N4148WS -> RED
- D3: value GRN -> 1N4148WS
- D4: value 1N4148WS -> YEL(593NM)
- D5: value YEL(593NM) -> 1N4148WS
- D6: value 1N4148WS -> YEL(570NM)
- D7: value YEL(570NM) -> 1N4148WS
- R1: value 1k -> 0R
- R12, R24, R30: value 1k -> 2k2
- R13: value 2k2 -> 3k3
- R14: value 3k3 -> 1k
- R15: value 4k7 -> 5k
- R16: value 10k -> 4k7
- R17: value 220R -> 10k
- R19, R25, R31, R35, R39, R41, R43, R45, R47, R49, R51, R53: value 5k -> 1k
- R21: value 220R -> 5k
- R22: value 10k -> 1k
- R23, R27: value 470R -> 10k
- R28: value 10k -> 3k3
- R29, R36, R38, R40, R42, R44, R46, R48, R50, R52: value 1k -> 5k
- R37: value 5k -> 4k7
- R56: value 470k -> 5k
- moved D45 122.3 mm to (45.1, 153.0), turned to 180 degrees
- moved R14 89.8 mm to (125.1, 45.1), turned to 270 degrees
- moved R15 87.8 mm to (127.6, 45.1), turned to 270 degrees
- moved R52 85.1 mm to (150.5, 45.1)
- moved R22 72.0 mm to (42.5, 40.0), turned to 0 degrees
- moved R29 71.5 mm to (44.3, 47.6), turned to 0 degrees
- moved R16 71.2 mm to (42.4, 37.5), turned to 0 degrees
- moved D19 68.6 mm to (125.1, 38.7), turned to 90 degrees
- moved R12 66.7 mm to (42.4, 32.4), turned to 0 degrees
- moved D20 66.6 mm to (125.1, 32.4), turned to 90 degrees
- moved R26 65.3 mm to (110.5, 45.1), turned to 270 degrees
- moved R20 64.9 mm to (104.8, 45.1), turned to 270 degrees
- moved D1 64.7 mm to (57.8, 32.4), turned to 90 degrees
- moved R13 64.4 mm to (42.4, 34.9), turned to 0 degrees
- moved R18 63.7 mm to (42.5, 55.2), turned to 0 degrees
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Connections:
- D1 pad 2: /12V_SAFE -> /12V_MREL
- D10 pad 2: /Ign2 -> Net-(D10-Pad2)
- D11 pad 2: Net-(D10-Pad1) -> /Ign3
- D12 pad 2: /Ign3 -> Net-(D11-Pad1)
- D13 pad 2: Net-(D12-Pad1) -> /Ign4
- D14 pad 2: /Ign4 -> Net-(D13-Pad1)
- D15 pad 2: Net-(D14-Pad1) -> /GP6
- D16 pad 2: /GP6 -> Net-(D15-Pad1)
- D17 pad 2: Net-(D16-Pad1) -> /GP5
- D18 pad 2: /GP5 -> Net-(D17-Pad1)
- D19 pad 2: Net-(D18-Pad1) -> Net-(D19-Pad2)
- D2 pad 2: /12V_KEY -> Net-(D1-Pad1)
- D20 pad 1: Net-(D20-Pad1) -> Net-(D19-Pad2)
- D20 pad 2: /MAIN_RELAY -> /12V_MREL
- D21 pad 2: Net-(D20-Pad1) -> Net-(D21-Pad2)
- D22 pad 1: Net-(D22-Pad1) -> Net-(D21-Pad2)
- D22 pad 2: Net-(D22-Pad2) -> /12V_MREL
- D23 pad 1: Net-(D22-Pad2) -> Net-(D23-Pad1)
- D23 pad 2: /12V_KEY -> Net-(D23-Pad2)
- D24 pad 1: Net-(D24-Pad1) -> Net-(D23-Pad2)
- D24 pad 2: Net-(D24-Pad2) -> /12V_MREL
- D25 pad 1: Net-(D24-Pad2) -> Net-(D25-Pad1)
- D25 pad 2: /12V_KEY -> Net-(D25-Pad2)
- D26 pad 1: Net-(D26-Pad1) -> Net-(D25-Pad2)
- D26 pad 2: Net-(D26-Pad2) -> /12V_MREL
- D27 pad 1: Net-(D26-Pad2) -> Net-(D27-Pad1)
- D27 pad 2: /12V_KEY -> Net-(D27-Pad2)
- D28 pad 1: Net-(D28-Pad1) -> Net-(D27-Pad2)
- D28 pad 2: Net-(D28-Pad2) -> /12V_MREL
- D29 pad 1: Net-(D28-Pad2) -> Net-(D29-Pad1)
- D29 pad 2: /12V_KEY -> Net-(D29-Pad2)
- D3 pad 2: Net-(D2-Pad1) -> /E-THROTTLE+
- D30 pad 1: Net-(D30-Pad1) -> Net-(D29-Pad2)
- D30 pad 2: Net-(D30-Pad2) -> /12V_MREL
- D31 pad 1: Net-(D30-Pad2) -> Net-(D31-Pad1)
- D31 pad 2: /12V_KEY -> Net-(D31-Pad2)
- D32 pad 1: Net-(D32-Pad1) -> Net-(D31-Pad2)
- D32 pad 2: Net-(D32-Pad2) -> /12V_MREL
- D33 pad 1: Net-(D32-Pad2) -> Net-(D33-Pad1)
- D33 pad 2: /12V_KEY -> Net-(D33-Pad2)
- D34 pad 1: Net-(D34-Pad1) -> Net-(D33-Pad2)
- D34 pad 2: Net-(D34-Pad2) -> /12V_MREL
- D35 pad 1: Net-(D34-Pad2) -> Net-(D35-Pad1)
- D35 pad 2: /12V_KEY -> Net-(D35-Pad2)
- D36 pad 1: Net-(D36-Pad1) -> Net-(D35-Pad2)
- D36 pad 2: Net-(D36-Pad2) -> /12V_MREL
- D37 pad 1: Net-(D36-Pad2) -> Net-(D37-Pad1)
- D37 pad 2: /12V_KEY -> Net-(D37-Pad2)
- D38 pad 1: Net-(D38-Pad1) -> Net-(D37-Pad2)
- D38 pad 2: Net-(D38-Pad2) -> /12V_MREL
- D39 pad 1: Net-(D38-Pad2) -> Net-(D39-Pad1)
- D39 pad 2: /12V_KEY -> Net-(D39-Pad2)
- D4 pad 2: /E-THROTTLE+ -> Net-(D3-Pad1)
- D40 pad 1: Net-(D40-Pad1) -> Net-(D39-Pad2)
- D40 pad 2: Net-(D40-Pad2) -> /12V_MREL
- D41 pad 1: Net-(D40-Pad2) -> Net-(D41-Pad1)
- D41 pad 2: /12V_KEY -> Net-(D41-Pad2)
- D42 pad 1: Net-(D42-Pad1) -> Net-(D41-Pad2)
- D42 pad 2: Net-(D42-Pad2) -> /12V_MREL
- D43 pad 1: Net-(D42-Pad2) -> Net-(D43-Pad1)
- D43 pad 2: /12V_KEY -> Net-(D43-Pad2)
- D44 pad 1: Net-(D44-Pad1) -> Net-(D43-Pad2)
- D44 pad 2: Net-(D44-Pad2) -> /12V_MREL
- D45 pad 1: Net-(D44-Pad2) -> Net-(D45-Pad1)
- D45 pad 2: /12V_KEY -> /PA15
- D5 pad 1: Net-(D5-Pad1) -> /E-THROTTLE+
- D5 pad 2: Net-(D4-Pad1) -> Net-(D5-Pad2)
- D6 pad 1: /E-THROTTLE+ -> Net-(D5-Pad2)
- D7 pad 1: Net-(D6-Pad2) -> Net-(D7-Pad1)
- D7 pad 2: Net-(D7-Pad2) -> /Ign1
- D8 pad 2: /Ign1 -> Net-(D7-Pad1)
- D9 pad 1: Net-(D9-Pad1) -> Net-(D10-Pad2)
- D9 pad 2: Net-(D8-Pad1) -> /Ign2
- J4 pad 1: /12V_KEY -> /12V_MREL
- J9 pad 2: /12V_KEY -> /12V_MREL
- R1 pad 1: Net-(D1-Pad1) -> /12V_MREL
- R1 pad 2: /LINBUS -> /12V_KEY
- R10 pad 2: Net-(D19-Pad1) -> Net-(D18-Pad1)
- R11 pad 2: Net-(D21-Pad1) -> /AT1
- R12 pad 2: /AT1 -> /AT2
- R13 pad 2: /AT2 -> /AT3
- R14 pad 1: GND -> Net-(D19-Pad1)
- R14 pad 2: /AT3 -> /AV10
- R15 pad 1: GND -> /12V_MREL
- R15 pad 2: /AT4 -> /AV10
- R16 pad 1: /12V_KEY -> GND
- R16 pad 2: /AV1 -> /AT4
- R17 pad 1: GND -> /5V1
- R18 pad 1: Net-(D22-Pad1) -> GND
- R18 pad 2: /AV10 -> /AV1
- R19 pad 1: /12V_KEY -> Net-(D21-Pad1)
- R19 pad 2: /AV10 -> /MAIN_RELAY
- R2 pad 1: Net-(D3-Pad1) -> Net-(D2-Pad1)
- R20 pad 1: /12V_KEY -> /12V_MREL
- R20 pad 2: /AV2 -> /MAIN_RELAY
- R21 pad 1: GND -> /5V1
- R22 pad 1: /12V_KEY -> GND
- R22 pad 2: /AV3 -> /AV2
- R23 pad 1: GND -> /5V1
- R24 pad 1: Net-(D24-Pad1) -> GND
- R24 pad 2: /AV6 -> /AV3
- R25 pad 1: /12V_KEY -> Net-(D23-Pad1)
- R26 pad 1: /12V_KEY -> /12V_MREL
- R26 pad 2: /AV4 -> /AV6
- R27 pad 1: GND -> /5V1
- R28 pad 1: /12V_KEY -> GND
- R28 pad 2: /AV5 -> /AV4
- R29 pad 1: GND -> /5V2
- R3 pad 1: Net-(D5-Pad1) -> Net-(D4-Pad1)
- R30 pad 1: Net-(D26-Pad1) -> GND
- R30 pad 2: /GP3 -> /AV5
- R31 pad 1: /12V_KEY -> Net-(D25-Pad1)
- R35 pad 1: /12V_KEY -> Net-(D27-Pad1)
- R35 pad 2: /AV7 -> /GP2
- R36 pad 1: GND -> /5V2
- R37 pad 1: /12V_KEY -> GND
- R37 pad 2: /GP2 -> /AV7
- R38 pad 1: Net-(D30-Pad1) -> /12V_MREL
- R38 pad 2: /GP1 -> /GP2
- R39 pad 1: /12V_KEY -> Net-(D29-Pad1)
- R4 pad 1: Net-(D7-Pad2) -> Net-(D6-Pad2)
- R40 pad 1: Net-(D32-Pad1) -> /12V_MREL
- R40 pad 2: /AV8 -> /GP1
- R41 pad 1: /12V_KEY -> Net-(D31-Pad1)
- R42 pad 1: Net-(D34-Pad1) -> /12V_MREL
- R42 pad 2: /INJECTOR-1 -> /AV8
- R43 pad 1: /12V_KEY -> Net-(D33-Pad1)
- R44 pad 1: Net-(D36-Pad1) -> /12V_MREL
- R44 pad 2: /INJECTOR-2 -> /INJECTOR-1
- R45 pad 1: /12V_KEY -> Net-(D35-Pad1)
- R46 pad 1: Net-(D38-Pad1) -> /12V_MREL
- R46 pad 2: /AV9 -> /INJECTOR-2
- R47 pad 1: /12V_KEY -> Net-(D37-Pad1)
- R48 pad 1: Net-(D40-Pad1) -> /12V_MREL
- R48 pad 2: /INJECTOR-3 -> /AV9
- R49 pad 1: /12V_KEY -> Net-(D39-Pad1)
- R5 pad 2: Net-(D9-Pad1) -> Net-(D8-Pad1)
- R50 pad 1: Net-(D42-Pad1) -> /12V_MREL
- R50 pad 2: /INJECTOR-4 -> /INJECTOR-3
- R51 pad 1: /12V_KEY -> Net-(D41-Pad1)
- R52 pad 1: Net-(D44-Pad1) -> /12V_MREL
- R52 pad 2: /GP4 -> /INJECTOR-4
- R53 pad 1: /12V_KEY -> Net-(D43-Pad1)
- R54 pad 1: /5V2 -> /12V_MREL
- R54 pad 2: Net-(R54-Pad2) -> /GP4
- R55 pad 1: /5V1 -> /5V2
- R56 pad 1: GND -> /5V1
- R56 pad 2: /CAM_SENSOR -> Net-(R56-Pad2)
- R57 pad 2: /CRNK+ -> /CAM_SENSOR
- R6 pad 2: Net-(D11-Pad1) -> Net-(D10-Pad1)
- R7 pad 2: Net-(D13-Pad1) -> Net-(D12-Pad1)
- R8 pad 2: Net-(D15-Pad1) -> Net-(D14-Pad1)
- R9 pad 2: Net-(D17-Pad1) -> Net-(D16-Pad1)
- SW1 pad 1: Net-(R54-Pad2) -> Net-(R55-Pad2)
- SW2 pad 1: Net-(R55-Pad2) -> Net-(R56-Pad2)
- TP3 pad 1: /12V_KEY -> /12V_MREL
- U1 pad 1: /12V_KEY -> /12V_MREL
- U1 pad 3: (no net) -> /LS2
- U1 pad 7: (no net) -> /LS1
- U1 pad J10: (no net) -> /PE6
- U1 pad J11: (no net) -> /PE5
- U1 pad J14: (no net) -> /OUT_7
- U1 pad J16: (no net) -> /PD0
- U1 pad J18: (no net) -> /PB7
- U1 pad J203: (no net) -> GND
- U1 pad J204: (no net) -> GND
- U1 pad J207: (no net) -> /VDD
- U1 pad J208: (no net) -> /VDD
- U1 pad J209: (no net) -> /5V
- U1 pad J210: (no net) -> /5V
- U1 pad J31: (no net) -> GND
- U1 pad J32: (no net) -> /Vrtc
- U1 pad J51: (no net) -> /IGN_OUT_1
- U1 pad J52: (no net) -> /IGN_OUT_2
- U1 pad J53: (no net) -> /IGN_OUT_3
- U1 pad J54: (no net) -> /IGN_OUT_4
- U1 pad J6: (no net) -> /PE0
- U1 pad J61: (no net) -> /OUT_14
- U1 pad J62: (no net) -> /OUT_15
- U1 pad J63: (no net) -> /OUT_16
- U1 pad J64: (no net) -> /OUT_17
- U1 pad J65: (no net) -> /OUT_18
- U1 pad J802: /12V_KEY -> /12V_MREL
- U1 pad J9: (no net) -> /PC13
Routing:
- net /12V_KEY: track 464.6 -> 5.01 mm
- net /AV6: track 101.0 -> 0.00 mm
- net /12V_MREL: track 0.00 -> 65.0 mm
- net /CAM_SENSOR: track 58.7 -> 0.00 mm
- net /12V_SAFE: track 56.8 -> 0.00 mm
- net /CRNK+: track 54.8 -> 0.00 mm
- net /GP4: track 52.3 -> 0.00 mm, vias 1 -> 0
- net /AT1: track 49.8 -> 0.00 mm
- net /AT4: track 48.6 -> 0.00 mm
- net /INJECTOR-4: track 46.6 -> 0.00 mm
- net /AT2: track 45.8 -> 0.00 mm
- net /Ign3: track 44.0 -> 0.00 mm
- net /Ign2: track 42.9 -> 0.00 mm
- net /E-THROTTLE-: track 42.7 -> 0.00 mm
- net /INJECTOR-3: track 42.6 -> 0.00 mm
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Other:
- board size 106.7 x 124.5 mm -> 129.5 x 127.6 mm
- board text added: "GP4 GP3 GP2 GP1 MRL AV6 AV8 AV9 AV10 IJ1 IJ2 IJ3 IJ4"
- board text added: "microRusEFI text fixture R0.1"
- board text removed: "12V-MREL"
- board text removed: "GP4 GP3 GP2 GP1 AV6 AV8 AV9 AV10 IJ1 IJ2 IJ3 IJ4"
- board text removed: "microRusEFI text fixture 0.1"

Commit message: draft
Parts:
- removed F1: 1A FUSE, rusefi_lib:Blank
- removed the R21 at (44.3, 42.5)
- removed the R30 at (42.5, 45.1)
- added D1: 1N4148WS, rusefi_lib:SM0805_jumper, F.Cu at (149.2, 144.1)
- added D2: GRN, rusefi_lib:SM0805_jumper, F.Cu at (149.2, 137.8)
- added D3: 1N4148WS, rusefi_lib:SM0805_jumper, F.Cu at (146.7, 144.1)
- added D4: GRN, rusefi_lib:SM0805_jumper, F.Cu at (146.7, 137.8)
- added R1: 1k, rusefi_lib:SM0805_jumper, F.Cu at (149.2, 131.4)
- added R2: 1k, rusefi_lib:SM0805_jumper, F.Cu at (146.7, 131.4)
- added R23: 5k, rusefi_lib:SM0805_jumper, F.Cu at (44.3, 47.6)
- added R32: 2k2, rusefi_lib:SM0805_jumper, F.Cu at (42.5, 60.3)
- moved D49 40.2 mm to (57.8, 114.9), turned to 0 degrees
- moved D64 40.2 mm to (57.8, 153.0), turned to 0 degrees
- moved R61 40.2 mm to (45.1, 114.9), turned to 0 degrees
- moved R76 40.2 mm to (45.1, 153.0), turned to 0 degrees
- moved D65 38.1 mm to (51.4, 114.9), turned to 0 degrees
- moved D80 38.1 mm to (51.4, 153.0), turned to 0 degrees
- moved D50 35.4 mm to (57.8, 117.5), turned to 0 degrees
- moved D63 35.4 mm to (57.8, 150.5), turned to 0 degrees
- moved R62 35.4 mm to (45.1, 117.5), turned to 0 degrees
- moved R75 35.4 mm to (45.1, 150.5), turned to 0 degrees
- moved D66 33.0 mm to (51.4, 117.5), turned to 0 degrees
- moved D79 33.0 mm to (51.4, 150.5), turned to 0 degrees
- moved D51 30.7 mm to (57.8, 120.0), turned to 0 degrees
- moved D62 30.7 mm to (57.8, 148.0), turned to 0 degrees
- moved R63 30.7 mm to (45.1, 120.0), turned to 0 degrees
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- renumbered D6 to D10, D7 to D11, D8 to D12, D9 to D13, D10 to D14, D11 to D15, D12 to D16, D13 to D17, D14 to D18, D15 to D19, D16 to D20, D17 to D21, D18 to D22, D19 to D23, D20 to D24, D21 to D25, D22 to D26, D23 to D27, D24 to D28, D25 to D29, D26 to D30, D27 to D31, D28 to D32, D29 to D33, D30 to D34, D31 to D35, D32 to D36, D33 to D37, D34 to D38, D35 to D39, D36 to D40, D37 to D41, D38 to D42, D39 to D43, D40 to D44, D41 to D45, D42 to D46, D43 to D47, D44 to D48, D45 to D49, D1 to D5, D46 to D50, D47 to D51, D48 to D52, D49 to D53, D50 to D54, D51 to D55, D52 to D56, D53 to D57, D54 to D58, D55 to D59, D2 to D6, D56 to D60, D57 to D61, D58 to D62, D59 to D63, D60 to D64, D61 to D65, D62 to D66, D63 to D67, D64 to D68, D65 to D69, D3 to D7, D66 to D70, D67 to D71, D68 to D72, D69 to D73, D70 to D74, D71 to D75, D72 to D76, D73 to D77, D74 to D78, D75 to D79, D4 to D8, D76 to D80, D77 to D81, D78 to D82, D79 to D83, D80 to D84, D81 to D85, D82 to D86, D83 to D87, D84 to D88, D85 to D89, D5 to D9, D86 to D90, D87 to D91, D88 to D92, D89 to D93, D90 to D94, D91 to D95, D92 to D96, D93 to D97, R8 to R10, R9 to R11, R10 to R12, R11 to R13, R12 to R14, R13 to R15, R14 to R16, R15 to R17, R16 to R18, R17 to R19, R18 to R20, R19 to R21, R20 to R22, R22 to R24, R23 to R25, R24 to R26, R25 to R27, R26 to R28, R27 to R29, R1 to R3, R28 to R30, R29 to R31, R31 to R33, R32 to R34, R35 to R37, R36 to R38, R37 to R39, R2 to R4, R38 to R40, R39 to R41, R40 to R42, R41 to R43, R42 to R44, R43 to R45, R44 to R46, R45 to R47, R46 to R48, R47 to R49, R3 to R5, R48 to R50, R49 to R51, R50 to R52, R51 to R53, R52 to R54, R53 to R55, R54 to R56, R55 to R57, R56 to R58, R57 to R59, R4 to R6, R58 to R60, R59 to R61, R60 to R62, R61 to R63, R62 to R64, R63 to R65, R64 to R66, R65 to R67, R66 to R68, R67 to R69, R5 to R7, R68 to R70, R69 to R71, R70 to R72, R71 to R73, R72 to R74, R73 to R75, R74 to R76, R75 to R77, R76 to R78, R77 to R79, R6 to R8, R78 to R80, R79 to R81, R80 to R82, R81 to R83, R82 to R84, R83 to R85, R84 to R86, R85 to R87, R86 to R88, R87 to R89, R7 to R9, R88 to R90, R89 to R91, R90 to R92, R91 to R93
Routing:
- net /12V_MREL: track 65.0 -> 541.7 mm
- net Net-(J1-Pad1): track 14.2 -> 10.6 mm
- net Net-(D70-Pad1): track 0.00 -> 3.18 mm
- net Net-(D69-Pad1): track 0.00 -> 3.18 mm
- net Net-(D68-Pad1): track 0.00 -> 3.18 mm
- net Net-(D67-Pad1): track 0.00 -> 3.18 mm
- net Net-(D66-Pad1): track 0.00 -> 3.18 mm
- net Net-(D65-Pad1): track 0.00 -> 3.18 mm
- net Net-(D83-Pad2): track 0.00 -> 3.17 mm
- net Net-(D81-Pad2): track 0.00 -> 3.17 mm
Other:
- net class 2.5A EXTERNAL removed
- net class 3,5A EXT HIGH VOLTAGE removed
- net class 3.5A EXTERNAL removed
- net class 5A EXTERNAL removed
- net class CUSTOM removed
- net class CUSTOM 0.6 removed
- net class MIN_EXTERN_188A removed
- net class MIN_EXTERN_241A removed
- board text added: "1 2 3 4 5 6"
- board text removed: "1 2 3 4 6 5"

Commit message: draft
Routing:
- net /5V1: track 0.00 -> 145.8 mm, vias 0 -> 1
- net /5V2: track 0.00 -> 136.9 mm, vias 0 -> 3
- net /VDD: track 0.00 -> 117.1 mm, vias 0 -> 1
- net /IGN_OUT_1: track 0.00 -> 115.2 mm, vias 0 -> 2
- net /5V: track 0.00 -> 113.4 mm, vias 0 -> 1
- net /GP4: track 0.00 -> 107.4 mm, vias 0 -> 5
- net /OUT_18: track 0.00 -> 104.5 mm
- net /OUT_7: track 0.00 -> 103.3 mm
- net /OUT_14: track 0.00 -> 102.0 mm
- net /OUT_17: track 0.00 -> 101.8 mm
- net /OUT_15: track 0.00 -> 100.9 mm
- net /OUT_16: track 0.00 -> 100.3 mm
- net /AT2: track 0.00 -> 98.8 mm, vias 0 -> 2
- net /AV1: track 0.00 -> 93.1 mm, vias 0 -> 1
- net /AV3: track 0.00 -> 92.3 mm, vias 0 -> 1
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
Commit message: R0.1
Other:
- board text added: "AT1"
- board text added: "AT2"
- board text added: "AT3"
- board text added: "AT4"
- board text added: "AV1"
- board text added: "AV2"
- board text added: "AV3"
- board text added: "AV4"
- board text added: "AV5"
- board text added: "AV7"
- board text added: "CAM"
- board text added: "CRANK"
- board text added: "IGN_OUT_1"
- board text added: "IGN_OUT_2"
- board text added: "IGN_OUT_3"
- board text added: "IGN_OUT_4"
- board text added: "LS1"
- board text added: "LS2"
- board text added: "OUT14"
- board text added: "OUT15"
- board text added: "OUT16"
- board text added: "OUT17"
- board text added: "OUT18"
- board text added: "OUT7"
- board text added: "PA15"
- board text added: "PB7"
- board text added: "PB8"
- board text added: "PB9"
- board text added: "PC10"
- board text added: "PC11"
- board text added: "PC12"
- board text added: "PC13"
- board text added: "PD0"
- board text added: "PE0"
- board text added: "PE5"
- board text added: "PE6"
- board text added: "VDD 3.3V"
Changed lines of the file:
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@@
   (general
     (thickness 1.6)
-    (drawings 48)
+    (drawings 96)
     (tracks 2042)
     (zones 0)
@@
     (40 Dwgs.User user)
     (41 Cmts.User user)
-    (42 Eco1.User user hide)
+    (42 Eco1.User user)
     (43 Eco2.User user)
     (44 Edge.Cuts user)
@@
       (xy 3.3528 0.39624)) (layer B.SilkS) (width 0.00254))
   )
+  (gr_text 12V (at 64.8335 105.918 90) (layer F.SilkS)
+    (effects (font (size 1.016 1.016) (thickness 0.1524)))
+  )
+  (gr_text IGN_OUT_1 (at 121.031 84.074) (layer F.SilkS)
+    (effects (font (size 0.75 0.75) (thickness 0.13)))
+  )
+  (gr_text IGN_OUT_4 (at 120.904 91.694) (layer F.SilkS)
+    (effects (font (size 0.75 0.75) (thickness 0.13)))
+  )
+  (gr_text IGN_OUT_3 (at 120.904 89.154) (layer F.SilkS)
+    (effects (font (size 0.75 0.75) (thickness 0.13)))
+  )
+  (gr_text IGN_OUT_2 (at 120.904 86.614) (layer F.SilkS)
+    (effects (font (size 0.75 0.75) (thickness 0.13)))
+  )
+  (gr_text OUT18 (at 142.24 108.712) (layer F.SilkS)
+    (effects (font (size 0.75 0.75) (thickness 0.13)))
+  )
+  (gr_text OUT17 (at 142.24 106.045) (layer F.SilkS)
+    (effects (font (size 0.75 0.75) (thickness 0.13)))
+  )
+  (gr_text OUT16 (at 142.24 103.505) (layer F.SilkS)
+    (effects (font (size 0.75 0.75) (thickness 0.13)))
+  )
+  (gr_text OUT15 (at 142.24 100.965) (layer F.SilkS)
+    (effects (font (size 0.75 0.75) (thickness 0.13)))
+  )
+  (gr_text OUT14 (at 142.24 98.425) (layer F.SilkS)
+    (effects (font (size 0.75 0.75) (thickness 0.13)))
+  )
+  (gr_text CRANK (at 157.353 76.2 90) (layer F.SilkS)
+    (effects (font (size 1.27 1.27) (thickness 0.13)))
+  )
+  (gr_text CAM (at 157.353 59.563 90) (layer F.SilkS)
+    (effects (font (size 1.27 1.27) (thickness 0.13)))
+  )
+  (gr_text 12V (at 57.658 49.276) (layer F.SilkS)
+    (effects (font (size 0.75 0.75) (thickness 0.13)))
+  )
+  (gr_text 5V (at 149.225 148.082 90) (layer F.SilkS)
+    (effects (font (size 0.75 0.75) (thickness 0.13)))
+  )
+  (gr_text "VDD 3.3V" (at 146.685 149.987 90) (layer F.SilkS)
+    (effects (font (size 0.75 0.75) (thickness 0.13)))
+  )
+  (gr_text IGN_OUT_4 (at 63.754 153.035) (layer F.SilkS)
+    (effects (font (size 0.75 0.75) (thickness 0.13)))
+  )
+  (gr_text IGN_OUT_3 (at 63.754 150.495) (layer F.SilkS)
+    (effects (font (size 0.75 0.75) (thickness 0.13)))
+  )
+  (gr_text IGN_OUT_2 (at 63.881 147.955) (layer F.SilkS)
+    (effects (font (size 0.75 0.75) (thickness 0.13)))
+  )
+  (gr_text IGN_OUT_1 (at 63.881 145.415) (layer F.SilkS)
+    (effects (font (size 0.75 0.75) (thickness 0.13)))
+  )
+  (gr_text PE5 (at 62.103 142.875) (layer F.SilkS)
+    (effects (font (size 0.75 0.75) (thickness 0.13)))
+  )
+  (gr_text PE6 (at 62.103 140.335) (layer F.SilkS)
+    (effects (font (size 0.75 0.75) (thickness 0.13)))
+  )
+  (gr_text PE0 (at 62.103 137.795) (layer F.SilkS)
+    (effects (font (size 0.75 0.75) (thickness 0.13)))
+  )
+  (gr_text PD0 (at 61.849 135.382) (layer F.SilkS)
+    (effects (font (size 0.75 0.75) (thickness 0.13)))
+  )
+  (gr_text PC13 (at 62.23 132.842) (layer F.SilkS)
+    (effects (font (size 0.75 0.75) (thickness 0.13)))
+  )
+  (gr_text PC12 (at 62.357 130.175) (layer F.SilkS)
+    (effects (font (size 0.75 0.75) (thickness 0.13)))
+  )
+  (gr_text PC11 (at 62.357 127.762) (layer F.SilkS)
+    (effects (font (size 0.75 0.75) (thickness 0.13)))
+  )
+  (gr_text PC10 (at 62.357 125.095) (layer F.SilkS)
+    (effects (font (size 0.75 0.75) (thickness 0.13)))
+  )
+  (gr_text PB9 (at 61.976 122.555) (layer F.SilkS)
+    (effects (font (size 0.75 0.75) (thickness 0.13)))
+  )
+  (gr_text PB8 (at 61.849 120.142) (layer F.SilkS)
+    (effects (font (size 0.75 0.75) (thickness 0.13)))
+  )
+  (gr_text PB7 (at 61.976 117.602) (layer F.SilkS)
+    (effects (font (size 0.75 0.75) (thickness 0.13)))
+  )
+  (gr_text PA15 (at 62.23 115.062) (layer F.SilkS)
+    (effects (font (size 0.75 0.75) (thickness 0.13)))
+  )
+  (gr_text LS2 (at 51.054 109.855) (layer F.SilkS)
+    (effects (font (size 0.75 0.75) (thickness 0.13)))
+  )
+  (gr_text LS1 (at 51.054 104.902) (layer F.SilkS)
+    (effects (font (size 0.75 0.75) (thickness 0.13)))
+  )
+  (gr_text OUT18 (at 51.435 99.695) (layer F.SilkS)
+    (effects (font (size 0.75 0.75) (thickness 0.13)))
+  )
+  (gr_text OUT17 (at 51.435 94.615) (layer F.SilkS)
+    (effects (font (size 0.75 0.75) (thickness 0.13)))
+  )
+  (gr_text OUT16 (at 51.435 89.535) (layer F.SilkS)
+    (effects (font (size 0.75 0.75) (thickness 0.13)))
+  )
+  (gr_text OUT15 (at 51.435 84.582) (layer F.SilkS)
+    (effects (font (size 0.75 0.75) (thickness 0.13)))
+  )
+  (gr_text OUT14 (at 51.435 79.502) (layer F.SilkS)
+    (effects (font (size 0.75 0.75) (thickness 0.13)))
+  )
+  (gr_text OUT7 (at 51.181 74.295) (layer F.SilkS)
+    (effects (font (size 0.75 0.75) (thickness 0.13)))
+  )
+  (gr_text AV7 (at 46.736 66.294) (layer F.SilkS)
+    (effects (font (size 0.75 0.75) (thickness 0.13)))
+  )
+  (gr_text AV5 (at 46.736 61.087) (layer F.SilkS)
+    (effects (font (size 0.75 0.75) (thickness 0.13)))
+  )
+  (gr_text AV4 (at 46.736 56.007) (layer F.SilkS)
+    (effects (font (size 0.75 0.75) (thickness 0.13)))
+  )
+  (gr_text AV3 (at 46.736 51.054) (layer F.SilkS)
+    (effects (font (size 0.75 0.75) (thickness 0.13)))
+  )
+  (gr_text AV2 (at 46.736 45.847) (layer F.SilkS)
+    (effects (font (size 0.75 0.75) (thickness 0.13)))
+  )
+  (gr_text AV1 (at 46.736 40.767) (layer F.SilkS)
+    (effects (font (size 0.75 0.75) (thickness 0.13)))
+  )
+  (gr_text AT4 (at 46.482 37.465) (layer F.SilkS)
+    (effects (font (size 0.75 0.75) (thickness 0.13)))
+  )
+  (gr_text AT3 (at 46.482 35.052) (layer F.SilkS)
+    (effects (font (size 0.75 0.75) (thickness 0.13)))
+  )
+  (gr_text AT2 (at 46.482 32.385) (layer F.SilkS)
+    (effects (font (size 0.75 0.75) (thickness 0.13)))
+  )
+  (gr_text AT1 (at 46.482 29.972) (layer F.SilkS)
+    (effects (font (size 0.75 0.75) (thickness 0.13)))
+  )
   (gr_text "1 2  3 4  5 6" (at 60.325 49.53) (layer F.SilkS)
     (effects (font (size 1.5 1.5) (thickness 0.13)) (justify left))
@@
     (effects (font (size 0.75 0.75) (thickness 0.13)))
   )
-  (gr_text GND (at 135.382 140.462) (layer F.SilkS)
-    (effects (font (size 0.75 0.75) (thickness 0.13)))
-  )
