File: zMRETestFixture.sch (KiCad schematic (older format))
At the start: 103 parts, among them J11 Conn_01x01, J12 Conn_01x01, J13 Conn_02x05_Counter_Clockwise, J14 Conn_01x01, J15 Conn_01x01, SW11 SW_Push, SW12 SW_Push, U11 molex_48pin_MRE

Commit message: draft
Parts:
- added D2, D4, D6: 1N4148WS, rusefi_lib:SM0805_jumper, symbol Device:D
- added D3: GRN, LED_SMD:LED_0805_2012Metric, symbol Device:LED
- added D5: YEL(593NM), LED_SMD:LED_0805_2012Metric, symbol Device:LED
- added D7: YEL(570NM), LED_SMD:LED_0805_2012Metric, symbol Device:LED
- added J5, J6: Conn_01x01, Connector_Pin:Pin_D0.7mm_L6.5mm_W1.8mm_FlatFork, symbol Connector_Generic:Conn_01x01
- added R2, R3, R4, R53, R54: 5k, rusefi_lib:SM0805_jumper, symbol Device:R
- renumbered D11 to D1, D14 to D10, D15 to D11, D16 to D12, D17 to D13, D18 to D14, D19 to D15, D20 to D16, D21 to D17, D22 to D18, D23 to D19, D24 to D20, D25 to D21, D26 to D22, D27 to D23, D28 to D24, D29 to D25, D30 to D26, D31 to D27, D32 to D28, D33 to D29, D34 to D30, D35 to D31, D36 to D32, D37 to D33, D38 to D34, D39 to D35, D40 to D36, D41 to D37, D42 to D38, D43 to D39, D44 to D40, D45 to D41, D46 to D42, D47 to D43, D12 to D8, D13 to D9, J11 to J1, J12 to J2, J14 to J3, J15 to J4, J13 to J7, LOGO11 to LOGO1, LOGO12 to LOGO2, LOGO13 to LOGO3, R11 to R1, R23 to R10, R26 to R11, R29 to R12, R32 to R13, R35 to R14, R18 to R17, R19 to R18, R21 to R19, R22 to R20, R24 to R21, R25 to R22, R27 to R23, R28 to R24, R30 to R25, R31 to R26, R33 to R27, R34 to R28, R36 to R29, R37 to R30, R38 to R31, R39 to R32, R41 to R33, R42 to R34, R40 to R35, R44 to R36, R45 to R37, R43 to R38, R46 to R39, R47 to R40, R48 to R41, R49 to R42, R50 to R43, R51 to R44, R52 to R45, R53 to R46, R54 to R47, R55 to R48, R56 to R49, R12 to R5, R57 to R50, R58 to R51, R59 to R52, R13 to R6, R14 to R7, R17 to R8, R20 to R9, SW11 to SW1, SW12 to SW2, TP11 to TP1, TP12 to TP2, TP13 to TP3, TP14 to TP4, TP15 to TP5, TP16 to TP6, U11 to U1
Connections:
- net 12V_KEY: now also D2.2 (A)
- net 5V1: now also R53.2
- net 5V2: now also R54.2
- net CAM_SENSOR: now also SW1.1, J5.1 (Pin_1), R53.1
- net CRNK+: now also J3.1 (Pin_1)
- net CRNK-: now also J4.1 (Pin_1)
- net E-THROTTLE+: now also D4.2 (A), D6.1 (K)
- net E-THROTTLE-: now also R3.2, R4.2
- net GND: now also SW1.2, SW2.2, R2.2
- net ????: now reaches SW2.1
- net ????: now also J6.1 (Pin_1), R54.1
- new net: D3.1 (K), R2.1
- new net: D2.1 (K), D3.2 (A)
- new net: D5.1 (K), R3.1
- new net: D4.1 (K), D5.2 (A)
- new net: D6.2 (A), D7.1 (K)
- new net: D7.2 (A), R4.1
Other:
- moved on the sheet: J3, J4, SW1, SW2

Commit message: draft
Parts:
- D11, D13, D15, D17, D19, D21, D23, D25, D27, D3, D5, D7, D9: footprint LED_SMD:LED_0805_2012Metric -> rusefi_lib:SM0805_jumper
Changed lines of the file:
@@
 F 0 "D9" H 4300 3375 50  0000 C CNN
 F 1 "BLU" H 4375 3475 50  0000 R CNN
-F 2 "LED_SMD:LED_0805_2012Metric" H 4150 3425 50  0001 C CNN
+F 2 "rusefi_lib:SM0805_jumper" H 4150 3425 50  0001 C CNN
 F 3 "~" H 4150 3425 50  0001 C CNN
 F 4 "C375453" H 4150 3425 50  0001 C CNN "LCSC"
@@
 F 0 "D11" H 4500 3375 50  0000 C CNN
 F 1 "BLU" H 4575 3475 50  0000 R CNN
-F 2 "LED_SMD:LED_0805_2012Metric" H 4350 3425 50  0001 C CNN
+F 2 "rusefi_lib:SM0805_jumper" H 4350 3425 50  0001 C CNN
 F 3 "~" H 4350 3425 50  0001 C CNN
 F 4 "C375453" H 4350 3425 50  0001 C CNN "LCSC"
@@
 F 0 "D13" H 4700 3375 50  0000 C CNN
 F 1 "BLU" H 4775 3475 50  0000 R CNN
-F 2 "LED_SMD:LED_0805_2012Metric" H 4550 3425 50  0001 C CNN
+F 2 "rusefi_lib:SM0805_jumper" H 4550 3425 50  0001 C CNN
 F 3 "~" H 4550 3425 50  0001 C CNN
 F 4 "C375453" H 4550 3425 50  0001 C CNN "LCSC"
@@
 F 0 "D15" H 4900 3375 50  0000 C CNN
 F 1 "BLU" H 4975 3475 50  0000 R CNN
-F 2 "LED_SMD:LED_0805_2012Metric" H 4750 3425 50  0001 C CNN
+F 2 "rusefi_lib:SM0805_jumper" H 4750 3425 50  0001 C CNN
 F 3 "~" H 4750 3425 50  0001 C CNN
 F 4 "C375453" H 4750 3425 50  0001 C CNN "LCSC"
@@
 F 0 "D17" H 5100 3375 50  0000 C CNN
 F 1 "BLU" H 5175 3475 50  0000 R CNN
-F 2 "LED_SMD:LED_0805_2012Metric" H 4950 3425 50  0001 C CNN
+F 2 "rusefi_lib:SM0805_jumper" H 4950 3425 50  0001 C CNN
 F 3 "~" H 4950 3425 50  0001 C CNN
 F 4 "C375453" H 4950 3425 50  0001 C CNN "LCSC"
@@
 F 0 "D19" H 5300 3375 50  0000 C CNN
 F 1 "BLU" H 5375 3475 50  0000 R CNN
-F 2 "LED_SMD:LED_0805_2012Metric" H 5150 3425 50  0001 C CNN
+F 2 "rusefi_lib:SM0805_jumper" H 5150 3425 50  0001 C CNN
 F 3 "~" H 5150 3425 50  0001 C CNN
 F 4 "C375453" H 5150 3425 50  0001 C CNN "LCSC"
@@
 F 0 "D21" H 5500 3375 50  0000 C CNN
 F 1 "BLU" H 5575 3475 50  0000 R CNN
-F 2 "LED_SMD:LED_0805_2012Metric" H 5350 3425 50  0001 C CNN
+F 2 "rusefi_lib:SM0805_jumper" H 5350 3425 50  0001 C CNN
 F 3 "~" H 5350 3425 50  0001 C CNN
 F 4 "C375453" H 5350 3425 50  0001 C CNN "LCSC"
@@
 F 0 "D23" H 5675 3375 50  0000 C CNN
 F 1 "BLU" H 5750 3475 50  0000 R CNN
-F 2 "LED_SMD:LED_0805_2012Metric" H 5525 3425 50  0001 C CNN
+F 2 "rusefi_lib:SM0805_jumper" H 5525 3425 50  0001 C CNN
 F 3 "~" H 5525 3425 50  0001 C CNN
 F 4 "C375453" H 5525 3425 50  0001 C CNN "LCSC"
@@
 F 0 "D25" H 5850 3375 50  0000 C CNN
 F 1 "BLU" H 5925 3475 50  0000 R CNN
-F 2 "LED_SMD:LED_0805_2012Metric" H 5700 3425 50  0001 C CNN
+F 2 "rusefi_lib:SM0805_jumper" H 5700 3425 50  0001 C CNN
 F 3 "~" H 5700 3425 50  0001 C CNN
 F 4 "C375453" H 5700 3425 50  0001 C CNN "LCSC"
@@
 F 0 "D27" H 6025 3375 50  0000 C CNN
 F 1 "BLU" H 6100 3475 50  0000 R CNN
-F 2 "LED_SMD:LED_0805_2012Metric" H 5875 3425 50  0001 C CNN
+F 2 "rusefi_lib:SM0805_jumper" H 5875 3425 50  0001 C CNN
 F 3 "~" H 5875 3425 50  0001 C CNN
 F 4 "C375453" H 5875 3425 50  0001 C CNN "LCSC"
@@
 F 0 "D3" H 2100 2275 50  0000 C CNN
 F 1 "GRN" H 2175 2375 50  0000 R CNN
-F 2 "LED_SMD:LED_0805_2012Metric" H 1950 2325 50  0001 C CNN
+F 2 "rusefi_lib:SM0805_jumper" H 1950 2325 50  0001 C CNN
 F 3 "~" H 1950 2325 50  0001 C CNN
 F 4 "C2297" H 1950 2325 50  0001 C CNN "LCSC"
@@
 F 0 "D5" H 2925 2275 50  0000 C CNN
 F 1 "YEL(593NM)" H 3100 2425 50  0000 R CNN
-F 2 "LED_SMD:LED_0805_2012Metric" H 2775 2325 50  0001 C CNN
+F 2 "rusefi_lib:SM0805_jumper" H 2775 2325 50  0001 C CNN
 F 3 "~" H 2775 2325 50  0001 C CNN
 F 4 "C2296" H 2775 2325 50  0001 C CNN "LCSC"
@@
 F 0 "D7" H 3200 2275 50  0000 C CNN
 F 1 "YEL(570NM)" H 3175 2450 50  0000 R CNN
-F 2 "LED_SMD:LED_0805_2012Metric" H 3050 2325 50  0001 C CNN
+F 2 "rusefi_lib:SM0805_jumper" H 3050 2325 50  0001 C CNN
 F 3 "~" H 3050 2325 50  0001 C CNN
 F 4 "C84257" H 3050 2325 50  0001 C CNN "LCSC"

Commit message: draft
Parts:
- removed R25: 5k, rusefi_lib:SM0805_jumper, symbol Device:R
- removed R26: 1k, rusefi_lib:SM0805_jumper, symbol Device:R
- renumbered R29 to R15, R30 to R16, R31 to R17, R32 to R18, R33 to R19, R34 to R20, R36 to R21, R37 to R22, R15 to R23, R16 to R24, R17 to R25, R18 to R26, R19 to R27, R20 to R28, R21 to R29, R22 to R30, R23 to R31, R24 to R32, R27 to R36, R28 to R37
Connections:
- net 5V1: now also R54.2; no longer R53.2
- net 5V2: now also R53.2; no longer R54.2
- net GP1: now also D16.2 (A); no longer D20.2 (A)
- net GP2: now also D18.2 (A); no longer D22.2 (A)
- net GP3: now also D20.2 (A); no longer D24.2 (A)
- net GP4: now also D22.2 (A); no longer D26.2 (A)
- net GP5: now also D24.2 (A); no longer D18.2 (A), U1.14
- net GP6: now also D26.2 (A); no longer D16.2 (A), U1.13
Other:
- moved on the sheet: R15, R16, R17, R18, R19, R20, R21, R22, R23, R24, R25, R26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

Commit message: draft
Parts:
- removed TP3, TP4: TP, TestPoint:TestPoint_Pad_D2.0mm, symbol Connector:TestPoint
Connections:
- net ????: no longer names the net of J6.1 (Pin_1), R54.1, SW2.1
Changed lines of the file:
@@
 AV10
-$Comp
-L Connector:TestPoint TP4
-U 1 1 5D358BCF
-P 16000 1050
-F 0 "TP4" V 16000 1225 50  0000 L CNN
-F 1 "TP" H 15950 1275 50  0001 L CNN
-F 2 "TestPoint:TestPoint_Pad_D2.0mm" H 16200 1050 50  0001 C CNN
-F 3 "~" H 16200 1050 50  0001 C CNN
-F 4 "DNP" H 7875 -4425 50  0001 C CNN "Part #"
-F 5 "DNP" H 7875 -4425 50  0001 C CNN "VEND"
-F 6 "DNP" H 7875 -4425 50  0001 C CNN "VEND#"
-F 7 "DNP" H 7875 -4425 50  0001 C CNN "Manufacturer"
-	1    16000 1050
-	0    1    1    0
-$EndComp
-$Comp
-L Connector:TestPoint TP3
-U 1 1 5D08B37F
-P 16000 925
-F 0 "TP3" V 16000 1100 50  0000 L CNN
-F 1 "TP" H 16058 952 50  0001 L CNN
-F 2 "TestPoint:TestPoint_Pad_D2.0mm" H 16200 925 50  0001 C CNN
-F 3 "~" H 16200 925 50  0001 C CNN
-F 4 "DNP" H 9850 -4000 50  0001 C CNN "Part #"
-F 5 "DNP" H 9850 -4000 50  0001 C CNN "VEND"
-F 6 "DNP" H 9850 -4000 50  0001 C CNN "VEND#"
-F 7 "DNP" H 9850 -4000 50  0001 C CNN "Manufacturer"
-	1    16000 925
-	0    1    1    0
-$EndComp
 $Comp
 L Device:LED D9
@@
 	1    0    0    -1
 $EndComp
-Text Label 16000 1050 2    60   ~ 12
-CRANK
 Text Label 16000 675  2    60   ~ 12
 5V
 Text Label 16000 800  2    60   ~ 12
 GND
-Text Label 16000 925  2    60   ~ 12
-CAM_MCU
 $Comp
 L Connector:TestPoint TP5
@@
 Wire Wire Line
 	3050 1875 3050 1775
-Text Label 11275 2350 0    50   ~ 0
-????
 $Comp
 L Connector_Generic:Conn_01x01 J6

Commit message: draft
Parts:
- added F1: 1A FUSE, rusefi_lib:Blank, symbol Device:Fuse
- added J8, J9: Conn_01x01_Female, rusefi_lib:KeyStone_3557, symbol Connector:Conn_01x01_Female
- added R53: 5k, rusefi_lib:SM0805_jumper, symbol Device:R
- added R56: 470k, rusefi_lib:SM0805_jumper, symbol Device:R
- R55: renamed from R53; value 5k -> 470k; LCSC C17677 -> C17709
- renumbered TP5 to TP3, TP6 to TP4
Connections:
- wire segments 153 -> 152
- no-connect marks 14 -> 16
Other:
- moved on the sheet: D2, D3, J1, J2, J5, J6, R2, R55, SW1, SW2

Commit message: Draft
Parts:
- removed D16, D18, D20, D22: 1N4148WS, rusefi_lib:SM0805_jumper, symbol Device:D
- removed D17, D19, D21, D23: BLU, rusefi_lib:SM0805_jumper, symbol Device:LED
- removed R10, R11, R12, R9: 1k, rusefi_lib:SM0805_jumper, symbol Device:R
- added D20, D22, D24, D26: RED, rusefi_lib:SM0805_jumper, symbol Device:LED
- added D21, D23, D25, D27, D44: 1N4148WS, rusefi_lib:SM0805_jumper, symbol Device:D
- added D45: GRN, rusefi_lib:SM0805_jumper, symbol Device:LED
- added R17, R23, R29, R35, R61: 1k, rusefi_lib:SM0805_jumper, symbol Device:R
- added R18, R24, R30, R36: 5k, rusefi_lib:SM0805_jumper, symbol Device:R
- renumbered D24 to D16, D25 to D17, D26 to D18, D27 to D19, J8 to J3, J9 to J4, J3 to J5, J4 to J6, J5 to J7, J6 to J8, J7 to J9, R14 to R10, R15 to R11, R16 to R12, R17 to R13, R18 to R14, R19 to R15, R20 to R16, R21 to R19, R22 to R20, R23 to R21, R24 to R22, R29 to R31, R30 to R32, R31 to R33, R32 to R34, R35 to R39, R36 to R40, R37 to R41, R38 to R42, R39 to R43, R40 to R44, R41 to R45, R42 to R46, R43 to R47, R44 to R48, R45 to R49, R46 to R50, R47 to R51, R48 to R52, R49 to R53, R50 to R54, R51 to R55, R52 to R56, R53 to R57, R54 to R58, R55 to R59, R56 to R60, R13 to R9
Connections:
- wire segments 152 -> 182
Other:
- moved on the sheet: D16, D17, D18, D19, R10, R9

Commit message: Draft
Parts:
- removed R11, R13, R15, R19, R31, R33: 5k, rusefi_lib:SM0805_jumper, symbol Device:R
- added R16, R22: 10k, rusefi_lib:SM0805_jumper, symbol Device:R
- R13: renamed from R14; value 1k -> 2k2; LCSC C17513 -> C17520
- R14: renamed from R16; value 1k -> 3k3; LCSC C17513 -> C26010
- R15: renamed from R20; value 1k -> 4k7; LCSC C17513 -> C17673
- R17: renamed from R32; value 1k -> 220R; LCSC C17513 -> C17557
- R21: renamed from R22; value 1k -> 220R; LCSC C17513 -> C17557
- R23: renamed from R34; value 1k -> 470R; LCSC C17513 -> C17710
- R27: renamed from R26; value 1k -> 470R; LCSC C17513 -> C17710
- R28: renamed from R40; value 5k -> 10k; LCSC C17677 -> C17414
- renumbered D44 to D20, D45 to D21, D20 to D44, D21 to D45, R61 to R11, R23 to R18, R24 to R19, R21 to R20, R29 to R24, R30 to R25, R25 to R26, R41 to R29, R35 to R30, R36 to R31, R39 to R34, R27 to R35, R28 to R36, R42 to R37, R43 to R38, R44 to R39, R45 to R40, R46 to R41, R47 to R42, R48 to R43, R49 to R44, R50 to R45, R51 to R46, R52 to R47, R53 to R48, R54 to R49, R55 to R50, R56 to R51, R17 to R52, R18 to R53, R57 to R54, R58 to R55, R59 to R56, R60 to R57
Connections:
- wire segments 182 -> 179
Other:
- note added: "0.258V"
- note added: "0.506V"
- note added: "0.537V"
- note added: "1.031V"
- note added: "1.091V"
- note added: "2.000V"
- moved on the sheet: R17, R20, R21, R23, R26, R27, R28, R29, R35, R36

Commit message: DRAFT
Parts:
- removed R17, R21: 220R, rusefi_lib:SM0805_jumper, symbol Device:R
- removed R23, R27: 470R, rusefi_lib:SM0805_jumper, symbol Device:R
- removed R29, R36: 1k, rusefi_lib:SM0805_jumper, symbol Device:R
- added D45, D46, D47, D48, D49, D50, D51, D52, D53, D54, D55, D56, D57, D58, D59, D60, D78, D80, D82, D84, D86, D88, D90, D93: 1N4148WS, rusefi_lib:SM0805_jumper, symbol Device:D
- added D61, D62, D63, D64, D65, D66, D67, D68, D69, D70, D71, D72, D73, D74, D75, D76: GRN, rusefi_lib:SM0805_jumper, symbol Device:LED
- added D77, D79, D81, D83, D85, D87, D89, D92: RED, rusefi_lib:SM0805_jumper, symbol Device:LED
- added J10, J11: Conn_01x01, Connector_Pin:Pin_D0.7mm_L6.5mm_W1.8mm_FlatFork, symbol Connector_Generic:Conn_01x01
- added R16, R20, R57, R58, R59, R60, R61, R62, R63, R64, R65, R66, R67, R68, R69, R70, R71, R72, R73, R75, R77, R79, R81, R83, R85, R88: 1k, rusefi_lib:SM0805_jumper, symbol Device:R
- added R22, R28: 2k2, rusefi_lib:SM0805_jumper, symbol Device:R
- added R26: 3k3, rusefi_lib:SM0805_jumper, symbol Device:R
- added R35: 4k7, rusefi_lib:SM0805_jumper, symbol Device:R
- added R74, R76, R78, R80, R82, R84, R87, R89: 5k, rusefi_lib:SM0805_jumper, symbol Device:R
- added unit 2 of U1
- added unit 3 of U1
- added unit 7 of U1
- added unit 8 of U1
- added unit 14 of U1
- added unit 6 of U1
- renumbered D2 to D1, D11 to D10, D12 to D11, D13 to D12, D14 to D13, D15 to D14, D16 to D15, D17 to D16, D18 to D17, D19 to D18, D20 to D19, D3 to D2, D21 to D20, D22 to D21, D23 to D22, D24 to D23, D25 to D24, D26 to D25, D27 to D26, D28 to D27, D29 to D28, D30 to D29, D4 to D3, D31 to D30, D32 to D31, D33 to D32, D34 to D33, D35 to D34, D36 to D35, D37 to D36, D38 to D37, D39 to D38, D40 to D39, D5 to D4, D41 to D40, D42 to D41, D43 to D42, D44 to D43, D45 to D44, D6 to D5, D7 to D6, D8 to D7, D9 to D8, D10 to D9, D1 to D91, R2 to R1, R11 to R10, R12 to R11, R13 to R12, R14 to R13, R15 to R14, R16 to R15, R18 to R17, R19 to R18, R20 to R19, R3 to R2, R22 to R21, R24 to R23, R25 to R24, R28 to R25, R26 to R27, R30 to R29, R4 to R3, R31 to R30, R34 to R33, R35 to R34, R37 to R36, R38 to R37, R39 to R38, R40 to R39, R5 to R4, R41 to R40, R42 to R41, R43 to R42, R44 to R43, R45 to R44, R46 to R45, R47 to R46, R48 to R47, R49 to R48, R50 to R49, R6 to R5, R51 to R50, R52 to R51, R53 to R52, R54 to R53, R55 to R54, R56 to R55, R57 to R56, R7 to R6, R8 to R7, R9 to R8, R1 to R86, R10 to R9
Connections:
- net labels added: IGN_OUT_1, IGN_OUT_2, IGN_OUT_3, IGN_OUT_4, NRST, OUT_14, OUT_15, OUT_16, OUT_17, OUT_18, OUT_7, PB7, PC13, PD0, PE0, PE5, PE6, SCK, SWDIO, SWO, Vrtc
- wire segments 179 -> 294
- no-connect marks 16 -> 20
Other:
- note added: "0.455V"
- note added: "0.833V"
- note added: "0.902V"
- note added: "1.241V"
- note added: "1.351V"
- note added: "1.528V"
- note added: "2.245V"
- note added: "2.423V"
- note added: "2.750V"
- note added: "3.176V"
- note removed: "0.258V"
- note removed: "0.506V"
- note removed: "0.537V"
- note removed: "1.031V"
- note removed: "1.091V"
- note removed: "2.000V"
- moved on the sheet: D91, R25, R27, R86, U1D, U1E, U1I, U1J, U1K, U1L, U1M
