File: TLE8888-1QK.kicad_sch (KiCad schematic)
At the start: 40 parts, among them J15 Conn_01x01, J17 Conn_01x01, Q1 IPD30N06S2L-23, U2 TLE8888QK

Commit message: 0.6.1 #171 #223
Parts:
- R15: value 15k -> DNP; LCSC DNP -> (none); Manufacturer StackPole -> DNP; Part # RMCF0603JG15K0 -> DNP; VEND# RMCF0603JG15K0CT-ND -> DNP
