File: hi-lo.kicad_sch (KiCad schematic)
At the start: 14 parts, among them U31 MIC4427, U32 MIC4427, U33 MIC4427

Commit message: KiCAD6 version
Parts:
- added D45: SS54, Diode_SMD:D_SMA, symbol Diode:B340
Connections:
- net 5V: now also D45.2 (A); no longer JP2.1 (A)
- new net: D45.1 (K), JP2.1 (A)
Changed lines of the file:
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@@
   (title_block
     (title "microRusEFI-2L")
-    (date "2020-05-24")
-    (rev "R0.5.2")
+    (date "2022-04-10")
+    (rev "R0.6.1RC")
     (company "rusEFI.com")
     (comment 1 "Donald Becker")
     (comment 2 "AI6OD")
+    (comment 3 "by JRD McLAREN")
   )
   (junction (at 116.84 162.56) (diameter 0) (color 0 0 0 0)
@@
     (stroke (width 0) (type default) (color 0 0 0 0))
   )
-  (wire (pts (xy 83.185 121.92) (xy 85.09 121.92))
-    (stroke (width 0) (type default) (color 0 0 0 0))
-  )
   (wire (pts (xy 138.43 135.89) (xy 146.05 135.89))
     (stroke (width 0) (type default) (color 0 0 0 0))
@@
     (effects (font (size 1.524 1.524) (thickness 0.3048) bold) (justify left))
   )
-  (hierarchical_label "5V" (shape input) (at 83.185 121.92 180)
+  (hierarchical_label "5V" (shape input) (at 77.47 121.92 180)
     (effects (font (size 1.524 1.524) (thickness 0.3048) bold) (justify right))
   )
@@
     (pin "1")
   )
+  (symbol (lib_id "Diode:B340") (at 81.28 121.92 180) (unit 1)
+    (in_bom yes) (on_board yes)
+    (property "Reference" "D45" (id 0) (at 77.47 124.46 0))
+    (property "Value" "SS54" (id 1) (at 82.55 124.46 0))
+    (property "Footprint" "Diode_SMD:D_SMA" (id 2) (at 81.28 117.475 0)
+      (effects (font (size 1.27 1.27)) hide)
+    )
+    (property "Datasheet" "http://www.jameco.com/Jameco/Products/ProdDS/1538777.pdf" (id 3) (at 81.28 121.92 0)
+      (effects (font (size 1.27 1.27)) hide)
+    )
+    (property "LCSC" "C22452" (id 4) (at 81.28 121.92 0)
+      (effects (font (size 1.27 1.27)) hide)
+    )
+    (pin "1")
+    (pin "2")
+  )
 )
