File: stm32.kicad_sch (KiCad schematic)
At the start: 47 parts, among them J1 USB_B_Micro, J19 Conn_01x06, J2 Conn_02x05_Odd_Even, J7 TC2030, SW1 SW_Push, SW2 SW_Push, SW3 SW_Push, SW4 SW_Push, U1 STM32F427VGT6, U3 molex_48pin_MRE, U5 LM1117-3.3, X1 8MHz 20pF, Y2 32768 Hz

Commit message: KiCAD6 version
Parts:
- C39: value 22uF -> 22uF 25V; footprint Capacitor_SMD:C_0603_1608Metric -> Capacitor_SMD:C_0805_2012Metric
- D14: footprint Capacitor_SMD:C_0805_2012Metric -> LED_SMD:LED_0603_1608Metric
- U3: footprint (none) -> rusefi_lib:Molex_48_MRE_R055
Changed lines of the file:
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@@
   (title_block
     (title "microRusEFI-2L")
-    (date "2020-05-24")
-    (rev "R0.5.2")
+    (date "2022-04-10")
+    (rev "R0.6.1RC")
     (company "rusEFI.com")
     (comment 1 "Donald Becker")
     (comment 2 "AI6OD")
+    (comment 3 "by JRD McLAREN")
   )
   (junction (at 123.19 142.24) (diameter 0) (color 0 0 0 0)
@@
     (property "Reference" "D14" (id 0) (at 308.61 99.06 0))
     (property "Value" "LED-GREEN" (id 1) (at 308.61 92.71 0))
-    (property "Footprint" "Capacitor_SMD:C_0805_2012Metric" (id 2) (at 617.093 43.18 90)
+    (property "Footprint" "LED_SMD:LED_0603_1608Metric" (id 2) (at 617.093 43.18 90)
       (effects (font (size 1.524 1.524)) hide)
     )
@@
     (in_bom yes) (on_board yes)
     (property "Reference" "C39" (id 0) (at 392.43 71.12 0))
-    (property "Value" "22uF" (id 1) (at 392.43 76.2 0))
-    (property "Footprint" "Capacitor_SMD:C_0603_1608Metric" (id 2) (at 303.022 40.64 90)
+    (property "Value" "22uF 25V" (id 1) (at 392.43 76.2 0))
+    (property "Footprint" "Capacitor_SMD:C_0805_2012Metric" (id 2) (at 303.022 40.64 90)
       (effects (font (size 1.524 1.524)) hide)
     )
@@
       (effects (font (size 1.524 1.524)) (justify left) hide)
     )
-    (property "Footprint" "" (id 2) (at 140.97 78.105 0)
+    (property "Footprint" "rusefi_lib:Molex_48_MRE_R055" (id 2) (at 140.97 78.105 0)
       (effects (font (size 1.524 1.524)) hide)
     )
@@
       (effects (font (size 1.524 1.524)) hide)
     )
+    (pin "1")
+    (pin "10")
+    (pin "11")
+    (pin "12")
+    (pin "13")
+    (pin "14")
+    (pin "15")
+    (pin "16")
+    (pin "17")
+    (pin "18")
+    (pin "19")
+    (pin "2")
+    (pin "20")
+    (pin "21")
+    (pin "22")
+    (pin "23")
+    (pin "24")
+    (pin "25")
+    (pin "26")
+    (pin "27")
+    (pin "28")
+    (pin "29")
+    (pin "3")
+    (pin "30")
+    (pin "31")
+    (pin "32")
+    (pin "33")
+    (pin "34")
+    (pin "35")
+    (pin "36")
+    (pin "37")
+    (pin "38")
+    (pin "39")
+    (pin "4")
+    (pin "40")
+    (pin "41")
+    (pin "42")
+    (pin "43")
+    (pin "44")
+    (pin "45")
+    (pin "46")
+    (pin "47")
+    (pin "48")
+    (pin "5")
+    (pin "6")
+    (pin "7")
+    (pin "8")
+    (pin "9")
+    (pin "M11")
+    (pin "M12")
+    (pin "M13")
+    (pin "M21")
+    (pin "M22")
+    (pin "M23")
+    (pin "M3")
+    (pin "M4")
+    (pin "M51")
+    (pin "M52")
+    (pin "M53")
+    (pin "M61")
+    (pin "M62")
+    (pin "M63")
+    (pin "M71")
+    (pin "M72")
+    (pin "M73")
+    (pin "J61")
+    (pin "J62")
+    (pin "J63")
+    (pin "J64")
+    (pin "J65")
     (pin "J31")
     (pin "J32")
-  )
-  (symbol (lib_id "rusefi_Molex_MRE_Connector:molex_48pin_MRE") (at 323.85 165.1 180) (unit 7)
-    (in_bom yes) (on_board yes)
-    (property "Reference" "U3" (id 0) (at 300.99 156.4386 0)
-      (effects (font (size 1.524 1.524)))
-    )
-    (property "Value" "molex_48pin_MRE" (id 1) (at 293.37 165.1 90)
-      (effects (font (size 1.524 1.524)) hide)
-    )
-    (property "Footprint" "" (id 2) (at 323.85 165.1 0)
-      (effects (font (size 1.524 1.524)) hide)
-    )
-    (property "Datasheet" "" (id 3) (at 323.85 165.1 0)
-      (effects (font (size 1.524 1.524)) hide)
-    )
+    (pin "J801")
+    (pin "J802")
+    (pin "J803")
+    (pin "J804")
+    (pin "J805")
+    (pin "J806")
+    (pin "J807")
+    (pin "J808")
+    (pin "J809")
+    (pin "J810")
+    (pin "LIN1")
+    (pin "J51")
+    (pin "J52")
+    (pin "J53")
+    (pin "J54")
     (pin "J201")
     (pin "J202")
@@
     (pin "J209")
     (pin "J210")
+    (pin "J6")
+    (pin "J18")
+    (pin "J9")
+    (pin "J10")
+    (pin "J11")
+    (pin "J16")
+    (pin "J14")
+    (pin "J12")
+    (pin "J13")
+    (pin "J20")
+    (pin "J21")
+    (pin "J22")
+    (pin "J23")
+    (pin "J49")
+    (pin "J50")
+  )
+  (symbol (lib_id "rusefi_Molex_MRE_Connector:molex_48pin_MRE") (at 323.85 165.1 180) (unit 7)
+    (in_bom yes) (on_board yes)
+    (property "Reference" "U3" (id 0) (at 300.99 156.4386 0)
+      (effects (font (size 1.524 1.524)))
+    )
+    (property "Value" "molex_48pin_MRE" (id 1) (at 293.37 165.1 90)
+      (effects (font (size 1.524 1.524)) hide)
+    )
+    (property "Footprint" "rusefi_lib:Molex_48_MRE_R055" (id 2) (at 323.85 165.1 0)
+      (effects (font (size 1.524 1.524)) hide)
+    )
+    (property "Datasheet" "" (id 3) (at 323.85 165.1 0)
+      (effects (font (size 1.524 1.524)) hide)
+    )
+    (pin "1")
+    (pin "10")
+    (pin "11")
+    (pin "12")
+    (pin "13")
+    (pin "14")
+    (pin "15")
+    (pin "16")
+    (pin "17")
+    (pin "18")
+    (pin "19")
+    (pin "2")
+    (pin "20")
+    (pin "21")
+    (pin "22")
+    (pin "23")
+    (pin "24")
+    (pin "25")
+    (pin "26")
+    (pin "27")
+    (pin "28")
+    (pin "29")
+    (pin "3")
+    (pin "30")
+    (pin "31")
+    (pin "32")
+    (pin "33")
+    (pin "34")
+    (pin "35")
+    (pin "36")
+    (pin "37")
+    (pin "38")
+    (pin "39")
+    (pin "4")
+    (pin "40")
+    (pin "41")
+    (pin "42")
+    (pin "43")
+    (pin "44")
+    (pin "45")
+    (pin "46")
+    (pin "47")
+    (pin "48")
+    (pin "5")
+    (pin "6")
+    (pin "7")
+    (pin "8")
+    (pin "9")
+    (pin "M11")
+    (pin "M12")
+    (pin "M13")
+    (pin "M21")
+    (pin "M22")
+    (pin "M23")
+    (pin "M3")
+    (pin "M4")
+    (pin "M51")
+    (pin "M52")
+    (pin "M53")
+    (pin "M61")
+    (pin "M62")
+    (pin "M63")
+    (pin "M71")
+    (pin "M72")
+    (pin "M73")
+    (pin "J61")
+    (pin "J62")
+    (pin "J63")
+    (pin "J64")
+    (pin "J65")
+    (pin "J31")
+    (pin "J32")
+    (pin "J801")
+    (pin "J802")
+    (pin "J803")
+    (pin "J804")
+    (pin "J805")
+    (pin "J806")
+    (pin "J807")
+    (pin "J808")
+    (pin "J809")
+    (pin "J810")
+    (pin "LIN1")
+    (pin "J51")
+    (pin "J52")
+    (pin "J53")
+    (pin "J54")
+    (pin "J201")
+    (pin "J202")
+    (pin "J203")
+    (pin "J204")
+    (pin "J205")
+    (pin "J206")
+    (pin "J207")
+    (pin "J208")
+    (pin "J209")
+    (pin "J210")
+    (pin "J6")
+    (pin "J18")
+    (pin "J9")
+    (pin "J10")
+    (pin "J11")
+    (pin "J16")
+    (pin "J14")
+    (pin "J12")
+    (pin "J13")
+    (pin "J20")
+    (pin "J21")
+    (pin "J22")
+    (pin "J23")
+    (pin "J49")
+    (pin "J50")
   )
   (symbol (lib_id "Connector_Generic:Conn_02x05_Odd_Even") (at 302.895 146.685 180) (unit 1)
