File: SDCard.kicad_sch (KiCad schematic)
At the start: 2 parts

Commit message: R0.6.1rc KICAD6
Parts:
- removed C42: ~, symbol Device:C
- J14: footprint (none) -> Connector_Card:microSD_HC_Wuerth_693072010801
Changed lines of the file:
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@@
   (no_connect (at 104.14 125.095))
   (no_connect (at 104.14 107.315))
-  (wire (pts (xy 167.005 121.92) (xy 167.005 120.015))
-    (stroke (width 0) (type default) (color 0 0 0 0))
-  )
   (wire (pts (xy 148.59 131.445) (xy 148.59 130.175))
-    (stroke (width 0) (type default) (color 0 0 0 0))
-  )
-  (wire (pts (xy 167.005 107.95) (xy 167.005 112.395))
     (stroke (width 0) (type default) (color 0 0 0 0))
   )
@@
     (effects (font (size 1.27 1.27) (thickness 0.254) bold) (justify right))
   )
-  (hierarchical_label "VDD" (shape input) (at 167.005 107.95 0)
-    (effects (font (size 1.27 1.27) (thickness 0.254) bold) (justify left))
-  )
   (hierarchical_label "PC12" (shape input) (at 102.235 112.395 180)
     (effects (font (size 1.27 1.27) (thickness 0.254) bold) (justify right))
@@
     (effects (font (size 1.27 1.27) (thickness 0.254) bold) (justify right))
   )
-  (symbol (lib_id "power:GND") (at 167.005 121.92 0) (unit 1)
-    (in_bom yes) (on_board yes)
-    (property "Reference" "#PWR0130" (id 0) (at 167.005 128.27 0)
-      (effects (font (size 1.27 1.27)) hide)
-    )
-    (property "Value" "~" (id 1) (at 167.132 126.3142 0))
-    (property "Footprint" "" (id 2) (at 167.005 121.92 0)
-      (effects (font (size 1.27 1.27)) hide)
-    )
-    (property "Datasheet" "" (id 3) (at 167.005 121.92 0)
-      (effects (font (size 1.27 1.27)) hide)
-    )
-    (pin "1")
-  )
   (symbol (lib_id "Connector:Micro_SD_Card") (at 127 114.935 0) (unit 1)
     (in_bom yes) (on_board yes)
     (property "Reference" "J14" (id 0) (at 125.73 96.7232 0))
     (property "Value" "~" (id 1) (at 125.73 99.0346 0))
-    (property "Footprint" "" (id 2) (at 156.21 107.315 0)
+    (property "Footprint" "Connector_Card:microSD_HC_Wuerth_693072010801" (id 2) (at 156.21 107.315 0)
       (effects (font (size 1.27 1.27)) hide)
     )
@@
     (pin "9")
   )
-  (symbol (lib_id "Device:C") (at 167.005 116.205 180) (unit 1)
-    (in_bom yes) (on_board yes)
-    (property "Reference" "C42" (id 0) (at 164.084 117.3734 0)
-      (effects (font (size 1.27 1.27)) (justify left))
-    )
-    (property "Value" "~" (id 1) (at 164.084 115.062 0)
-      (effects (font (size 1.27 1.27)) (justify left))
-    )
-    (property "Footprint" "" (id 2) (at 166.0398 112.395 0)
-      (effects (font (size 1.27 1.27)) hide)
-    )
-    (property "Datasheet" "~" (id 3) (at 167.005 116.205 0)
-      (effects (font (size 1.27 1.27)) hide)
-    )
-    (property "Part #" "C0603C104J5RACTU" (id 4) (at 319.405 67.31 0)
-      (effects (font (size 1.27 1.27)) hide)
-    )
-    (property "VEND" "DIGI" (id 5) (at 319.405 67.31 0)
-      (effects (font (size 1.27 1.27)) hide)
-    )
-    (property "VEND#" "399-7844-1-ND" (id 6) (at 319.405 67.31 0)
-      (effects (font (size 1.27 1.27)) hide)
-    )
-    (property "Manufacturer" "KEMET" (id 7) (at 319.405 67.31 0)
-      (effects (font (size 1.27 1.27)) hide)
-    )
-    (property "LCSC" "C14663" (id 8) (at 167.005 116.205 0)
-      (effects (font (size 1.27 1.27)) hide)
-    )
-    (pin "1")
-    (pin "2")
-  )
   (symbol (lib_id "power:GND") (at 148.59 131.445 0) (unit 1)
